Commit message: updated x500 motor params

File: models/mrs_robots_description/urdf/x500.xacro (robot description, xacro)
@@ -37,5 +37,5 @@
   <!-- ================================================================== -->
   <!-- Robot parameters and arguments {-->
-  <xacro:property name="mass" value="3.5" /> <!-- [kg] --> <!-- TODO -->
+  <xacro:property name="mass" value="2.0" /> <!-- [kg] --> <!-- TODO -->
   <xacro:property name="body_radius" value="0.275" /> <!-- [m] -->
   <xacro:property name="body_height" value="0.15" /> <!-- [m] -->
@@ -52,5 +52,5 @@
   <!-- Motor constants {-->
   <xacro:property name="rotor_velocity_slowdown_sim" value="0.0159236" /> <!-- TODO -->
-  <xacro:property name="motor_constant" value="23.0" /> <!-- [kg.m/s^2] --> <!-- TODO -->
+  <xacro:property name="motor_constant" value="12.68433" /> <!-- [kg.m/s^2] --> <!-- TODO -->
   <xacro:property name="moment_constant" value="0.016" /> <!-- [m] --> <!-- TODO -->
   <xacro:property name="time_constant_up" value="${1.0 / 80.0}" /> <!-- [s] --> <!-- TODO -->

Commit message: added x500 ouster support

File: models/mrs_robots_description/urdf/x500.xacro (robot description, xacro)
@@ -177,33 +177,35 @@
   <!--}-->
   <!-- onboard computer (up! extreme) {-->
-  <xacro:visual_macro
-    robot_namespace="${namespace}"
-    name="pc_mount"
-    mesh_file="${pc_mount_mesh}"
-    mesh_scale="${mesh_scale}"
-    parent="base_link"
-    color="Default">
-    <origin xyz="0 0 0" rpy="0 0 0" />
-  </xacro:visual_macro>
-  <xacro:colored_box
-    robot_namespace="${namespace}"
-    name="computer_board"
-    size_x="0.125"
-    size_y="0.125"
-    size_z="0.002"
-    parent="base_link"
-    color="Grass">
-    <origin xyz="0 0 0.058" rpy="0 0 0" />
-  </xacro:colored_box>
-  <xacro:colored_box
-    robot_namespace="${namespace}"
-    name="computer_heatsink"
-    size_x="0.071"
-    size_y="0.071"
-    size_z="0.027"
-    parent="base_link"
-    color="Grey">
-    <origin xyz="0.009 0.012 0.074" rpy="0 0 0" />
-  </xacro:colored_box>
+  <xacro:unless value="${optionals['enable_ouster']}">
+    <xacro:visual_macro
+      robot_namespace="${namespace}"
+      name="pc_mount"
+      mesh_file="${pc_mount_mesh}"
+      mesh_scale="${mesh_scale}"
+      parent="base_link"
+      color="Default">
+      <origin xyz="0 0 0" rpy="0 0 0" />
+    </xacro:visual_macro>
+    <xacro:colored_box
+      robot_namespace="${namespace}"
+      name="computer_board"
+      size_x="0.125"
+      size_y="0.125"
+      size_z="0.002"
+      parent="base_link"
+      color="Grass">
+      <origin xyz="0 0 0.058" rpy="0 0 0" />
+    </xacro:colored_box>
+    <xacro:colored_box
+      robot_namespace="${namespace}"
+      name="computer_heatsink"
+      size_x="0.071"
+      size_y="0.071"
+      size_z="0.027"
+      parent="base_link"
+      color="Grey">
+      <origin xyz="0.009 0.012 0.074" rpy="0 0 0" />
+    </xacro:colored_box>
+  </xacro:unless>
   <!--}-->
   <!-- pixhawk {-->
@@ -581,3 +583,94 @@
   </xacro:if>
   <!--}-->
+  <!-- Ouster {-->
+  <xacro:if value="${optionals['enable_ouster']}">
+    <xacro:property name="ouster_model" value="${optionals['ouster_model']}" />
+    <!-- OS1-16 Generation 1 (default) -->
+    <xacro:property name="lasers" value="16" />
+    <xacro:property name="vfov_angle" value="33.2" />
+    <xacro:property name="range" value="120" />
+    <xacro:if value="${ouster_model == 'OS1-16'}">
+      <xacro:property name="lasers" value="16" />
+      <xacro:property name="vfov_angle" value="33.2" />
+      <xacro:property name="range" value="120" />
+    </xacro:if>
+    <!-- OS0 {-->
+    <!-- OS0-32 -->
+    <xacro:if value="${ouster_model == 'OS0-32'}">
+      <xacro:property name="lasers" value="32" />
+      <xacro:property name="vfov_angle" value="90" />
+      <xacro:property name="range" value="55" />
+    </xacro:if>
+    <!-- OS0-64 -->
+    <xacro:if value="${ouster_model == 'OS0-64'}">
+      <xacro:property name="lasers" value="64" />
+      <xacro:property name="vfov_angle" value="90" />
+      <xacro:property name="range" value="55" />
+    </xacro:if>
+    <!-- OS0-128 -->
+    <xacro:if value="${ouster_model == 'OS0-128'}">
+      <xacro:property name="lasers" value="128" />
+      <xacro:property name="vfov_angle" value="90" />
+      <xacro:property name="range" value="55" />
+    </xacro:if>
+    <!--}-->
+    <!-- OS1 Generation 2 {-->
+    <!-- OS1-32 Generation 2 -->
+    <xacro:if value="${ouster_model == 'OS1-32'}">
+      <xacro:property name="lasers" value="32" />
+      <xacro:property name="vfov_angle" value="45" />
+      <xacro:property name="range" value="120" />
+    </xacro:if>
+    <!-- OS1-64 Generation 2 -->
+    <xacro:if value="${ouster_model == 'OS1-64'}">
+      <xacro:property name="lasers" value="64" />
+      <xacro:property name="vfov_angle" value="45" />
+      <xacro:property name="range" value="120" />
+    </xacro:if>
+    <!-- OS1-128 Generation 2 -->
+    <xacro:if value="${ouster_model == 'OS1-128'}">
+      <xacro:property name="lasers" value="128" />
+      <xacro:property name="vfov_angle" value="45" />
+      <xacro:property name="range" value="120" />
+    </xacro:if>
+    <!--}-->
+    <!-- OS2 {-->
+    <!-- OS2-32 -->
+    <xacro:if value="${ouster_model == 'OS2-32'}">
+      <xacro:property name="lasers" value="32" />
+      <xacro:property name="vfov_angle" value="22.5" />
+      <xacro:property name="range" value="240" />
+    </xacro:if>
+    <!-- OS2-64 -->
+    <xacro:if value="${ouster_model == 'OS2-64'}">
+      <xacro:property name="lasers" value="64" />
+      <xacro:property name="vfov_angle" value="22.5" />
+      <xacro:property name="range" value="240" />
+    </xacro:if>
+    <!-- OS2-128 -->
+    <xacro:if value="${ouster_model == 'OS2-128'}">
+      <xacro:property name="lasers" value="128" />
+      <xacro:property name="vfov_angle" value="22.5" />
+      <xacro:property name="range" value="240" />
+    </xacro:if>
+    <!--}-->
+  <xacro:ouster_macro
+    namespace="${namespace}"
+    sensor_name="os"
+    x="0"
+    y="0"
+    z="0.066"
+    roll="0"
+    pitch="0"
+    yaw="0"
+    rot_freq="10"
+    lasers="${lasers}"
+    vfov_angle="${vfov_angle}"
+    max_range="${range}"
+    noise="0.03"
+    enable_gpu_ray="${optionals['use_gpu_ray']}"
+    >
+  </xacro:ouster_macro>
+  </xacro:if>
+  <!--}-->
 </robot>
