Commit message: update motor constants

File: models/mrs_robots_description/urdf/naki.xacro (robot description, xacro)
@@ -37,5 +37,5 @@
   <!-- ================================================================== -->
   <!-- Robot parameters and arguments {-->
-  <xacro:property name="mass" value="5.00" /> <!-- [kg] -->
+  <xacro:property name="mass" value="7.00" /> <!-- [kg] -->
   <xacro:property name="body_radius" value="0.29" /> <!-- [m] -->
   <xacro:property name="body_height" value="0.45" /> <!-- [m] -->
@@ -56,5 +56,5 @@
   <!-- Motor constants {-->
   <xacro:property name="rotor_velocity_slowdown_sim" value="0.0159236" />
-  <xacro:property name="motor_constant" value="10.04544" /> <!-- [kg.m/s^2] -->
+  <xacro:property name="motor_constant" value="23.44" /> <!-- [N] -->
   <xacro:property name="moment_constant" value="0.016" /> <!-- [m] -->
   <xacro:property name="time_constant_up" value="${1.0 / 80.0}" /> <!-- [s] -->
