Commit message: added OS1-32g1

File: models/mrs_robots_description/urdf/t650.xacro (robot description, xacro)
@@ -596,4 +596,11 @@
       <xacro:property name="sensor_name" value="os1" />
       <xacro:property name="lasers" value="16" />
+      <xacro:property name="vfov_angle" value="33.2" />
+      <xacro:property name="range" value="120" />
+    </xacro:if>
+    <!-- OS1-32 Generation 1 -->
+    <xacro:if value="${ouster_model == 'OS1-32G1'}">
+      <xacro:property name="sensor_name" value="os1" />
+      <xacro:property name="lasers" value="32" />
       <xacro:property name="vfov_angle" value="33.2" />
       <xacro:property name="range" value="120" />

Commit message: working t650

File: models/mrs_robots_description/urdf/t650.xacro (robot description, xacro)
@@ -6,4 +6,6 @@
   -->
   <xacro:property name="namespace" value="$(arg namespace)" />
+  <xacro:property name='model_params_file' value="$(arg model_params_file)"/>
+  <xacro:property name="optionals" value="${load_yaml(model_params_file)}" />
   <xacro:arg name='name' default='t650' />
   <xacro:arg name='mavlink_addr' default='INADDR_ANY' />
@@ -484,5 +486,5 @@
   <!-- ================================================================== -->
   <!-- Ground truth {-->
-  <xacro:if value="$(arg enable_ground_truth)">
+  <xacro:if value="${optionals['enable_ground_truth']}">
     <xacro:odometry_plugin_macro
       namespace="${namespace}"
@@ -503,5 +505,5 @@
   <!-- ======================= rangefinder sensors ======================-->
   <!-- Garmin {-->
-  <xacro:if value="$(arg enable_rangefinder)">
+  <xacro:if value="${optionals['enable_rangefinder']}">
     <xacro:garmin_macro
       namespace="${namespace}"
@@ -519,5 +521,5 @@
   <!--}-->
   <!-- Garmin looking up {-->
-  <xacro:if value="$(arg enable_rangefinder_up)">
+  <xacro:if value="${optionals['enable_rangefinder_up']}">
     <xacro:garmin_macro
       namespace="${namespace}"
@@ -536,5 +538,5 @@
   <!-- ========================== LIDAR sensors ========================= -->
   <!-- Scanse Sweep {-->
-  <xacro:if value="$(arg enable_scanse_sweep)">
+  <xacro:if value="${optionals['enable_scanse_sweep']}">
     <xacro:scanse_sweep_macro
       namespace="${namespace}"
@@ -550,5 +552,5 @@
   <!--}-->
   <!-- Rplidar {-->
-  <xacro:if value="$(arg enable_rplidar)">
+  <xacro:if value="${optionals['enable_rplidar']}">
     <xacro:rplidar_macro
       namespace="${namespace}"
@@ -564,5 +566,5 @@
   <!--}-->
   <!-- Velodyne  {-->
-  <xacro:if value="$(arg enable_velodyne)">
+  <xacro:if value="${optionals['enable_velodyne']}">
     <!-- VLP-16 (default) -->
     <xacro:property name="sensor_name" value="velodyne" />
@@ -584,5 +586,5 @@
       max_range="${range}"
       noise="0.01"
-      enable_gpu_ray="$(arg use_gpu_ray)"
+      enable_gpu_ray="${optionals['use_gpu_ray']}"
       >
     </xacro:velodyne_macro>
@@ -590,6 +592,6 @@
   <!--}-->
   <!-- Ouster {-->
-  <xacro:if value="$(arg enable_ouster)">
-  <xacro:property name="ouster_model" value="$(arg ouster_model)" />
+  <xacro:if value="${optionals['enable_ouster']}">
+  <xacro:property name="ouster_model" value="${optionals['ouster_model']}" />
     <!-- OS1-16 Generation 1 (default) -->
     <xacro:property name="sensor_name" value="os1" />
@@ -693,5 +695,5 @@
     max_range="${range}"
     noise="0.03"
-    enable_gpu_ray="$(arg use_gpu_ray)"
+    enable_gpu_ray="${optionals['use_gpu_ray']}"
     >
   </xacro:ouster_macro>
@@ -701,5 +703,5 @@
   <!-- Bluefox placements{-->
   <!-- reverse {-->
-  <xacro:if value="$(arg enable_bluefox_camera_reverse)">
+  <xacro:if value="${optionals['enable_bluefox_camera_reverse']}">
     <xacro:bluefox_camera_macro
       namespace="${namespace}"
@@ -723,5 +725,5 @@
   <!--}-->
   <!-- classic {-->
-  <xacro:if value="$(arg enable_bluefox_camera)">
+  <xacro:if value="${optionals['enable_bluefox_camera']}">
     <xacro:bluefox_camera_macro
       namespace="${namespace}"
@@ -747,5 +749,5 @@
   <!-- Realsense placements {-->
   <!-- front {-->
-  <xacro:if value="$(arg enable_realsense_front)">
+  <xacro:if value="${optionals['enable_realsense_front']}">
     <!-- sensor -->
     <xacro:realsense_macro
@@ -754,5 +756,5 @@
       camera_suffix="realsense_front"
       parent_frame_name="${namespace}/fcu"
-      enable_realistic_realsense="$(arg use_realistic_realsense)"
+      enable_realistic_realsense="${optionals['use_realistic_realsense']}"
       x="0.17"
       y="-0.011"
@@ -765,5 +767,5 @@
   <!--}-->
   <!-- up {-->
-  <xacro:if value="$(arg enable_realsense_up)">
+  <xacro:if value="${optionals['enable_realsense_up']}">
     <!-- sensor -->
     <xacro:realsense_macro
@@ -772,5 +774,5 @@
       camera_suffix="realsense_up"
       parent_frame_name="${namespace}/fcu"
-      enable_realistic_realsense="$(arg use_realistic_realsense)"
+      enable_realistic_realsense="${optionals['use_realistic_realsense']}"
       x="0.08"
       y="0"
@@ -785,5 +787,5 @@
   <!-- Mobius placements {-->
   <!-- front {-->
-  <xacro:if value="$(arg enable_mobius_camera_front)">
+  <xacro:if value="${optionals['enable_mobius_camera_front']}">
     <xacro:mobius_camera_macro
       namespace="${namespace}"
@@ -806,5 +808,5 @@
   <!--} mobius placements -->
   <!-- Thermal camera {-->
-  <xacro:if value="$(arg enable_thermal_camera)">
+  <xacro:if value="${optionals['enable_thermal_camera']}">
     <!-- top -->
     <xacro:thermal_camera_macro
@@ -873,5 +875,5 @@
   <!--}-->
   <!-- UV camera {-->
-  <xacro:if value="$(arg enable_uv_camera)">
+  <xacro:if value="${optionals['enable_uv_camera']}">
     <xacro:uvcam_macro
       namespace="${namespace}"
@@ -880,5 +882,5 @@
       frame_rate="80"
       camera_publish_topic="/${namespace}/uvdar_bluefox_left/image_raw"
-      calibration_file="$(arg uvcam_calib_file)">
+      calibration_file="${optionals['uvcam_calib_file']}">
     <origin xyz="0.037 0.1175 0.057" rpy="0 0 ${rad70}" />
     </xacro:uvcam_macro>
@@ -889,5 +891,5 @@
       frame_rate="80"
       camera_publish_topic="/${namespace}/uvdar_bluefox_right/image_raw"
-      calibration_file="$(arg uvcam_calib_file)">
+      calibration_file="${optionals['uvcam_calib_file']}">
     <origin xyz="0.037 -0.1175 0.057" rpy="0 0 -${rad70}" />
     </xacro:uvcam_macro>
@@ -895,5 +897,5 @@
   <!--}-->
   <!-- Servo camera {-->
-  <xacro:if value="$(arg enable_servo_camera)">
+  <xacro:if value="${optionals['enable_servo_camera']}">
     <xacro:servo_camera_macro
       namespace="${namespace}"
@@ -914,5 +916,5 @@
   <!-- ========================== other sensors ========================= -->
   <!-- Teraranger Tower Evo {-->
-  <xacro:if value="$(arg enable_teraranger_tower_evo)">
+  <xacro:if value="${optionals['enable_teraranger_tower_evo']}">
     <xacro:teraranger_tower_evo_macro
       namespace="${namespace}"
@@ -926,5 +928,5 @@
   <!--}-->
   <!-- Magnetic gripper {-->
-  <xacro:if value="$(arg enable_magnetic_gripper)">
+  <xacro:if value="${optionals['enable_magnetic_gripper']}">
     <xacro:magnet_gripper_macro
       namespace="${namespace}"
@@ -937,5 +939,5 @@
   <!--}-->
   <!-- Timepix {-->
-  <xacro:if value="$(arg enable_timepix)">
+  <xacro:if value="${optionals['enable_timepix']}">
     <xacro:timepix_macro
       namespace="${namespace}"
@@ -948,5 +950,5 @@
   <!--}-->
 <!-- Water gun {-->
-<xacro:if value="$(arg enable_water_gun)">
+<xacro:if value="${optionals['enable_water_gun']}">
   <xacro:water_gun_macro
     namespace="${namespace}"
@@ -1016,8 +1018,8 @@
   </xacro:macro>
   <!--}-->
-  <xacro:if value="$(arg enable_uv_leds)">
+  <xacro:if value="${optionals['enable_uv_leds']}">
     <xacro:uvled_hexarotor
-      f1="$(arg uvled_fr_l)"
-      f2="$(arg uvled_fr_r)"
+      f1="${optionals['uvled_fr_l']}"
+      f2="${optionals['uvled_fr_r']}"
       namespace="${namespace}"
       parent_link="base_link"/>
@@ -1025,5 +1027,5 @@
   <!--}-->
   <!-- Light {-->
-  <xacro:if value="$(arg enable_light)">
+  <xacro:if value="${optionals['enable_light']}">
     <xacro:light_macro
       namespace="${namespace}"
@@ -1047,5 +1049,5 @@
   <!-- ============================= holders ============================ -->
   <!-- Ouster and Velodyne mount {-->
-  <xacro:if value="${('$(arg enable_ouster)' == 'true') or ('$(arg enable_velodyne)' == 'true')}">
+  <xacro:if value="${(optionals['enable_ouster'] == 'true') or (optionals['enable_velodyne'] == 'true')}">
     <xacro:visual_macro
       robot_namespace="${namespace}"
@@ -1060,5 +1062,5 @@
   <!--}-->
   <!-- Rplidar and scanse mount {-->
-  <xacro:if value="${('$(arg enable_rplidar)' == 'true') or ('$(arg enable_scanse_sweep)' == 'true')}">
+  <xacro:if value="${(optionals['enable_rplidar'] == 'true') or (optionals['enable_scanse_sweep'] == 'true')}">
     <xacro:visual_macro
       robot_namespace="${namespace}"
@@ -1073,5 +1075,5 @@
   <!--}-->
   <!-- Realsense front mount {-->
-  <xacro:if value="$(arg enable_realsense_front)">
+  <xacro:if value="${optionals['enable_realsense_front']}">
     <xacro:visual_macro
       robot_namespace="${namespace}"
@@ -1086,5 +1088,5 @@
   <!--}-->
   <!-- Bluefox and garmin mount {-->
-  <xacro:if value="${('$(arg enable_bluefox_camera)' == 'true') or ('$(arg enable_bluefox_camera_reverse)' == 'true') or ('$(arg enable_rangefinder)' == 'true') or ('$(arg wall_challenge)' == 'true')}">
+  <xacro:if value="${(optionals['enable_bluefox_camera'] == 'true') or (optionals['enable_bluefox_camera_reverse'] == 'true') or (optionals['enable_rangefinder'] == 'true') or (optionals['wall_challenge'] == 'true')}">
     <xacro:visual_macro
       robot_namespace="${namespace}"
@@ -1099,5 +1101,5 @@
   <!--}-->
   <!-- UVDAR mount {-->
-  <xacro:if value="$(arg enable_uv_camera)">
+  <xacro:if value="${optionals['enable_uv_camera']}">
     <xacro:visual_macro
       robot_namespace="${namespace}"
@@ -1113,5 +1115,5 @@
   <!-- ========================== other sensors ========================= -->
 <!-- Parachute {-->
-<xacro:if value="$(arg enable_parachute)">
+<xacro:if value="${optionals['enable_parachute']}">
   <xacro:parachute_macro
     namespace="${namespace}"
@@ -1127,5 +1129,5 @@
 <!--}-->
   <!-- Pendulum {-->
-  <xacro:if value="$(arg enable_pendulum)">
+  <xacro:if value="${optionals['enable_pendulum']}">
     <xacro:pendulum
       parent="base_link">
@@ -1134,5 +1136,5 @@
   <!--}-->
   <!-- Ball holder {-->
-  <xacro:if value="$(arg enable_ball_holder)">
+  <xacro:if value="${optionals['enable_ball_holder']}">
     <xacro:ball_holder
       parent="base_link">
@@ -1142,5 +1144,5 @@
   <!-- MBZIRC profiles {-->
   <!-- Wall challenge {-->
-  <xacro:if value="$(arg wall_challenge)">
+  <xacro:if value="${optionals['wall_challenge']}">
     <!-- Garmin {-->
     <xacro:garmin_macro
@@ -1203,5 +1205,5 @@
       camera_suffix="realsense_down"
       parent_frame_name="${namespace}/fcu"
-      enable_realistic_realsense="$(arg use_realistic_realsense)"
+      enable_realistic_realsense="${optionals['use_realistic_realsense']}"
       x="0.15"
       y="0.15"
@@ -1216,5 +1218,5 @@
   <!--}-->
   <!-- Fire challenge (blanket dropping) {-->
-  <xacro:if value="$(arg fire_challenge_blanket)">
+  <xacro:if value="${optionals['fire_challenge_blanket']}">
     <!-- Garmin {-->
     <xacro:garmin_macro

Commit message: Adding the downward UVDAR

File: models/mrs_robots_description/urdf/t650.xacro (robot description, xacro)
@@ -1172,17 +1172,17 @@
   </xacro:if>
   <!--}-->
-  <!-- UVDAR mount {-->
-  <xacro:if value="${optionals['enable_uv_camera']}">
-    <xacro:visual_macro
-      robot_namespace="${namespace}"
-      name="uvdar_mount"
-      mesh_file="${uvdar_mount_mesh}"
-      mesh_scale="${mesh_scale_milimeters}"
-      parent="base_link"
-      color="DarkGrey">
-    <origin xyz="0.025 0 0.043" rpy="0 0 0" />
-    </xacro:visual_macro>
-  </xacro:if>
-  <!--}-->
+  <!--<!-1- Downward UVDAR mount {-1->-->
+  <!--<xacro:if value="${optionals['enable_uv_camera']}">-->
+  <!--  <xacro:visual_macro-->
+  <!--    robot_namespace="${namespace}"-->
+  <!--    name="uvdar_mount"-->
+  <!--    mesh_file="${uvdar_mount_mesh}"-->
+  <!--    mesh_scale="${mesh_scale_milimeters}"-->
+  <!--    parent="base_link"-->
+  <!--    color="DarkGrey">-->
+  <!--  <origin xyz="0.025 0 0.043" rpy="0 0 0" />-->
+  <!--  </xacro:visual_macro>-->
+  <!--</xacro:if>-->
+  <!--<!-1-}-1->-->
   <!-- ========================== other sensors ========================= -->
 <!-- Parachute {-->
@@ -1363,3 +1363,17 @@
   <!--}-->
   <!--}-->
+  <!-- Downward UV cameras {-->
+  <xacro:if value="${optionals['enable_downward_uv_camera']}">
+    <xacro:uvcam_macro
+      namespace="${namespace}"
+      parent_link="base_link"
+      number="1"
+      frame_rate="60"
+      camera_publish_topic="/${namespace}/uvdar_bluefox_bottom/image_raw"
+      calibration_file="${optionals['uvcam_calib_file']}"
+      occlusions="${optionals['uvcam_occlusions']}">
+    <origin xyz="0.0 0.0 -0.10" rpy="0 ${rad90} 0" />
+    </xacro:uvcam_macro>
+  </xacro:if>
+  <!--}-->
 </robot>

Commit message: partial merge of marine branch

File: models/mrs_robots_description/urdf/t650.xacro (robot description, xacro)
@@ -1350,3 +1350,17 @@
   <!--}-->
   <!--}-->
+  <!-- Downward UV cameras {-->
+  <xacro:if value="${optionals['enable_downward_uv_camera']}">
+    <xacro:uvcam_macro
+      namespace="${namespace}"
+      parent_link="base_link"
+      number="1"
+      frame_rate="60"
+      camera_publish_topic="/${namespace}/uvdar_bluefox_bottom/image_raw"
+      calibration_file="${optionals['uvcam_calib_file']}"
+      occlusions="${optionals['uvcam_occlusions']}">
+    <origin xyz="0.0 0.0 -0.10" rpy="0 ${rad90} 0" />
+    </xacro:uvcam_macro>
+  </xacro:if>
+  <!--}-->
 </robot>
