Commit message: Add servo camera and light into robots components

File: models/mrs_robots_description/urdf/component_snippets.xacro (robot description, xacro)
@@ -1748,5 +1748,5 @@
       </link>
       <gazebo>
-        <plugin name="servo_camera_plugin" filename="libservo_camera_plugin.so">
+        <plugin name="servo_camera_plugin" filename="libMRSGazeboServoCameraPlugin.so">
           <offset_x>${offset_x}</offset_x>
           <offset_y>${offset_y}</offset_y>
@@ -2069,5 +2069,5 @@
       </link>
       <gazebo>
-        <plugin name="light_gazebo_plugin" filename="liblight_gazebo_plugin.so">
+        <plugin name="light_gazebo_plugin" filename="libMRSGazeboLightPlugin.so">
           <offset_x>${offset_x}</offset_x>
           <offset_y>${offset_y}</offset_y>

File: models/mrs_robots_description/urdf/f450.xacro (robot description, xacro)
@@ -935,4 +935,22 @@
   </xacro:if>
   <!--}-->
+  <!-- Servo camera {-->
+  <xacro:if value="$(arg enable_servo_camera)">
+    <xacro:servo_camera_macro
+      namespace="${namespace}"
+      name="servo_camera_macro"
+      parent="base_link"
+      offset_x="0.2"
+      offset_y="0.0"
+      offset_z="-0.10"
+      offset_roll="0.0"
+      offset_yaw="0.0"
+      offset_pitch="0.0"
+      max_pitch_rate="0.1"
+      camera_type="servo_camera"
+      update_rate="30.0">
+    </xacro:servo_camera_macro>
+  </xacro:if>
+  <!--}-->
   <!-- ========================== other sensors ========================= -->
   <!-- Teraranger Tower Evo {-->
@@ -1047,5 +1065,5 @@
       name="light_macro"
       parent="base_link"
-      offset_x="0.16"
+      offset_x="0.2"
       offset_y="0.0"
       offset_z="-0.10"
@@ -1054,7 +1072,6 @@
       offset_pitch="0.0"
       max_pitch_rate="0.1"
-      initial_on="0"
+      initial_on="1"
       update_rate="30.0">
-      <origin xyz="0 0 0" rpy="0 0 0" />
     </xacro:light_macro>
   </xacro:if>

File: models/mrs_robots_description/urdf/t650.xacro (robot description, xacro)
@@ -865,4 +865,22 @@
   </xacro:if>
   <!--}-->
+  <!-- Servo camera {-->
+  <xacro:if value="$(arg enable_servo_camera)">
+    <xacro:servo_camera_macro
+      namespace="${namespace}"
+      name="servo_camera_macro"
+      parent="base_link"
+      offset_x="0.2"
+      offset_y="0.0"
+      offset_z="-0.10"
+      offset_roll="0.0"
+      offset_yaw="0.0"
+      offset_pitch="0.0"
+      max_pitch_rate="0.1"
+      camera_type="servo_camera"
+      update_rate="30.0">
+    </xacro:servo_camera_macro>
+  </xacro:if>
+  <!--}-->
   <!-- ========================== other sensors ========================= -->
   <!-- Teraranger Tower Evo {-->
@@ -976,4 +994,22 @@
       namespace="${namespace}"
       parent_link="base_link"/>
+  </xacro:if>
+  <!--}-->
+  <!-- Light {-->
+  <xacro:if value="$(arg enable_light)">
+    <xacro:light_macro
+      namespace="${namespace}"
+      name="light_macro"
+      parent="base_link"
+      offset_x="0.2"
+      offset_y="0.0"
+      offset_z="-0.10"
+      offset_roll="0.0"
+      offset_yaw="0.0"
+      offset_pitch="0.0"
+      max_pitch_rate="0.1"
+      initial_on="1"
+      update_rate="30.0">
+    </xacro:light_macro>
   </xacro:if>
   <!--}-->

Commit message: update pluginized components

File: models/mrs_robots_description/urdf/component_snippets.xacro (robot description, xacro)
@@ -2012,5 +2012,9 @@
     </gazebo>
     <gazebo>
-      <plugin name="gazebo_timepix" filename="libgazebo_timepix.so" />
+      <plugin name="gazebo_timepix" filename="libgazebo_timepix.so" >
+        <exposition_time>0.1</exposition_time>  <!-- [s] -->
+        <material>si</material>                 <!-- string -->
+        <size>0.0003 0.01408 0.01408</size>     <!-- [m m m] -->
+      </plugin>
     </gazebo>
   </xacro:macro>
@@ -2035,5 +2039,5 @@
     </gazebo>
     <gazebo>
-      <plugin name="water_gun_plugin" filename="libwater_gun_plugin.so">
+      <plugin name="water_gun_plugin" filename="libMRSGazeboWaterGunPlugin.so">
         <muzzle_velocity>${muzzle_velocity}</muzzle_velocity>
         <offset_x>${offset_x}</offset_x>
@@ -2172,5 +2176,5 @@
     </gazebo>
     <gazebo>
-      <plugin name="parachute_plugin" filename="libparachute_plugin.so">
+      <plugin name="parachute_plugin" filename="libMRSGazeboParachutePlugin.so">
         <air_density>1.225</air_density>
         <drag_coeff>500</drag_coeff>

Commit message: added mash for terabee thermal camera

File: models/mrs_robots_description/urdf/component_snippets.xacro (robot description, xacro)
@@ -1634,7 +1634,7 @@
     <link name="${namespace}/${camera_frame_name}/thermal_camera_link">
       <visual>
-        <origin xyz="0 0 0" rpy="${rad90} 0 0" />
-        <geometry>
-          <mesh filename="package://mrs_robots_description/meshes/sensors/bluefox.dae" scale="1 1 1" />
+        <origin xyz="0 0 0" rpy="0 0 0" />
+        <geometry>
+          <mesh filename="package://mrs_robots_description/meshes/sensors/teraranger_evo_thermal_33.dae" scale="0.001 0.001 0.001" />
         </geometry>
       </visual>

Commit message: add diagnostics topic sdf param to 3d lidars (velodyne and ouster)

File: models/mrs_robots_description/urdf/component_snippets.xacro (robot description, xacro)
@@ -1075,4 +1075,5 @@
   <xacro:macro name="velodyne_macro" params="namespace sensor_name x y z yaw pitch roll rot_freq lasers max_range noise vfov_angle enable_gpu_ray">
     <xacro:property name="topic_lidar" value="/${namespace}/${sensor_name}/scan" />
+    <xacro:property name="topic_diag" value="/${namespace}/${sensor_name}/diag" />
     <xacro:property name="frame_sensor" value="${namespace}/${sensor_name}_sensor" />
     <xacro:property name="frame_lidar" value="${namespace}/${sensor_name}" />
@@ -1174,4 +1175,5 @@
           <lidar_yaw>0</lidar_yaw>
           <topicName>${topic_lidar}</topicName>
+          <topicDiagName>${topic_diag}</topicDiagName>
           <lidarFrameName>${frame_lidar}</lidarFrameName>
           <min_range>0.1</min_range>
@@ -1203,4 +1205,5 @@
     <xacro:property name="topic_lidar" value="/${namespace}/${sensor_name}_cloud_node/points" />
     <xacro:property name="topic_imu" value="/${namespace}/${sensor_name}_cloud_node/imu" />
+    <xacro:property name="topic_diag" value="/${namespace}/${sensor_name}_cloud_node/diag" />
       <!-- tf from sensor to lidar -->
     <xacro:property name="lidar_x" value="0" />
@@ -1311,4 +1314,5 @@
           <lidar_yaw>${lidar_yaw}</lidar_yaw>
           <topicName>${topic_lidar}</topicName>
+          <topicDiagName>${topic_diag}</topicDiagName>
           <min_range>0.1</min_range>
           <max_range>${max_range}</max_range>

Commit message: modified water gun and fire_challenge settings

File: models/mrs_robots_description/urdf/component_snippets.xacro (robot description, xacro)
@@ -1689,5 +1689,5 @@
       </sensor>
     </gazebo>
-    <gazebo reference="${namespace}/thermal_camera_link">
+    <gazebo reference="${namespace}/${camera_frame_name}/thermal_camera_link">
       <material>Gazebo/${color}</material>
     </gazebo>
@@ -2026,13 +2026,22 @@
   <!--}-->
   <!-- Macro to add a water gun {-->
-  <xacro:macro name="water_gun_macro" params="namespace name parent muzzle_velocity particle_capacity spread color spawning_reservoir offset_x offset_y offset_z size_x size_y size_z *origin">
-    <joint name="${name}_joint" type="fixed">
+  <xacro:macro name="water_gun_macro" params="namespace name parent muzzle_velocity particle_capacity spread spawning_reservoir offset_x offset_y offset_z size_x size_y size_z *origin">
+    <joint name="${name}_body_joint" type="fixed">
       <xacro:insert_block name="origin" />
       <parent link="${parent}" />
-      <child link="${name}_link" />
-    </joint>
-    <link name="${name}_link">
-      <visual>
-        <origin xyz="${offset_x - size_x} ${offset_y} ${offset_z}" rpy="0 0 0" />
+      <child link="${name}_body_link" />
+    </joint>
+    <joint name="${name}_bag_joint" type="fixed">
+      <parent link="${name}_body_link" />
+      <child link="${name}_bag_link" />
+    </joint>
+    <joint name="${name}_nozzle_joint" type="fixed">
+      <origin xyz="${offset_x - 0.08/2} ${offset_y} ${offset_z - 0.006/2}" rpy="0 ${rad90} 0" />
+      <parent link="${parent}" />
+      <child link="${name}_nozzle_link" />
+    </joint>
+    <link name="${name}_body_link"/>
+    <link name="${name}_bag_link">
+      <visual>
         <geometry>
           <box size="${size_x} ${size_y} ${size_z}" />
@@ -2040,6 +2049,16 @@
       </visual>
     </link>
-    <gazebo reference="${name}_link">
-      <material>Gazebo/${color}</material>
+    <gazebo reference="${name}_bag_link">
+      <material>Gazebo/Blue</material>
+    </gazebo>
+    <link name="${name}_nozzle_link">
+      <visual>
+        <geometry>
+          <cylinder length="0.08" radius="0.006" />
+        </geometry>
+      </visual>
+    </link>
+    <gazebo reference="${name}_nozzle_link">
+      <material>Gazebo/DarkGrey</material>
     </gazebo>
     <gazebo>

File: models/mrs_robots_description/urdf/t650.xacro (robot description, xacro)
@@ -789,7 +789,7 @@
       image_width="32"
       image_height="32"
-      x="0.13"
-      y="0"
-      z="-0.085"
+      x="0.15"
+      y="0.06"
+      z="-0.025"
       roll="0"
       pitch="-${rad30}"
@@ -797,5 +797,5 @@
       parent_frame_name="${namespace}/fcu"
       sensor_base_frame_name="${namespace}/thermal/top"
-      color="Yellow">
+      color="DarkGrey">
     </xacro:thermal_camera_macro>
     <!-- middle -->
@@ -810,7 +810,7 @@
       image_width="32"
       image_height="32"
-      x="0.13"
-      y="0"
-      z="-0.085"
+      x="0.16"
+      y="0.06"
+      z="-0.055"
       roll="0"
       pitch="0"
@@ -818,5 +818,5 @@
       parent_frame_name="${namespace}/fcu"
       sensor_base_frame_name="${namespace}/thermal/middle"
-      color="Yellow">
+      color="DarkGrey">
     </xacro:thermal_camera_macro>
     <!-- bottom -->
@@ -831,6 +831,6 @@
       image_width="32"
       image_height="32"
-      x="0.13"
-      y="0"
+      x="0.15"
+      y="0.06"
       z="-0.085"
       roll="0"
@@ -839,5 +839,5 @@
       parent_frame_name="${namespace}/fcu"
       sensor_base_frame_name="${namespace}/thermal/bottom"
-      color="Yellow">
+      color="DarkGrey">
     </xacro:thermal_camera_macro>
   </xacro:if>
@@ -922,18 +922,17 @@
   <xacro:water_gun_macro
     namespace="${namespace}"
-    name="water_gun_macro"
+    name="water_gun"
     parent="base_link"
-    color="Red"
-    muzzle_velocity="10.0"
+    muzzle_velocity="15.0"
     particle_capacity="30"
     spread="1.0"
     spawning_reservoir="the_void"
-    offset_x="0.2"
+    offset_x="0.21"
     offset_y="0.0"
-    offset_z="-0.1"
+    offset_z="-0.085"
     size_x="0.2"
-    size_y="0.05"
-    size_z="0.05">
-  <origin xyz="0 0 0" rpy="0 0 0" />
+    size_y="0.08"
+    size_z="0.03">
+  <origin xyz="0 0 -0.11" rpy="0 0 0" />
 </xacro:water_gun_macro>
   </xacro:if>
@@ -1187,144 +1186,4 @@
   </xacro:if>
   <!--}-->
-  <!-- Fire challenge {-->
-  <xacro:if value="$(arg fire_challenge)">
-    <!-- Garmin {-->
-    <xacro:garmin_macro
-      namespace="${namespace}"
-      parent_link="base_link"
-      orientation=""
-      x="0.177"
-      y="0.0735"
-      z="-0.07"
-      roll="0"
-      pitch="1.57079632679"
-      yaw="0"
-      >
-    </xacro:garmin_macro>
-    <!--}-->
-    <!-- Garmin up {-->
-    <xacro:garmin_macro
-      namespace="${namespace}"
-      parent_link="base_link"
-      orientation="_up"
-      x="0.0"
-      y="-0.08"
-      z="0.01"
-      roll="0"
-      pitch="-1.57079632679"
-      yaw="0"
-      >
-    </xacro:garmin_macro>
-    <!--}-->
-    <!-- Rplidar {-->
-    <xacro:rplidar_macro
-      namespace="${namespace}"
-      x="0.0"
-      y="0.0"
-      z="0.205"
-      roll="0"
-      pitch="0"
-      yaw="0"
-      >
-    </xacro:rplidar_macro>
-    <!--}-->
-    <!-- Realsense front {-->
-    <xacro:realsense_macro
-      namespace="${namespace}"
-      parent_link="base_link"
-      camera_suffix="realsense_front"
-      parent_frame_name="${namespace}/fcu"
-      enable_realistic_realsense="$(arg use_realistic_realsense)"
-      x="0.184"
-      y="0"
-      z="-0.04"
-      roll="0"
-      pitch="0"
-      yaw="0">
-    </xacro:realsense_macro>
-    <!--}-->
-    <!-- Thermal camera {-->
-    <xacro:thermal_camera_macro
-      namespace="${namespace}"
-      camera_frame_name="thermal/top_optical"
-      camera_topic_name="/${namespace}/thermal/top"
-      parent_link="base_link"
-      camera_suffix="thermal/top"
-      frame_rate="14.0"
-      hfov="0.575959"
-      image_width="32"
-      image_height="32"
-      x="0.13"
-      y="0.055"
-      z="-0.085"
-      roll="0"
-      pitch="-0.523598776"
-      yaw="0"
-      parent_frame_name="${namespace}/fcu"
-      sensor_base_frame_name="${namespace}/thermal/top"
-      color="Yellow">
-    </xacro:thermal_camera_macro>
-    <xacro:thermal_camera_macro
-      namespace="${namespace}"
-      camera_frame_name="thermal/middle_optical"
-      camera_topic_name="/${namespace}/thermal/middle"
-      parent_link="base_link"
-      camera_suffix="thermal/middle"
-      frame_rate="14.0"
-      hfov="0.575959"
-      image_width="32"
-      image_height="32"
-      x="0.13"
-      y="0.055"
-      z="-0.085"
-      roll="0"
-      pitch="0"
-      yaw="0"
-      parent_frame_name="${namespace}/fcu"
-      sensor_base_frame_name="${namespace}/thermal/middle"
-      color="Yellow">
-    </xacro:thermal_camera_macro>
-    <xacro:thermal_camera_macro
-      namespace="${namespace}"
-      camera_frame_name="thermal/bottom_optical"
-      camera_topic_name="/${namespace}/thermal/bottom"
-      parent_link="base_link"
-      camera_suffix="thermal/bottom"
-      frame_rate="14.0"
-      hfov="0.575959"
-      image_width="32"
-      image_height="32"
-      x="0.13"
-      y="0.055"
-      z="-0.085"
-      roll="0"
-      pitch="0.523598776"
-      yaw="0"
-      parent_frame_name="${namespace}/fcu"
-      sensor_base_frame_name="${namespace}/thermal/bottom"
-      color="Yellow">
-    </xacro:thermal_camera_macro>
-    <!--}-->
-    <!-- Water gun {-->
-    <xacro:water_gun_macro
-      namespace="${namespace}"
-      name="water_gun_macro"
-      parent="base_link"
-      color="Red"
-      muzzle_velocity="10.0"
-      particle_capacity="30"
-      spread="1.0"
-      spawning_reservoir="the_void"
-      offset_x="0.2"
-      offset_y="0.0"
-      offset_z="-0.1"
-      size_x="0.2"
-      size_y="0.05"
-      size_z="0.05">
-      <origin xyz="0 0 0" rpy="0 -0.1 0" />
-    </xacro:water_gun_macro>
-    <!--}-->
-  </xacro:if>
-  <!--}-->
   <!-- Fire challenge (blanket dropping) {-->
   <xacro:if value="$(arg fire_challenge_blanket)">

Commit message: Added a bluefox fisheye camera. Set up only for f450 down orientation

File: models/mrs_robots_description/urdf/component_snippets.xacro (robot description, xacro)
@@ -811,4 +811,80 @@
             <stddev>${noise_stddev}</stddev>
           </noise>
+        </camera>
+        <plugin name="${namespace}_camera_${camera_suffix}_controller" filename="libMRSGazeboCameraPlugin.so">
+          <alwaysOn>true</alwaysOn>
+          <updateRate>${frame_rate}</updateRate>
+          <cameraName>${camera_suffix}</cameraName>
+          <imageTopicName>image_raw</imageTopicName>
+          <cameraInfoTopicName>camera_info</cameraInfoTopicName>
+          <frameName>/${camera_frame_name}</frameName>
+          <hackBaseline>0.0</hackBaseline>
+          <distortionK1>0.0</distortionK1>
+          <distortionK2>0.0</distortionK2>
+          <distortionK3>0.0</distortionK3>
+          <distortionT1>0.0</distortionT1>
+          <distortionT2>0.0</distortionT2>
+          <parentFrameName>${parent_frame_name}</parentFrameName>
+          <sensorBaseFrameName>${sensor_base_frame_name}</sensorBaseFrameName>
+          <x>${x}</x>
+          <y>${y}</y>
+          <z>${z}</z>
+          <roll>${roll}</roll>
+          <pitch>${pitch}</pitch>
+          <yaw>${yaw}</yaw>
+        </plugin>
+      </sensor>
+    </gazebo>
+    <gazebo reference="${namespace}/camera_${camera_suffix}_link">
+      <material>Gazebo/DarkGrey</material>
+    </gazebo>
+  </xacro:macro>
+  <!--}-->
+  <!-- Macro to add the fisheye_camera_plugin {-->
+  <xacro:macro name="fisheye_macro"
+    params="namespace parent_link camera_suffix camera_frame_name sensor_base_frame_name frame_rate parent_frame_name
+    horizontal_fov image_width image_height min_distance max_distance lens_type lens_c1 lens_c2 lens_f lens_fun lens_scale lens_cutoff_angle lens_texture_size x y z roll pitch yaw
+   noise_mean noise_stddev *visual">
+    <link name="${namespace}/camera_${camera_suffix}_link">
+      <xacro:insert_block name="visual" />
+    </link>
+    <joint name="${namespace}/camera_${camera_suffix}_joint" type="fixed">
+      <origin xyz="${x} ${y} ${z}" rpy="${roll} ${pitch} ${yaw}"/>
+      <parent link="${parent_link}" />
+      <child link="${namespace}/camera_${camera_suffix}_link" />
+    </joint>
+    <gazebo reference="${namespace}/camera_${camera_suffix}_link">
+      <sensor type="wideanglecamera" name="${namespace}_camera_${camera_suffix}">
+        <update_rate>${frame_rate}</update_rate>
+        <camera name="head">
+          <horizontal_fov>${horizontal_fov}</horizontal_fov>
+          <image>
+            <width>${image_width}</width>
+            <height>${image_height}</height>
+          </image>
+          <clip>
+            <near>${min_distance}</near>
+            <far>${max_distance}</far>
+          </clip>
+          <noise>
+            <type>gaussian</type>
+            <!-- Noise is sampled independently per pixel on each frame.
+            That pixel's noise value is added to each of its color
+            channels, which at that point lie in the range [0,1]. -->
+            <mean>${noise_mean}</mean>
+            <stddev>${noise_stddev}</stddev>
+          </noise>
+          <lens>
+            <type>${lens_type}</type>
+            <custom_function>
+              <c1>${lens_c1}</c1>
+              <c2>${lens_c2}</c2>
+              <f>${lens_f}</f>
+              <fun>${lens_fun}</fun>
+            </custom_function>
+            <scale_to_hfov>${lens_scale}</scale_to_hfov>
+            <cutoff_angle>${lens_cutoff_angle}</cutoff_angle>
+            <env_texture_size>${lens_texture_size}</env_texture_size>
+          </lens>
         </camera>
         <plugin name="${namespace}_camera_${camera_suffix}_controller" filename="libMRSGazeboCameraPlugin.so">
@@ -1595,4 +1671,47 @@
   </xacro:macro>
   <!--}-->
+  <!-- Macro to add a Fisheye camera {-->
+  <xacro:macro name="fisheye_camera_macro"
+    params="namespace parent_link camera_suffix frame_rate noise x y z roll pitch yaw camera_frame_name sensor_base_frame_name parent_frame_name">
+    <xacro:fisheye_macro
+      namespace="${namespace}"
+      parent_link="${parent_link}"
+      camera_suffix="${camera_suffix}"
+      camera_frame_name="${camera_frame_name}"
+      sensor_base_frame_name="${sensor_base_frame_name}"
+      frame_rate="${frame_rate}"
+      horizontal_fov="3.14"
+      image_width="752"
+      image_height="480"
+      lens_type="custom"
+      lens_c1="1.05"
+      lens_c2="4"
+      lens_f="1.0"
+      lens_fun="tan"
+      lens_scale="true"
+      lens_cutoff_angle="1.57"
+      lens_texture_size="512"
+      min_distance="0.02"
+      max_distance="100"
+      noise_mean="0.0"
+      noise_stddev="${noise}"
+      parent_frame_name="${parent_frame_name}"
+      x="${x}"
+      y="${y}"
+      z="${z}"
+      yaw="${yaw}"
+      pitch="${pitch}"
+      roll="${roll}"
+      >
+      <visual>
+        <origin xyz="0 0 0" rpy="${rad90} 0 0" />
+        <geometry>
+          <mesh filename="package://mrs_robots_description/meshes/sensors/bluefox.dae"
+            scale="1 1 1" />
+        </geometry>
+      </visual>
+    </xacro:fisheye_macro>
+  </xacro:macro>
+  <!--}-->
   <!-- Macro to add a Mobius camera {-->
   <xacro:macro name="mobius_camera_macro"

File: models/mrs_robots_description/urdf/f450.xacro (robot description, xacro)
@@ -729,4 +729,27 @@
   <!--}-->
   <!-- ========================= camera sensors ========================= -->
+  <!-- Fisheye camera placements{-->
+  <!-- classic {-->
+  <xacro:if value="$(arg enable_fisheye_camera)">
+    <xacro:fisheye_camera_macro
+      namespace="${namespace}"
+      parent_link="base_link"
+      camera_suffix="fisheye_camera"
+      frame_rate="45"
+      noise="0.000"
+      parent_frame_name="${namespace}/fcu"
+      camera_frame_name="${namespace}/fisheye_camera_optical"
+      sensor_base_frame_name="${namespace}/fisheye_camera"
+      x="0.05"
+      y="0"
+      z="-${arm_height + 0.055}"
+      roll="0"
+      pitch="${rad90}"
+      yaw="0.0"
+      >
+  </xacro:fisheye_camera_macro>
+</xacro:if>
+<!--}-->
+  <!--} Fisheye camera placements -->
   <!-- Bluefox placements{-->
   <!-- reverse {-->
