Commit message: Fisheye (#8)
* Added a bluefox fisheye camera. Set up only for f450 down orientation

* Added a bluefox fisheye camera. Set up only for f450 down orientation

* Update f450.xacro

polishing

* Update spawn.py

polishing

* Update component_snippets.xacro

- lowered max_distance to 40 meters 
- added more precise horizontal_fov and lens_cutoff_angle using predefined variables

Co-authored-by: Jan Bednar <bednaj14@fel.cvut.cz>
Co-authored-by: Vojtech Spurny <vojtech.spurny@fel.cvut.cz>

File: models/mrs_robots_description/urdf/component_snippets.xacro (robot description, xacro)
@@ -811,4 +811,80 @@
             <stddev>${noise_stddev}</stddev>
           </noise>
+        </camera>
+        <plugin name="${namespace}_camera_${camera_suffix}_controller" filename="libMRSGazeboCameraPlugin.so">
+          <alwaysOn>true</alwaysOn>
+          <updateRate>${frame_rate}</updateRate>
+          <cameraName>${camera_suffix}</cameraName>
+          <imageTopicName>image_raw</imageTopicName>
+          <cameraInfoTopicName>camera_info</cameraInfoTopicName>
+          <frameName>/${camera_frame_name}</frameName>
+          <hackBaseline>0.0</hackBaseline>
+          <distortionK1>0.0</distortionK1>
+          <distortionK2>0.0</distortionK2>
+          <distortionK3>0.0</distortionK3>
+          <distortionT1>0.0</distortionT1>
+          <distortionT2>0.0</distortionT2>
+          <parentFrameName>${parent_frame_name}</parentFrameName>
+          <sensorBaseFrameName>${sensor_base_frame_name}</sensorBaseFrameName>
+          <x>${x}</x>
+          <y>${y}</y>
+          <z>${z}</z>
+          <roll>${roll}</roll>
+          <pitch>${pitch}</pitch>
+          <yaw>${yaw}</yaw>
+        </plugin>
+      </sensor>
+    </gazebo>
+    <gazebo reference="${namespace}/camera_${camera_suffix}_link">
+      <material>Gazebo/DarkGrey</material>
+    </gazebo>
+  </xacro:macro>
+  <!--}-->
+  <!-- Macro to add the fisheye_camera_plugin {-->
+  <xacro:macro name="fisheye_macro"
+    params="namespace parent_link camera_suffix camera_frame_name sensor_base_frame_name frame_rate parent_frame_name
+    horizontal_fov image_width image_height min_distance max_distance lens_type lens_c1 lens_c2 lens_f lens_fun lens_scale lens_cutoff_angle lens_texture_size x y z roll pitch yaw
+   noise_mean noise_stddev *visual">
+    <link name="${namespace}/camera_${camera_suffix}_link">
+      <xacro:insert_block name="visual" />
+    </link>
+    <joint name="${namespace}/camera_${camera_suffix}_joint" type="fixed">
+      <origin xyz="${x} ${y} ${z}" rpy="${roll} ${pitch} ${yaw}"/>
+      <parent link="${parent_link}" />
+      <child link="${namespace}/camera_${camera_suffix}_link" />
+    </joint>
+    <gazebo reference="${namespace}/camera_${camera_suffix}_link">
+      <sensor type="wideanglecamera" name="${namespace}_camera_${camera_suffix}">
+        <update_rate>${frame_rate}</update_rate>
+        <camera name="head">
+          <horizontal_fov>${horizontal_fov}</horizontal_fov>
+          <image>
+            <width>${image_width}</width>
+            <height>${image_height}</height>
+          </image>
+          <clip>
+            <near>${min_distance}</near>
+            <far>${max_distance}</far>
+          </clip>
+          <noise>
+            <type>gaussian</type>
+            <!-- Noise is sampled independently per pixel on each frame.
+            That pixel's noise value is added to each of its color
+            channels, which at that point lie in the range [0,1]. -->
+            <mean>${noise_mean}</mean>
+            <stddev>${noise_stddev}</stddev>
+          </noise>
+          <lens>
+            <type>${lens_type}</type>
+            <custom_function>
+              <c1>${lens_c1}</c1>
+              <c2>${lens_c2}</c2>
+              <f>${lens_f}</f>
+              <fun>${lens_fun}</fun>
+            </custom_function>
+            <scale_to_hfov>${lens_scale}</scale_to_hfov>
+            <cutoff_angle>${lens_cutoff_angle}</cutoff_angle>
+            <env_texture_size>${lens_texture_size}</env_texture_size>
+          </lens>
         </camera>
         <plugin name="${namespace}_camera_${camera_suffix}_controller" filename="libMRSGazeboCameraPlugin.so">
@@ -1600,4 +1676,47 @@
   </xacro:macro>
   <!--}-->
+  <!-- Macro to add a Fisheye camera {-->
+  <xacro:macro name="fisheye_camera_macro"
+    params="namespace parent_link camera_suffix frame_rate noise x y z roll pitch yaw camera_frame_name sensor_base_frame_name parent_frame_name">
+    <xacro:fisheye_macro
+      namespace="${namespace}"
+      parent_link="${parent_link}"
+      camera_suffix="${camera_suffix}"
+      camera_frame_name="${camera_frame_name}"
+      sensor_base_frame_name="${sensor_base_frame_name}"
+      frame_rate="${frame_rate}"
+      horizontal_fov="${rad180}"
+      image_width="752"
+      image_height="480"
+      lens_type="custom"
+      lens_c1="1.05"
+      lens_c2="4"
+      lens_f="1.0"
+      lens_fun="tan"
+      lens_scale="true"
+      lens_cutoff_angle="${rad90}"
+      lens_texture_size="512"
+      min_distance="0.02"
+      max_distance="40"
+      noise_mean="0.0"
+      noise_stddev="${noise}"
+      parent_frame_name="${parent_frame_name}"
+      x="${x}"
+      y="${y}"
+      z="${z}"
+      yaw="${yaw}"
+      pitch="${pitch}"
+      roll="${roll}"
+      >
+      <visual>
+        <origin xyz="0 0 0" rpy="${rad90} 0 0" />
+        <geometry>
+          <mesh filename="package://mrs_robots_description/meshes/sensors/bluefox.dae"
+            scale="1 1 1" />
+        </geometry>
+      </visual>
+    </xacro:fisheye_macro>
+  </xacro:macro>
+  <!--}-->
   <!-- Macro to add a Mobius camera {-->
   <xacro:macro name="mobius_camera_macro"

File: models/mrs_robots_description/urdf/f450.xacro (robot description, xacro)
@@ -729,4 +729,27 @@
   <!--}-->
   <!-- ========================= camera sensors ========================= -->
+  <!-- Fisheye camera placements{-->
+  <!-- classic {-->
+  <xacro:if value="$(arg enable_fisheye_camera)">
+    <xacro:fisheye_camera_macro
+      namespace="${namespace}"
+      parent_link="base_link"
+      camera_suffix="fisheye_camera"
+      frame_rate="45"
+      noise="0.000"
+      parent_frame_name="${namespace}/fcu"
+      camera_frame_name="${namespace}/fisheye_camera_optical"
+      sensor_base_frame_name="${namespace}/fisheye_camera"
+      x="0.05"
+      y="0"
+      z="-${arm_height + 0.055}"
+      roll="0"
+      pitch="${rad90}"
+      yaw="0.0"
+      >
+    </xacro:fisheye_camera_macro>
+  </xacro:if>
+  <!--}-->
+  <!--} Fisheye camera placements -->
   <!-- Bluefox placements{-->
   <!-- reverse {-->

Commit message: changes for firmware version v1.11.0

File: models/mrs_robots_description/urdf/component_snippets.xacro (robot description, xacro)
@@ -396,11 +396,44 @@
   <!--  {-->
   <!-- Macro to add the gps_plugin {-->
-  <xacro:macro name="gps_plugin_macro" params="namespace gps_noise gps_indoor_jamming">
+  <xacro:macro name="gps_macro"
+    params="gps_name pos_x pos_y pos_z namespace gps_noise gps_xy_random_walk
+            gps_z_random_walk gps_xy_noise_density gps_z_noise_density
+            update_rate gps_vxy_noise_density gps_vz_noise_density parent_link">
     <gazebo>
-      <plugin name="gps_plugin" filename="libMRSGazeboGPSPlugin.so">
-        <robotNamespace>${namespace}</robotNamespace>
-        <gpsNoise>${gps_noise}</gpsNoise>
-        <indoorJamming>${gps_indoor_jamming}</indoorJamming>
-      </plugin>
+      <model name="${gps_name}">
+        <link name="link">
+          <pose>${pos_x} ${pos_y} ${pos_z} 0 0 0</pose>
+          <inertial>
+            <pose>0 0 0 0 0 0</pose>
+            <mass>0.01</mass>
+            <inertia>
+              <ixx>2.1733e-6</ixx>
+              <ixy>0</ixy>
+              <ixz>0</ixz>
+              <iyy>2.1733e-6</iyy>
+              <iyz>0</iyz>
+              <izz>1.8e-7</izz>
+            </inertia>
+          </inertial>
+          <sensor name="gps" type="gps">
+            <pose>0 0 0 0 0 0</pose>
+            <plugin name="gps_plugin" filename="libgazebo_gps_plugin.so">
+              <robotNamespace>${namespace}</robotNamespace>
+              <gpsNoise>${gps_noise}</gpsNoise>
+              <gpsXYRandomWalk>${gps_xy_random_walk}</gpsXYRandomWalk>
+              <gpsZRandomWalk>${gps_z_random_walk}</gpsZRandomWalk>
+              <gpsXYNoiseDensity>${gps_xy_noise_density}</gpsXYNoiseDensity>
+              <gpsZNoiseDensity>${gps_z_noise_density}</gpsZNoiseDensity>
+              <gpsVXYNoiseDensity>${gps_vxy_noise_density}</gpsVXYNoiseDensity>
+              <gpsVZNoiseDensity>${gps_vz_noise_density}</gpsVZNoiseDensity>
+              <update_rate>${update_rate}</update_rate>
+            </plugin>
+          </sensor>
+        </link>
+      </model>
+      <joint name="${gps_name}_joint" type="fixed">
+        <parent>${parent_link}</parent>
+        <child>${gps_name}::link</child>
+      </joint>
     </gazebo>
   </xacro:macro>
@@ -421,5 +454,5 @@
   <!--}-->
   <!-- Macro to add the barometer_plugin{-->
-  <xacro:macro name="barometer_plugin_macro" params="namespace pub_rate baro_topic">
+  <xacro:macro name="barometer_plugin_macro" params="namespace pub_rate baro_topic baro_drift_pa_per_sec">
     <gazebo>
       <plugin name="barometer_plugin" filename="libgazebo_barometer_plugin.so">
@@ -427,4 +460,5 @@
         <pubRate>${pub_rate}</pubRate>
         <baroTopic>${baro_topic}</baroTopic>
+        <baroDriftPaPerSec>${baro_drift_pa_per_sec}</baroDriftPaPerSec>
       </plugin>
     </gazebo>
@@ -432,10 +466,9 @@
   <!--}-->
   <!-- Macro to add the mavlink_interface_plugin{-->
-  <xacro:macro name="mavlink_interface_macro" params="namespace imu_sub_topic gps_sub_topic mag_sub_topic baro_sub_topic mavlink_addr mavlink_udp_port mavlink_tcp_port serial_enabled serial_device baudrate qgc_addr qgc_udp_port sdk_addr sdk_udp_port hil_mode hil_state_level vehicle_is_tailsitter send_vision_estimation send_odometry enable_lockstep use_tcp">
+  <xacro:macro name="mavlink_interface_macro" params="namespace imu_sub_topic mag_sub_topic baro_sub_topic mavlink_addr mavlink_udp_port mavlink_tcp_port serial_enabled serial_device baudrate qgc_addr qgc_udp_port sdk_addr sdk_udp_port hil_mode hil_state_level vehicle_is_tailsitter send_vision_estimation send_odometry enable_lockstep use_tcp">
     <gazebo>
       <plugin name="mavlink_interface" filename="libgazebo_mavlink_interface.so">
         <robotNamespace>${namespace}</robotNamespace>
         <imuSubTopic>${imu_sub_topic}</imuSubTopic>
-        <gpsSubTopic>${gps_sub_topic}</gpsSubTopic>
         <magSubTopic>${mag_sub_topic}</magSubTopic>
         <baroSubTopic>${baro_sub_topic}</baroSubTopic>
@@ -529,11 +562,12 @@
   <!--}-->
   <!-- Macro to add the imu_plugin{-->
+  <!-- Macro to add an IMU. -->
   <xacro:macro name="imu_plugin_macro"
     params="namespace imu_suffix parent_link imu_topic
-    mass_imu_sensor gyroscope_noise_density gyroscopoe_random_walk
-    gyroscope_bias_correlation_time gyroscope_turn_on_bias_sigma
-    accelerometer_noise_density accelerometer_random_walk
-    accelerometer_bias_correlation_time accelerometer_turn_on_bias_sigma
-    *inertia *origin">
+      mass_imu_sensor gyroscope_noise_density gyroscope_random_walk
+      gyroscope_bias_correlation_time gyroscope_turn_on_bias_sigma
+      accelerometer_noise_density accelerometer_random_walk
+      accelerometer_bias_correlation_time accelerometer_turn_on_bias_sigma
+      *inertia *origin">
     <!-- IMU link -->
     <link name="${namespace}/imu${imu_suffix}_link">
@@ -553,11 +587,11 @@
     <gazebo>
       <plugin filename="libgazebo_imu_plugin.so" name="rotors_gazebo_imu${imu_suffix}_plugin">
-        <!-- A good description of the IMU parameters can be found in the kalibr documentation:
-        https://github.com/ethz-asl/kalibr/wiki/IMU-Noise-Model-and-Intrinsics -->
+      <!-- A good description of the IMU parameters can be found in the kalibr documentation:
+           https://github.com/ethz-asl/kalibr/wiki/IMU-Noise-Model-and-Intrinsics -->
         <robotNamespace>${namespace}</robotNamespace> <!-- (string, required): ros namespace in which the messages are published -->
         <linkName>${namespace}/imu${imu_suffix}_link</linkName> <!-- (string, required): name of the body which holds the IMU sensor -->
         <imuTopic>${imu_topic}</imuTopic> <!-- (string): name of the sensor output topic and prefix of service names (defaults to imu) -->
         <gyroscopeNoiseDensity>${gyroscope_noise_density}</gyroscopeNoiseDensity> <!-- Gyroscope noise density (two-sided spectrum) [rad/s/sqrt(Hz)] -->
-        <gyroscopeRandomWalk>${gyroscopoe_random_walk}</gyroscopeRandomWalk> <!-- Gyroscope bias random walk [rad/s/s/sqrt(Hz)] -->
+        <gyroscopeRandomWalk>${gyroscope_random_walk}</gyroscopeRandomWalk> <!-- Gyroscope bias random walk [rad/s/s/sqrt(Hz)] -->
         <gyroscopeBiasCorrelationTime>${gyroscope_bias_correlation_time}</gyroscopeBiasCorrelationTime> <!-- Gyroscope bias correlation time constant [s] -->
         <gyroscopeTurnOnBiasSigma>${gyroscope_turn_on_bias_sigma}</gyroscopeTurnOnBiasSigma> <!-- Gyroscope turn on bias standard deviation [rad/s] -->

File: models/mrs_robots_description/urdf/f450.xacro (robot description, xacro)
@@ -425,5 +425,4 @@
     namespace="${namespace}"
     imu_sub_topic="/imu"
-    gps_sub_topic="/gps"
     mag_sub_topic="/mag"
     baro_sub_topic="/baro"
@@ -448,22 +447,26 @@
   </xacro:mavlink_interface_macro>
   <!--}-->
-    <!-- GPS {-->
-  <xacro:gps_plugin_macro
+  <!-- GPS {-->
+  <xacro:gps_macro
+    gps_name="gps0"
+    pos_x="0.0"
+    pos_y="0.0"
+    pos_z="0.0"
+    gps_noise="true"
+    gps_xy_random_walk="2.0"
+    gps_z_random_walk="4.0"
+    gps_xy_noise_density="2.0e-4"
+    gps_z_noise_density="4.0e-4"
+    gps_vxy_noise_density="0.2"
+    gps_vz_noise_density="0.4"
+    update_rate="10"
     namespace="${namespace}"
-    gps_noise="true"
-    gps_indoor_jamming="$(arg gps_indoor_jamming)">
-    >
-  </xacro:gps_plugin_macro>
-  <xacro:if value="$(arg gps_indoor_jamming)">
-    <xacro:gps_satelites_blocking_macro
-      namespace="${namespace}"
-      parent_link="base_link">
-    </xacro:gps_satelites_blocking_macro>
-  </xacro:if>
+    parent_link="base_link">
+  </xacro:gps_macro>
   <!--}-->
   <!-- Magnetometer {-->
   <xacro:magnetometer_plugin_macro
     namespace="${namespace}"
-    pub_rate="20"
+    pub_rate="100"
     noise_density="0.0004"
     random_walk="0.0000064"
@@ -476,6 +479,7 @@
   <xacro:barometer_plugin_macro
   namespace="${namespace}"
-  pub_rate="10"
+  pub_rate="50"
   baro_topic="/baro"
+  baro_drift_pa_per_sec="0"
   >
   </xacro:barometer_plugin_macro>
@@ -488,9 +492,9 @@
     imu_topic="/imu"
     mass_imu_sensor="0.015"
-    gyroscope_noise_density="0.0003394"
-    gyroscopoe_random_walk="0.000038785"
+    gyroscope_noise_density="0.00018665"
+    gyroscope_random_walk="0.000038785"
     gyroscope_bias_correlation_time="1000.0"
     gyroscope_turn_on_bias_sigma="0.0087"
-    accelerometer_noise_density="0.004"
+    accelerometer_noise_density="0.00186"
     accelerometer_random_walk="0.006"
     accelerometer_bias_correlation_time="300.0"

File: models/mrs_robots_description/urdf/f550.xacro (robot description, xacro)
@@ -484,5 +484,4 @@
     namespace="${namespace}"
     imu_sub_topic="/imu"
-    gps_sub_topic="/gps"
     mag_sub_topic="/mag"
     baro_sub_topic="/baro"
@@ -508,21 +507,25 @@
   <!--}-->
   <!-- GPS {-->
-  <xacro:gps_plugin_macro
-    namespace="${namespace}"
+  <xacro:gps_macro
+    gps_name="gps0"
+    pos_x="0.0"
+    pos_y="0.0"
+    pos_z="0.0"
     gps_noise="true"
-    gps_indoor_jamming="$(arg gps_indoor_jamming)">
-    >
-  </xacro:gps_plugin_macro>
-  <xacro:if value="$(arg gps_indoor_jamming)">
-    <xacro:gps_satelites_blocking_macro
-      namespace="${namespace}"
-      parent_link="base_link">
-    </xacro:gps_satelites_blocking_macro>
-  </xacro:if>
+    gps_xy_random_walk="2.0"
+    gps_z_random_walk="4.0"
+    gps_xy_noise_density="2.0e-4"
+    gps_z_noise_density="4.0e-4"
+    gps_vxy_noise_density="0.2"
+    gps_vz_noise_density="0.4"
+    update_rate="10"
+    namespace="uav1"
+    parent_link="base_link">
+  </xacro:gps_macro>
   <!--}-->
   <!-- Magnetometer {-->
   <xacro:magnetometer_plugin_macro
     namespace="${namespace}"
-    pub_rate="20"
+    pub_rate="100"
     noise_density="0.0004"
     random_walk="0.0000064"
@@ -535,6 +538,7 @@
   <xacro:barometer_plugin_macro
     namespace="${namespace}"
-    pub_rate="10"
+    pub_rate="50"
     baro_topic="/baro"
+    baro_drift_pa_per_sec="0"
     >
   </xacro:barometer_plugin_macro>
@@ -547,9 +551,9 @@
     imu_topic="/imu"
     mass_imu_sensor="0.015"
-    gyroscope_noise_density="0.0003394"
-    gyroscopoe_random_walk="0.000038785"
+    gyroscope_noise_density="0.00018665"
+    gyroscope_random_walk="0.000038785"
     gyroscope_bias_correlation_time="1000.0"
     gyroscope_turn_on_bias_sigma="0.0087"
-    accelerometer_noise_density="0.004"
+    accelerometer_noise_density="0.00186"
     accelerometer_random_walk="0.006"
     accelerometer_bias_correlation_time="300.0"

File: models/mrs_robots_description/urdf/t650.xacro (robot description, xacro)
@@ -400,5 +400,4 @@
     namespace="${namespace}"
     imu_sub_topic="/imu"
-    gps_sub_topic="/gps"
     mag_sub_topic="/mag"
     baro_sub_topic="/baro"
@@ -424,21 +423,25 @@
   <!--}-->
   <!-- GPS {-->
-  <xacro:gps_plugin_macro
-    namespace="${namespace}"
+  <xacro:gps_macro
+    gps_name="gps0"
+    pos_x="0.0"
+    pos_y="0.0"
+    pos_z="0.0"
     gps_noise="true"
-    gps_indoor_jamming="$(arg gps_indoor_jamming)">
-    >
-  </xacro:gps_plugin_macro>
-  <xacro:if value="$(arg gps_indoor_jamming)">
-    <xacro:gps_satelites_blocking_macro
-      namespace="${namespace}"
-      parent_link="base_link">
-    </xacro:gps_satelites_blocking_macro>
-  </xacro:if>
+    gps_xy_random_walk="2.0"
+    gps_z_random_walk="4.0"
+    gps_xy_noise_density="2.0e-4"
+    gps_z_noise_density="4.0e-4"
+    gps_vxy_noise_density="0.2"
+    gps_vz_noise_density="0.4"
+    update_rate="10"
+    namespace="uav1"
+    parent_link="base_link">
+  </xacro:gps_macro>
   <!--}-->
   <!-- Magnetometer {-->
   <xacro:magnetometer_plugin_macro
     namespace="${namespace}"
-    pub_rate="20"
+    pub_rate="100"
     noise_density="0.0004"
     random_walk="0.0000064"
@@ -451,6 +454,7 @@
   <xacro:barometer_plugin_macro
     namespace="${namespace}"
-    pub_rate="10"
+    pub_rate="50"
     baro_topic="/baro"
+    baro_drift_pa_per_sec="0"
     >
   </xacro:barometer_plugin_macro>
@@ -463,9 +467,9 @@
     imu_topic="/imu"
     mass_imu_sensor="0.015"
-    gyroscope_noise_density="0.0003394"
-    gyroscopoe_random_walk="0.000038785"
+    gyroscope_noise_density="0.00018665"
+    gyroscope_random_walk="0.000038785"
     gyroscope_bias_correlation_time="1000.0"
     gyroscope_turn_on_bias_sigma="0.0087"
-    accelerometer_noise_density="0.004"
+    accelerometer_noise_density="0.00186"
     accelerometer_random_walk="0.006"
     accelerometer_bias_correlation_time="300.0"

Commit message: updated model for gps

File: models/mrs_robots_description/urdf/component_snippets.xacro (robot description, xacro)
@@ -401,38 +401,37 @@
             update_rate gps_vxy_noise_density gps_vz_noise_density parent_link">
     <gazebo>
-      <model name="${gps_name}">
-        <link name="link">
-          <pose>${pos_x} ${pos_y} ${pos_z} 0 0 0</pose>
-          <inertial>
-            <pose>0 0 0 0 0 0</pose>
-            <mass>0.01</mass>
-            <inertia>
-              <ixx>2.1733e-6</ixx>
-              <ixy>0</ixy>
-              <ixz>0</ixz>
-              <iyy>2.1733e-6</iyy>
-              <iyz>0</iyz>
-              <izz>1.8e-7</izz>
-            </inertia>
-          </inertial>
-          <sensor name="gps" type="gps">
-            <pose>0 0 0 0 0 0</pose>
-            <plugin name="gps_plugin" filename="libgazebo_gps_plugin.so">
-              <robotNamespace>${namespace}</robotNamespace>
-              <gpsNoise>${gps_noise}</gpsNoise>
-              <gpsXYRandomWalk>${gps_xy_random_walk}</gpsXYRandomWalk>
-              <gpsZRandomWalk>${gps_z_random_walk}</gpsZRandomWalk>
-              <gpsXYNoiseDensity>${gps_xy_noise_density}</gpsXYNoiseDensity>
-              <gpsZNoiseDensity>${gps_z_noise_density}</gpsZNoiseDensity>
-              <gpsVXYNoiseDensity>${gps_vxy_noise_density}</gpsVXYNoiseDensity>
-              <gpsVZNoiseDensity>${gps_vz_noise_density}</gpsVZNoiseDensity>
-              <update_rate>${update_rate}</update_rate>
-            </plugin>
-          </sensor>
-        </link>
-      </model>
+      <link name="${gps_name}_link">
+        <pose>${pos_x} ${pos_y} ${pos_z} 0 0 0</pose>
+        <inertial>
+          <pose>0 0 0 0 0 0</pose>
+          <mass>0.01</mass>
+          <inertia>
+            <ixx>2.1733e-6</ixx>
+            <ixy>0</ixy>
+            <ixz>0</ixz>
+            <iyy>2.1733e-6</iyy>
+            <iyz>0</iyz>
+            <izz>1.8e-7</izz>
+          </inertia>
+        </inertial>
+        <sensor name="gps" type="gps">
+          <pose>0 0 0 0 0 0</pose>
+          <plugin name="gps_plugin" filename="libgazebo_gps_plugin.so">
+            <robotNamespace>${namespace}</robotNamespace>
+            <gpsNoise>${gps_noise}</gpsNoise>
+            <gpsXYRandomWalk>${gps_xy_random_walk}</gpsXYRandomWalk>
+            <gpsZRandomWalk>${gps_z_random_walk}</gpsZRandomWalk>
+            <gpsXYNoiseDensity>${gps_xy_noise_density}</gpsXYNoiseDensity>
+            <gpsZNoiseDensity>${gps_z_noise_density}</gpsZNoiseDensity>
+            <gpsVXYNoiseDensity>${gps_vxy_noise_density}</gpsVXYNoiseDensity>
+            <gpsVZNoiseDensity>${gps_vz_noise_density}</gpsVZNoiseDensity>
+            <update_rate>${update_rate}</update_rate>
+            <topic>${gps_name}</topic>
+          </plugin>
+        </sensor>
+      </link>
       <joint name="${gps_name}_joint" type="fixed">
         <parent>${parent_link}</parent>
-        <child>${gps_name}::link</child>
+        <child>${gps_name}_link</child>
       </joint>
     </gazebo>
