Commit message: revert back to old version of firmware (v1.10.1)

File: models/mrs_robots_description/urdf/component_snippets.xacro (robot description, xacro)
@@ -396,43 +396,11 @@
   <!--  {-->
   <!-- Macro to add the gps_plugin {-->
-  <xacro:macro name="gps_macro"
-    params="gps_name pos_x pos_y pos_z namespace gps_noise gps_xy_random_walk
-            gps_z_random_walk gps_xy_noise_density gps_z_noise_density
-            update_rate gps_vxy_noise_density gps_vz_noise_density parent_link">
+  <xacro:macro name="gps_plugin_macro" params="namespace gps_noise gps_indoor_jamming">
     <gazebo>
-      <link name="${gps_name}_link">
-        <pose>${pos_x} ${pos_y} ${pos_z} 0 0 0</pose>
-        <inertial>
-          <pose>0 0 0 0 0 0</pose>
-          <mass>0.01</mass>
-          <inertia>
-            <ixx>2.1733e-6</ixx>
-            <ixy>0</ixy>
-            <ixz>0</ixz>
-            <iyy>2.1733e-6</iyy>
-            <iyz>0</iyz>
-            <izz>1.8e-7</izz>
-          </inertia>
-        </inertial>
-        <sensor name="gps" type="gps">
-          <pose>0 0 0 0 0 0</pose>
-          <plugin name="gps_plugin" filename="libgazebo_gps_plugin.so">
-            <robotNamespace>${namespace}</robotNamespace>
-            <gpsNoise>${gps_noise}</gpsNoise>
-            <gpsXYRandomWalk>${gps_xy_random_walk}</gpsXYRandomWalk>
-            <gpsZRandomWalk>${gps_z_random_walk}</gpsZRandomWalk>
-            <gpsXYNoiseDensity>${gps_xy_noise_density}</gpsXYNoiseDensity>
-            <gpsZNoiseDensity>${gps_z_noise_density}</gpsZNoiseDensity>
-            <gpsVXYNoiseDensity>${gps_vxy_noise_density}</gpsVXYNoiseDensity>
-            <gpsVZNoiseDensity>${gps_vz_noise_density}</gpsVZNoiseDensity>
-            <update_rate>${update_rate}</update_rate>
-            <topic>${gps_name}</topic>
-          </plugin>
-        </sensor>
-      </link>
-      <joint name="${gps_name}_joint" type="fixed">
-        <parent>${parent_link}</parent>
-        <child>${gps_name}_link</child>
-      </joint>
+      <plugin name="gps_plugin" filename="libMRSGazeboGPSPlugin.so">
+        <robotNamespace>${namespace}</robotNamespace>
+        <gpsNoise>${gps_noise}</gpsNoise>
+        <indoorJamming>${gps_indoor_jamming}</indoorJamming>
+      </plugin>
     </gazebo>
   </xacro:macro>
@@ -453,5 +421,5 @@
   <!--}-->
   <!-- Macro to add the barometer_plugin{-->
-  <xacro:macro name="barometer_plugin_macro" params="namespace pub_rate baro_topic baro_drift_pa_per_sec">
+  <xacro:macro name="barometer_plugin_macro" params="namespace pub_rate baro_topic">
     <gazebo>
       <plugin name="barometer_plugin" filename="libgazebo_barometer_plugin.so">
@@ -459,5 +427,4 @@
         <pubRate>${pub_rate}</pubRate>
         <baroTopic>${baro_topic}</baroTopic>
-        <baroDriftPaPerSec>${baro_drift_pa_per_sec}</baroDriftPaPerSec>
       </plugin>
     </gazebo>
@@ -465,9 +432,10 @@
   <!--}-->
   <!-- Macro to add the mavlink_interface_plugin{-->
-  <xacro:macro name="mavlink_interface_macro" params="namespace imu_sub_topic mag_sub_topic baro_sub_topic mavlink_addr mavlink_udp_port mavlink_tcp_port serial_enabled serial_device baudrate qgc_addr qgc_udp_port sdk_addr sdk_udp_port hil_mode hil_state_level vehicle_is_tailsitter send_vision_estimation send_odometry enable_lockstep use_tcp">
+  <xacro:macro name="mavlink_interface_macro" params="namespace imu_sub_topic gps_sub_topic mag_sub_topic baro_sub_topic mavlink_addr mavlink_udp_port mavlink_tcp_port serial_enabled serial_device baudrate qgc_addr qgc_udp_port sdk_addr sdk_udp_port hil_mode hil_state_level vehicle_is_tailsitter send_vision_estimation send_odometry enable_lockstep use_tcp">
     <gazebo>
       <plugin name="mavlink_interface" filename="libgazebo_mavlink_interface.so">
         <robotNamespace>${namespace}</robotNamespace>
         <imuSubTopic>${imu_sub_topic}</imuSubTopic>
+        <gpsSubTopic>${gps_sub_topic}</gpsSubTopic>
         <magSubTopic>${mag_sub_topic}</magSubTopic>
         <baroSubTopic>${baro_sub_topic}</baroSubTopic>
@@ -561,12 +529,11 @@
   <!--}-->
   <!-- Macro to add the imu_plugin{-->
-  <!-- Macro to add an IMU. -->
   <xacro:macro name="imu_plugin_macro"
     params="namespace imu_suffix parent_link imu_topic
-      mass_imu_sensor gyroscope_noise_density gyroscope_random_walk
-      gyroscope_bias_correlation_time gyroscope_turn_on_bias_sigma
-      accelerometer_noise_density accelerometer_random_walk
-      accelerometer_bias_correlation_time accelerometer_turn_on_bias_sigma
-      *inertia *origin">
+    mass_imu_sensor gyroscope_noise_density gyroscopoe_random_walk
+    gyroscope_bias_correlation_time gyroscope_turn_on_bias_sigma
+    accelerometer_noise_density accelerometer_random_walk
+    accelerometer_bias_correlation_time accelerometer_turn_on_bias_sigma
+    *inertia *origin">
     <!-- IMU link -->
     <link name="${namespace}/imu${imu_suffix}_link">
@@ -586,11 +553,11 @@
     <gazebo>
       <plugin filename="libgazebo_imu_plugin.so" name="rotors_gazebo_imu${imu_suffix}_plugin">
-      <!-- A good description of the IMU parameters can be found in the kalibr documentation:
-           https://github.com/ethz-asl/kalibr/wiki/IMU-Noise-Model-and-Intrinsics -->
+        <!-- A good description of the IMU parameters can be found in the kalibr documentation:
+        https://github.com/ethz-asl/kalibr/wiki/IMU-Noise-Model-and-Intrinsics -->
         <robotNamespace>${namespace}</robotNamespace> <!-- (string, required): ros namespace in which the messages are published -->
         <linkName>${namespace}/imu${imu_suffix}_link</linkName> <!-- (string, required): name of the body which holds the IMU sensor -->
         <imuTopic>${imu_topic}</imuTopic> <!-- (string): name of the sensor output topic and prefix of service names (defaults to imu) -->
         <gyroscopeNoiseDensity>${gyroscope_noise_density}</gyroscopeNoiseDensity> <!-- Gyroscope noise density (two-sided spectrum) [rad/s/sqrt(Hz)] -->
-        <gyroscopeRandomWalk>${gyroscope_random_walk}</gyroscopeRandomWalk> <!-- Gyroscope bias random walk [rad/s/s/sqrt(Hz)] -->
+        <gyroscopeRandomWalk>${gyroscopoe_random_walk}</gyroscopeRandomWalk> <!-- Gyroscope bias random walk [rad/s/s/sqrt(Hz)] -->
         <gyroscopeBiasCorrelationTime>${gyroscope_bias_correlation_time}</gyroscopeBiasCorrelationTime> <!-- Gyroscope bias correlation time constant [s] -->
         <gyroscopeTurnOnBiasSigma>${gyroscope_turn_on_bias_sigma}</gyroscopeTurnOnBiasSigma> <!-- Gyroscope turn on bias standard deviation [rad/s] -->

File: models/mrs_robots_description/urdf/f450.xacro (robot description, xacro)
@@ -425,4 +425,5 @@
     namespace="${namespace}"
     imu_sub_topic="/imu"
+    gps_sub_topic="/gps"
     mag_sub_topic="/mag"
     baro_sub_topic="/baro"
@@ -447,26 +448,22 @@
   </xacro:mavlink_interface_macro>
   <!--}-->
-  <!-- GPS {-->
-  <xacro:gps_macro
-    gps_name="gps0"
-    pos_x="0.0"
-    pos_y="0.0"
-    pos_z="0.0"
+    <!-- GPS {-->
+  <xacro:gps_plugin_macro
+    namespace="${namespace}"
     gps_noise="true"
-    gps_xy_random_walk="2.0"
-    gps_z_random_walk="4.0"
-    gps_xy_noise_density="2.0e-4"
-    gps_z_noise_density="4.0e-4"
-    gps_vxy_noise_density="0.2"
-    gps_vz_noise_density="0.4"
-    update_rate="10"
-    namespace="${namespace}"
-    parent_link="base_link">
-  </xacro:gps_macro>
+    gps_indoor_jamming="$(arg gps_indoor_jamming)">
+    >
+  </xacro:gps_plugin_macro>
+  <xacro:if value="$(arg gps_indoor_jamming)">
+    <xacro:gps_satelites_blocking_macro
+      namespace="${namespace}"
+      parent_link="base_link">
+    </xacro:gps_satelites_blocking_macro>
+  </xacro:if>
   <!--}-->
   <!-- Magnetometer {-->
   <xacro:magnetometer_plugin_macro
     namespace="${namespace}"
-    pub_rate="100"
+    pub_rate="20"
     noise_density="0.0004"
     random_walk="0.0000064"
@@ -479,7 +476,6 @@
   <xacro:barometer_plugin_macro
   namespace="${namespace}"
-  pub_rate="50"
+  pub_rate="10"
   baro_topic="/baro"
-  baro_drift_pa_per_sec="0"
   >
   </xacro:barometer_plugin_macro>
@@ -492,9 +488,9 @@
     imu_topic="/imu"
     mass_imu_sensor="0.015"
-    gyroscope_noise_density="0.00018665"
-    gyroscope_random_walk="0.000038785"
+    gyroscope_noise_density="0.0003394"
+    gyroscopoe_random_walk="0.000038785"
     gyroscope_bias_correlation_time="1000.0"
     gyroscope_turn_on_bias_sigma="0.0087"
-    accelerometer_noise_density="0.00186"
+    accelerometer_noise_density="0.004"
     accelerometer_random_walk="0.006"
     accelerometer_bias_correlation_time="300.0"

File: models/mrs_robots_description/urdf/f550.xacro (robot description, xacro)
@@ -484,4 +484,5 @@
     namespace="${namespace}"
     imu_sub_topic="/imu"
+    gps_sub_topic="/gps"
     mag_sub_topic="/mag"
     baro_sub_topic="/baro"
@@ -507,25 +508,21 @@
   <!--}-->
   <!-- GPS {-->
-  <xacro:gps_macro
-    gps_name="gps0"
-    pos_x="0.0"
-    pos_y="0.0"
-    pos_z="0.0"
+  <xacro:gps_plugin_macro
+    namespace="${namespace}"
     gps_noise="true"
-    gps_xy_random_walk="2.0"
-    gps_z_random_walk="4.0"
-    gps_xy_noise_density="2.0e-4"
-    gps_z_noise_density="4.0e-4"
-    gps_vxy_noise_density="0.2"
-    gps_vz_noise_density="0.4"
-    update_rate="10"
-    namespace="${namespace}"
-    parent_link="base_link">
-  </xacro:gps_macro>
+    gps_indoor_jamming="$(arg gps_indoor_jamming)">
+    >
+  </xacro:gps_plugin_macro>
+  <xacro:if value="$(arg gps_indoor_jamming)">
+    <xacro:gps_satelites_blocking_macro
+      namespace="${namespace}"
+      parent_link="base_link">
+    </xacro:gps_satelites_blocking_macro>
+  </xacro:if>
   <!--}-->
   <!-- Magnetometer {-->
   <xacro:magnetometer_plugin_macro
     namespace="${namespace}"
-    pub_rate="100"
+    pub_rate="20"
     noise_density="0.0004"
     random_walk="0.0000064"
@@ -538,7 +535,6 @@
   <xacro:barometer_plugin_macro
     namespace="${namespace}"
-    pub_rate="50"
+    pub_rate="10"
     baro_topic="/baro"
-    baro_drift_pa_per_sec="0"
     >
   </xacro:barometer_plugin_macro>
@@ -551,9 +547,9 @@
     imu_topic="/imu"
     mass_imu_sensor="0.015"
-    gyroscope_noise_density="0.00018665"
-    gyroscope_random_walk="0.000038785"
+    gyroscope_noise_density="0.0003394"
+    gyroscopoe_random_walk="0.000038785"
     gyroscope_bias_correlation_time="1000.0"
     gyroscope_turn_on_bias_sigma="0.0087"
-    accelerometer_noise_density="0.00186"
+    accelerometer_noise_density="0.004"
     accelerometer_random_walk="0.006"
     accelerometer_bias_correlation_time="300.0"
@@ -1022,5 +1018,6 @@
       frame_rate="80"
       camera_publish_topic="/${namespace}/uvdar_bluefox_left/image_raw"
-      calibration_file="$(arg uvcam_calib_file)">
+      calibration_file="$(arg uvcam_calib_file)"
+      occlusions="$(arg uvcam_occlusions)">
     <origin xyz="0.037 0.1175 0.05" rpy="0 0 ${rad70}" />
     </xacro:uvcam_macro>
@@ -1031,5 +1028,6 @@
       frame_rate="80"
       camera_publish_topic="/${namespace}/uvdar_bluefox_right/image_raw"
-      calibration_file="$(arg uvcam_calib_file)">
+      calibration_file="$(arg uvcam_calib_file)"
+      occlusions="$(arg uvcam_occlusions)">
     <origin xyz="0.037 -0.1175 0.05" rpy="0 0 -${rad70}" />
     </xacro:uvcam_macro>

File: models/mrs_robots_description/urdf/t650.xacro (robot description, xacro)
@@ -400,4 +400,5 @@
     namespace="${namespace}"
     imu_sub_topic="/imu"
+    gps_sub_topic="/gps"
     mag_sub_topic="/mag"
     baro_sub_topic="/baro"
@@ -423,25 +424,21 @@
   <!--}-->
   <!-- GPS {-->
-  <xacro:gps_macro
-    gps_name="gps0"
-    pos_x="0.0"
-    pos_y="0.0"
-    pos_z="0.0"
+  <xacro:gps_plugin_macro
+    namespace="${namespace}"
     gps_noise="true"
-    gps_xy_random_walk="2.0"
-    gps_z_random_walk="4.0"
-    gps_xy_noise_density="2.0e-4"
-    gps_z_noise_density="4.0e-4"
-    gps_vxy_noise_density="0.2"
-    gps_vz_noise_density="0.4"
-    update_rate="10"
-    namespace="${namespace}"
-    parent_link="base_link">
-  </xacro:gps_macro>
+    gps_indoor_jamming="$(arg gps_indoor_jamming)">
+    >
+  </xacro:gps_plugin_macro>
+  <xacro:if value="$(arg gps_indoor_jamming)">
+    <xacro:gps_satelites_blocking_macro
+      namespace="${namespace}"
+      parent_link="base_link">
+    </xacro:gps_satelites_blocking_macro>
+  </xacro:if>
   <!--}-->
   <!-- Magnetometer {-->
   <xacro:magnetometer_plugin_macro
     namespace="${namespace}"
-    pub_rate="100"
+    pub_rate="20"
     noise_density="0.0004"
     random_walk="0.0000064"
@@ -454,7 +451,6 @@
   <xacro:barometer_plugin_macro
     namespace="${namespace}"
-    pub_rate="50"
+    pub_rate="10"
     baro_topic="/baro"
-    baro_drift_pa_per_sec="0"
     >
   </xacro:barometer_plugin_macro>
@@ -467,9 +463,9 @@
     imu_topic="/imu"
     mass_imu_sensor="0.015"
-    gyroscope_noise_density="0.00018665"
-    gyroscope_random_walk="0.000038785"
+    gyroscope_noise_density="0.0003394"
+    gyroscopoe_random_walk="0.000038785"
     gyroscope_bias_correlation_time="1000.0"
     gyroscope_turn_on_bias_sigma="0.0087"
-    accelerometer_noise_density="0.00186"
+    accelerometer_noise_density="0.004"
     accelerometer_random_walk="0.006"
     accelerometer_bias_correlation_time="300.0"
@@ -880,5 +876,6 @@
       frame_rate="80"
       camera_publish_topic="/${namespace}/uvdar_bluefox_left/image_raw"
-      calibration_file="$(arg uvcam_calib_file)">
+      calibration_file="$(arg uvcam_calib_file)"
+      occlusions="$(arg uvcam_occlusions)">
     <origin xyz="0.037 0.1175 0.057" rpy="0 0 ${rad70}" />
     </xacro:uvcam_macro>
@@ -889,5 +886,6 @@
       frame_rate="80"
       camera_publish_topic="/${namespace}/uvdar_bluefox_right/image_raw"
-      calibration_file="$(arg uvcam_calib_file)">
+      calibration_file="$(arg uvcam_calib_file)"
+      occlusions="$(arg uvcam_occlusions)">
     <origin xyz="0.037 -0.1175 0.057" rpy="0 0 -${rad70}" />
     </xacro:uvcam_macro>
