Commit message: revert unwanted changes of 3ed3e6e2e3f7cb8dd891e3bf70f89c0a23b26ae7

File: models/mrs_robots_description/urdf/component_snippets.xacro (robot description, xacro)
@@ -396,11 +396,43 @@
   <!--  {-->
   <!-- Macro to add the gps_plugin {-->
-  <xacro:macro name="gps_plugin_macro" params="namespace gps_noise gps_indoor_jamming">
+  <xacro:macro name="gps_macro"
+    params="gps_name pos_x pos_y pos_z namespace gps_noise gps_xy_random_walk
+            gps_z_random_walk gps_xy_noise_density gps_z_noise_density
+            update_rate gps_vxy_noise_density gps_vz_noise_density parent_link">
     <gazebo>
-      <plugin name="gps_plugin" filename="libMRSGazeboGPSPlugin.so">
-        <robotNamespace>${namespace}</robotNamespace>
-        <gpsNoise>${gps_noise}</gpsNoise>
-        <indoorJamming>${gps_indoor_jamming}</indoorJamming>
-      </plugin>
+      <link name="${gps_name}_link">
+        <pose>${pos_x} ${pos_y} ${pos_z} 0 0 0</pose>
+        <inertial>
+          <pose>0 0 0 0 0 0</pose>
+          <mass>0.01</mass>
+          <inertia>
+            <ixx>2.1733e-6</ixx>
+            <ixy>0</ixy>
+            <ixz>0</ixz>
+            <iyy>2.1733e-6</iyy>
+            <iyz>0</iyz>
+            <izz>1.8e-7</izz>
+          </inertia>
+        </inertial>
+        <sensor name="gps" type="gps">
+          <pose>0 0 0 0 0 0</pose>
+          <plugin name="gps_plugin" filename="libgazebo_gps_plugin.so">
+            <robotNamespace>${namespace}</robotNamespace>
+            <gpsNoise>${gps_noise}</gpsNoise>
+            <gpsXYRandomWalk>${gps_xy_random_walk}</gpsXYRandomWalk>
+            <gpsZRandomWalk>${gps_z_random_walk}</gpsZRandomWalk>
+            <gpsXYNoiseDensity>${gps_xy_noise_density}</gpsXYNoiseDensity>
+            <gpsZNoiseDensity>${gps_z_noise_density}</gpsZNoiseDensity>
+            <gpsVXYNoiseDensity>${gps_vxy_noise_density}</gpsVXYNoiseDensity>
+            <gpsVZNoiseDensity>${gps_vz_noise_density}</gpsVZNoiseDensity>
+            <update_rate>${update_rate}</update_rate>
+            <topic>${gps_name}</topic>
+          </plugin>
+        </sensor>
+      </link>
+      <joint name="${gps_name}_joint" type="fixed">
+        <parent>${parent_link}</parent>
+        <child>${gps_name}_link</child>
+      </joint>
     </gazebo>
   </xacro:macro>
@@ -421,5 +453,5 @@
   <!--}-->
   <!-- Macro to add the barometer_plugin{-->
-  <xacro:macro name="barometer_plugin_macro" params="namespace pub_rate baro_topic">
+  <xacro:macro name="barometer_plugin_macro" params="namespace pub_rate baro_topic baro_drift_pa_per_sec">
     <gazebo>
       <plugin name="barometer_plugin" filename="libgazebo_barometer_plugin.so">
@@ -427,4 +459,5 @@
         <pubRate>${pub_rate}</pubRate>
         <baroTopic>${baro_topic}</baroTopic>
+        <baroDriftPaPerSec>${baro_drift_pa_per_sec}</baroDriftPaPerSec>
       </plugin>
     </gazebo>
@@ -432,10 +465,9 @@
   <!--}-->
   <!-- Macro to add the mavlink_interface_plugin{-->
-  <xacro:macro name="mavlink_interface_macro" params="namespace imu_sub_topic gps_sub_topic mag_sub_topic baro_sub_topic mavlink_addr mavlink_udp_port mavlink_tcp_port serial_enabled serial_device baudrate qgc_addr qgc_udp_port sdk_addr sdk_udp_port hil_mode hil_state_level vehicle_is_tailsitter send_vision_estimation send_odometry enable_lockstep use_tcp">
+  <xacro:macro name="mavlink_interface_macro" params="namespace imu_sub_topic mag_sub_topic baro_sub_topic mavlink_addr mavlink_udp_port mavlink_tcp_port serial_enabled serial_device baudrate qgc_addr qgc_udp_port sdk_addr sdk_udp_port hil_mode hil_state_level vehicle_is_tailsitter send_vision_estimation send_odometry enable_lockstep use_tcp">
     <gazebo>
       <plugin name="mavlink_interface" filename="libgazebo_mavlink_interface.so">
         <robotNamespace>${namespace}</robotNamespace>
         <imuSubTopic>${imu_sub_topic}</imuSubTopic>
-        <gpsSubTopic>${gps_sub_topic}</gpsSubTopic>
         <magSubTopic>${mag_sub_topic}</magSubTopic>
         <baroSubTopic>${baro_sub_topic}</baroSubTopic>
@@ -529,11 +561,12 @@
   <!--}-->
   <!-- Macro to add the imu_plugin{-->
+  <!-- Macro to add an IMU. -->
   <xacro:macro name="imu_plugin_macro"
     params="namespace imu_suffix parent_link imu_topic
-    mass_imu_sensor gyroscope_noise_density gyroscopoe_random_walk
-    gyroscope_bias_correlation_time gyroscope_turn_on_bias_sigma
-    accelerometer_noise_density accelerometer_random_walk
-    accelerometer_bias_correlation_time accelerometer_turn_on_bias_sigma
-    *inertia *origin">
+      mass_imu_sensor gyroscope_noise_density gyroscope_random_walk
+      gyroscope_bias_correlation_time gyroscope_turn_on_bias_sigma
+      accelerometer_noise_density accelerometer_random_walk
+      accelerometer_bias_correlation_time accelerometer_turn_on_bias_sigma
+      *inertia *origin">
     <!-- IMU link -->
     <link name="${namespace}/imu${imu_suffix}_link">
@@ -553,11 +586,11 @@
     <gazebo>
       <plugin filename="libgazebo_imu_plugin.so" name="rotors_gazebo_imu${imu_suffix}_plugin">
-        <!-- A good description of the IMU parameters can be found in the kalibr documentation:
-        https://github.com/ethz-asl/kalibr/wiki/IMU-Noise-Model-and-Intrinsics -->
+      <!-- A good description of the IMU parameters can be found in the kalibr documentation:
+           https://github.com/ethz-asl/kalibr/wiki/IMU-Noise-Model-and-Intrinsics -->
         <robotNamespace>${namespace}</robotNamespace> <!-- (string, required): ros namespace in which the messages are published -->
         <linkName>${namespace}/imu${imu_suffix}_link</linkName> <!-- (string, required): name of the body which holds the IMU sensor -->
         <imuTopic>${imu_topic}</imuTopic> <!-- (string): name of the sensor output topic and prefix of service names (defaults to imu) -->
         <gyroscopeNoiseDensity>${gyroscope_noise_density}</gyroscopeNoiseDensity> <!-- Gyroscope noise density (two-sided spectrum) [rad/s/sqrt(Hz)] -->
-        <gyroscopeRandomWalk>${gyroscopoe_random_walk}</gyroscopeRandomWalk> <!-- Gyroscope bias random walk [rad/s/s/sqrt(Hz)] -->
+        <gyroscopeRandomWalk>${gyroscope_random_walk}</gyroscopeRandomWalk> <!-- Gyroscope bias random walk [rad/s/s/sqrt(Hz)] -->
         <gyroscopeBiasCorrelationTime>${gyroscope_bias_correlation_time}</gyroscopeBiasCorrelationTime> <!-- Gyroscope bias correlation time constant [s] -->
         <gyroscopeTurnOnBiasSigma>${gyroscope_turn_on_bias_sigma}</gyroscopeTurnOnBiasSigma> <!-- Gyroscope turn on bias standard deviation [rad/s] -->

File: models/mrs_robots_description/urdf/f450.xacro (robot description, xacro)
@@ -427,5 +427,4 @@
     namespace="${namespace}"
     imu_sub_topic="/imu"
-    gps_sub_topic="/gps"
     mag_sub_topic="/mag"
     baro_sub_topic="/baro"
@@ -450,22 +449,26 @@
   </xacro:mavlink_interface_macro>
   <!--}-->
-    <!-- GPS {-->
-  <xacro:gps_plugin_macro
+  <!-- GPS {-->
+  <xacro:gps_macro
+    gps_name="gps0"
+    pos_x="0.0"
+    pos_y="0.0"
+    pos_z="0.0"
+    gps_noise="true"
+    gps_xy_random_walk="2.0"
+    gps_z_random_walk="4.0"
+    gps_xy_noise_density="2.0e-4"
+    gps_z_noise_density="4.0e-4"
+    gps_vxy_noise_density="0.2"
+    gps_vz_noise_density="0.4"
+    update_rate="10"
     namespace="${namespace}"
-    gps_noise="true"
-    gps_indoor_jamming="$(arg gps_indoor_jamming)">
-    >
-  </xacro:gps_plugin_macro>
-  <xacro:if value="$(arg gps_indoor_jamming)">
-    <xacro:gps_satelites_blocking_macro
-      namespace="${namespace}"
-      parent_link="base_link">
-    </xacro:gps_satelites_blocking_macro>
-  </xacro:if>
+    parent_link="base_link">
+  </xacro:gps_macro>
   <!--}-->
   <!-- Magnetometer {-->
   <xacro:magnetometer_plugin_macro
     namespace="${namespace}"
-    pub_rate="20"
+    pub_rate="100"
     noise_density="0.0004"
     random_walk="0.0000064"
@@ -478,6 +481,7 @@
   <xacro:barometer_plugin_macro
   namespace="${namespace}"
-  pub_rate="10"
+  pub_rate="50"
   baro_topic="/baro"
+  baro_drift_pa_per_sec="0"
   >
   </xacro:barometer_plugin_macro>
@@ -490,9 +494,9 @@
     imu_topic="/imu"
     mass_imu_sensor="0.015"
-    gyroscope_noise_density="0.0003394"
-    gyroscopoe_random_walk="0.000038785"
+    gyroscope_noise_density="0.00018665"
+    gyroscope_random_walk="0.000038785"
     gyroscope_bias_correlation_time="1000.0"
     gyroscope_turn_on_bias_sigma="0.0087"
-    accelerometer_noise_density="0.004"
+    accelerometer_noise_density="0.00186"
     accelerometer_random_walk="0.006"
     accelerometer_bias_correlation_time="300.0"

File: models/mrs_robots_description/urdf/f550.xacro (robot description, xacro)
@@ -486,5 +486,4 @@
     namespace="${namespace}"
     imu_sub_topic="/imu"
-    gps_sub_topic="/gps"
     mag_sub_topic="/mag"
     baro_sub_topic="/baro"
@@ -510,21 +509,25 @@
   <!--}-->
   <!-- GPS {-->
-  <xacro:gps_plugin_macro
+  <xacro:gps_macro
+    gps_name="gps0"
+    pos_x="0.0"
+    pos_y="0.0"
+    pos_z="0.0"
+    gps_noise="true"
+    gps_xy_random_walk="2.0"
+    gps_z_random_walk="4.0"
+    gps_xy_noise_density="2.0e-4"
+    gps_z_noise_density="4.0e-4"
+    gps_vxy_noise_density="0.2"
+    gps_vz_noise_density="0.4"
+    update_rate="10"
     namespace="${namespace}"
-    gps_noise="true"
-    gps_indoor_jamming="$(arg gps_indoor_jamming)">
-    >
-  </xacro:gps_plugin_macro>
-  <xacro:if value="$(arg gps_indoor_jamming)">
-    <xacro:gps_satelites_blocking_macro
-      namespace="${namespace}"
-      parent_link="base_link">
-    </xacro:gps_satelites_blocking_macro>
-  </xacro:if>
+    parent_link="base_link">
+  </xacro:gps_macro>
   <!--}-->
   <!-- Magnetometer {-->
   <xacro:magnetometer_plugin_macro
     namespace="${namespace}"
-    pub_rate="20"
+    pub_rate="100"
     noise_density="0.0004"
     random_walk="0.0000064"
@@ -537,6 +540,7 @@
   <xacro:barometer_plugin_macro
     namespace="${namespace}"
-    pub_rate="10"
+    pub_rate="50"
     baro_topic="/baro"
+    baro_drift_pa_per_sec="0"
     >
   </xacro:barometer_plugin_macro>
@@ -549,9 +553,9 @@
     imu_topic="/imu"
     mass_imu_sensor="0.015"
-    gyroscope_noise_density="0.0003394"
-    gyroscopoe_random_walk="0.000038785"
+    gyroscope_noise_density="0.00018665"
+    gyroscope_random_walk="0.000038785"
     gyroscope_bias_correlation_time="1000.0"
     gyroscope_turn_on_bias_sigma="0.0087"
-    accelerometer_noise_density="0.004"
+    accelerometer_noise_density="0.00186"
     accelerometer_random_walk="0.006"
     accelerometer_bias_correlation_time="300.0"

File: models/mrs_robots_description/urdf/t650.xacro (robot description, xacro)
@@ -402,5 +402,4 @@
     namespace="${namespace}"
     imu_sub_topic="/imu"
-    gps_sub_topic="/gps"
     mag_sub_topic="/mag"
     baro_sub_topic="/baro"
@@ -426,21 +425,25 @@
   <!--}-->
   <!-- GPS {-->
-  <xacro:gps_plugin_macro
+  <xacro:gps_macro
+    gps_name="gps0"
+    pos_x="0.0"
+    pos_y="0.0"
+    pos_z="0.0"
+    gps_noise="true"
+    gps_xy_random_walk="2.0"
+    gps_z_random_walk="4.0"
+    gps_xy_noise_density="2.0e-4"
+    gps_z_noise_density="4.0e-4"
+    gps_vxy_noise_density="0.2"
+    gps_vz_noise_density="0.4"
+    update_rate="10"
     namespace="${namespace}"
-    gps_noise="true"
-    gps_indoor_jamming="$(arg gps_indoor_jamming)">
-    >
-  </xacro:gps_plugin_macro>
-  <xacro:if value="$(arg gps_indoor_jamming)">
-    <xacro:gps_satelites_blocking_macro
-      namespace="${namespace}"
-      parent_link="base_link">
-    </xacro:gps_satelites_blocking_macro>
-  </xacro:if>
+    parent_link="base_link">
+  </xacro:gps_macro>
   <!--}-->
   <!-- Magnetometer {-->
   <xacro:magnetometer_plugin_macro
     namespace="${namespace}"
-    pub_rate="20"
+    pub_rate="100"
     noise_density="0.0004"
     random_walk="0.0000064"
@@ -453,6 +456,7 @@
   <xacro:barometer_plugin_macro
     namespace="${namespace}"
-    pub_rate="10"
+    pub_rate="50"
     baro_topic="/baro"
+    baro_drift_pa_per_sec="0"
     >
   </xacro:barometer_plugin_macro>
@@ -465,9 +469,9 @@
     imu_topic="/imu"
     mass_imu_sensor="0.015"
-    gyroscope_noise_density="0.0003394"
-    gyroscopoe_random_walk="0.000038785"
+    gyroscope_noise_density="0.00018665"
+    gyroscope_random_walk="0.000038785"
     gyroscope_bias_correlation_time="1000.0"
     gyroscope_turn_on_bias_sigma="0.0087"
-    accelerometer_noise_density="0.004"
+    accelerometer_noise_density="0.00186"
     accelerometer_random_walk="0.006"
     accelerometer_bias_correlation_time="300.0"

Commit message: updated the ball hodler

File: models/mrs_robots_description/urdf/component_snippets.xacro (robot description, xacro)
@@ -4777,32 +4777,15 @@
         </inertial>
     </link>
-    <joint name="ball_holder2_rod_joint" type="fixed">
-        <parent link="ball_holder2_spherical_joint_helper_link2"/>
-        <child link="ball_holder2_rod"/>
-        <origin xyz="0.0 0.0 -0.79" rpy="0.0 0.0 0.0"/>
-    </joint>
-    <link name="ball_holder2_rod">
-        <inertial>
-            <mass value="0.025" />
-            <inertia ixx="0.00004712" ixy="0.0" ixz="0.0" iyy="0.00004712" iyz="0.0" izz="0.00000112"/>
-        </inertial>
-        <visual>
-            <geometry>
-                <cylinder radius="0.0075" length="0.450" />
-            </geometry>
-            <origin rpy="0.0 0.0 0.0" xyz="0.0 0.0 0.0" />
-        </visual>
-    </link>
     <joint name="ball_holder_ball_joint" type="revolute">
-        <parent link="ball_holder2_rod"/>
+        <parent link="ball_holder_rod"/>
         <child link="ball_holder_ball"/>
         <axis xyz="0 1 0"/>
         <dynamics damping="0.05" friction="0.08"/>
         <limit upper="0" lower="0" effort="0" velocity="0" />
-        <origin xyz="0.0 0.0 -0.225" rpy="0.0 0.0 0.0"/>
+        <origin xyz="0.0 0.0 -0.5" rpy="0.0 0.0 0.0"/>
     </joint>
     <link name="ball_holder_ball">
         <inertial>
-            <mass value="0.1" />
+            <mass value="0.2" />
             <inertia ixx="0.00000012" ixy="0.0" ixz="0.0" iyy="0.00000012" iyz="0.0" izz="0.00000012"/>
         </inertial>

Commit message: new platform: X500

File: models/mrs_robots_description/urdf/component_snippets.xacro (robot description, xacro)
@@ -56,5 +56,5 @@
   <!-- ================================================================== -->
   <!--  {-->
-  <!-- Macro for visualization of mash {-->
+  <!-- Macro for visualization of mesh {-->
   <xacro:macro name="visual_macro"
     params="robot_namespace name mesh_file mesh_scale color parent *origin">
@@ -69,4 +69,24 @@
         <geometry>
           <mesh filename="${mesh_file}" scale="${mesh_scale}" />
+        </geometry>
+      </visual>
+    </link>
+    <gazebo reference="${name}_link">
+      <material>Gazebo/${color}</material>
+    </gazebo>
+  </xacro:macro>
+  <!--}-->
+  <!-- Macro for visualization of colored box {-->
+  <xacro:macro name="colored_box"
+    params="robot_namespace name size_x size_y size_z color parent *origin">
+    <joint name="${name}_joint" type="fixed">
+      <xacro:insert_block name="origin" />
+      <parent link="${parent}" />
+      <child link="${name}_link" />
+    </joint>
+    <link name="${name}_link">
+      <visual>
+        <geometry>
+          <box size="${size_x} ${size_y} ${size_z}" />
         </geometry>
       </visual>

File: models/mrs_robots_description/urdf/t650.xacro (robot description, xacro)
@@ -306,5 +306,5 @@
     rolling_moment_coefficient="${rolling_moment_coefficient}"
     mesh_file="${prop_mesh_file}"
-    mesh_scale="${mesh_scale_prop_cw}">
+    mesh_scale="${mesh_scale_prop_ccw}">
     <origin xyz="${arm_length * sin45} -${arm_length * sin45} ${propeller_offset}"  rpy="0 0 0" />
     <xacro:insert_block name="rotor_inertia" />
@@ -325,5 +325,5 @@
     rolling_moment_coefficient="${rolling_moment_coefficient}"
     mesh_file="${prop_mesh_file}"
-    mesh_scale="${mesh_scale_prop_cw}">
+    mesh_scale="${mesh_scale_prop_ccw}">
     <origin xyz="-${arm_length * sin45} ${arm_length * sin45} ${propeller_offset}" rpy="0 0 0" />
     <xacro:insert_block name="rotor_inertia" />
@@ -365,5 +365,5 @@
     rolling_moment_coefficient="${rolling_moment_coefficient}"
     mesh_file="${prop_mesh_file}"
-    mesh_scale="${mesh_scale_prop_ccw}">
+    mesh_scale="${mesh_scale_prop_cw}">
     <origin xyz="-${arm_length * sin45} -${arm_length * sin45} ${propeller_offset}" rpy="0 0 0" />
     <xacro:insert_block name="rotor_inertia" />

Commit message: update imu_vio for f330

File: models/mrs_robots_description/urdf/component_snippets.xacro (robot description, xacro)
@@ -619,4 +619,24 @@
         <accelerometerBiasCorrelationTime>${accelerometer_bias_correlation_time}</accelerometerBiasCorrelationTime> <!-- Accelerometer bias correlation time constant [s] -->
         <accelerometerTurnOnBiasSigma>${accelerometer_turn_on_bias_sigma}</accelerometerTurnOnBiasSigma> <!-- Accelerometer turn on bias standard deviation [m/s^2] -->
+      </plugin>
+    </gazebo>
+  </xacro:macro>
+  <!--}-->
+  <!-- Macro to add custom imu{-->
+  <!-- Macro to add a custom IMU. -->
+  <xacro:macro name="custom_imu_plugin_macro"
+    params="namespace body_name topic_name service_name gaussian_noise update_rate
+    frame_name x y z roll pitch yaw">
+    <gazebo>
+      <plugin name="imu_plugin" filename="libgazebo_ros_imu.so">
+        <alwaysOn>true</alwaysOn>
+        <bodyName>${body_name}</bodyName>
+        <topicName>${topic_name}</topicName>
+        <serviceName>${service_name}</serviceName>
+        <gaussianNoise>${gaussian_noise}</gaussianNoise>
+        <updateRate>${update_rate}</updateRate>
+        <frameName>${frame_name}</frameName>
+        <xyzOffset>${x} ${y} ${z}</xyzOffset>
+        <rpyOffset>${roll} ${pitch} ${yaw}</rpyOffset>
       </plugin>
     </gazebo>

File: models/mrs_robots_description/urdf/f330.xacro (robot description, xacro)
@@ -576,14 +576,20 @@
   <!--}-->
   <!-- High rate IMU {-->
-  <gazebo>
-    <plugin name="imu_plugin" filename="libgazebo_ros_imu.so">
-      <alwaysOn>true</alwaysOn>
-      <bodyName>base_link</bodyName>
-      <topicName>imu_vio</topicName>
-      <serviceName>imu_vio_service</serviceName>
-      <gaussianNoise>0.0</gaussianNoise>
-      <updateRate>125.0</updateRate>
-    </plugin>
-  </gazebo>
+  <xacro:custom_imu_plugin_macro
+    namespace="${namespace}"
+    body_name="base_link"
+    topic_name ="imu_vio"
+    service_name ="imu_vio_service"
+    gaussian_noise="0.0"
+    update_rate="125.0"
+    frame_name="${namespace}/fisheye_camera_optical"
+    x="0"
+    y="0"
+    z="0"
+    roll="${rad90}"
+    pitch="${rad90}"
+    yaw="0"
+    >
+  </xacro:custom_imu_plugin_macro>
   <!--}-->
   </xacro:if>
