Commit message: vio update

File: models/mrs_robots_description/urdf/component_snippets.xacro (robot description, xacro)
@@ -986,4 +986,106 @@
     </gazebo>
     <gazebo reference="${namespace}/camera_${camera_suffix}_link">
+      <material>Gazebo/DarkGrey</material>
+    </gazebo>
+  </xacro:macro>
+  <!--}-->
+  <!-- Macro to add a fisheye camera with integrated imu {-->
+  <xacro:macro name="vio_macro"
+    params="namespace parent_link camera_frame_name sensor_base_frame_name frame_rate parent_frame_name
+    horizontal_fov image_width image_height min_distance max_distance lens_type lens_c1 lens_c2 lens_f lens_fun lens_scale lens_cutoff_angle lens_texture_size x y z roll pitch yaw
+   camera_noise_mean camera_noise_stddev imu_rate imu_topic imu_noise_mean">
+    <link name="${namespace}/vio_link">
+      <visual>
+        <origin xyz="0 0 0" rpy="${rad90} 0 0" />
+        <geometry>
+          <mesh filename="package://mrs_robots_description/meshes/sensors/bluefox.dae" scale="1 1 1" />
+        </geometry>
+      </visual>
+    </link>
+    <joint name="${namespace}/vio_joint" type="fixed">
+      <origin xyz="${x} ${y} ${z}" rpy="${roll} ${pitch} ${yaw}"/>
+      <parent link="${parent_link}" />
+      <child link="${namespace}/vio_link" />
+    </joint>
+    <gazebo reference="${namespace}/vio_link">
+      <!-- wide angle camera {-->
+      <sensor type="wideanglecamera" name="${namespace}_vio_camera">
+        <update_rate>${frame_rate}</update_rate>
+        <camera name="head">
+          <horizontal_fov>${horizontal_fov}</horizontal_fov>
+          <image>
+            <width>${image_width}</width>
+            <height>${image_height}</height>
+          </image>
+          <clip>
+            <near>${min_distance}</near>
+            <far>${max_distance}</far>
+          </clip>
+          <noise>
+            <type>gaussian</type>
+            <!-- Noise is sampled independently per pixel on each frame.
+            That pixel's noise value is added to each of its color
+            channels, which at that point lie in the range [0,1]. -->
+            <mean>${camera_noise_mean}</mean>
+            <stddev>${camera_noise_stddev}</stddev>
+          </noise>
+          <lens>
+            <type>${lens_type}</type>
+            <custom_function>
+              <c1>${lens_c1}</c1>
+              <c2>${lens_c2}</c2>
+              <f>${lens_f}</f>
+              <fun>${lens_fun}</fun>
+            </custom_function>
+            <scale_to_hfov>${lens_scale}</scale_to_hfov>
+            <cutoff_angle>${lens_cutoff_angle}</cutoff_angle>
+            <env_texture_size>${lens_texture_size}</env_texture_size>
+          </lens>
+        </camera>
+        <plugin name="${namespace}_vio_camera_controller" filename="libMRSGazeboCameraPlugin.so">
+          <alwaysOn>true</alwaysOn>
+          <updateRate>${frame_rate}</updateRate>
+          <cameraName>vio_camera</cameraName>
+          <imageTopicName>image_raw</imageTopicName>
+          <cameraInfoTopicName>camera_info</cameraInfoTopicName>
+          <frameName>/${camera_frame_name}</frameName>
+          <hackBaseline>0.0</hackBaseline>
+          <distortionK1>0.0</distortionK1>
+          <distortionK2>0.0</distortionK2>
+          <distortionK3>0.0</distortionK3>
+          <distortionT1>0.0</distortionT1>
+          <distortionT2>0.0</distortionT2>
+          <parentFrameName>${parent_frame_name}</parentFrameName>
+          <sensorBaseFrameName>${sensor_base_frame_name}</sensorBaseFrameName>
+          <x>${x}</x>
+          <y>${y}</y>
+          <z>${z}</z>
+          <roll>${roll}</roll>
+          <pitch>${pitch}</pitch>
+          <yaw>${yaw}</yaw>
+        </plugin>
+      </sensor>
+      <!--}-->
+    <!-- imu {-->
+    <sensor name="imu_sensor" type="imu">
+      <always_on>true</always_on>
+      <update_rate>${imu_rate}</update_rate>
+      <visualize>true</visualize>
+      <topic>__default_topic__</topic>
+      <plugin filename="libgazebo_ros_imu_sensor.so" name="imu_plugin">
+        <topicName>${imu_topic}</topicName>
+        <bodyName>${namespace}/vio_link</bodyName>
+        <updateRateHZ>${imu_rate}</updateRateHZ>
+        <gaussianNoise>${imu_noise_mean}</gaussianNoise>
+        <xyzOffset>0 0 0</xyzOffset>
+        <rpyOffset>0 0 0</rpyOffset>
+        <frameName>${namespace}/vio_link</frameName>
+        <initialOrientationAsReference>false</initialOrientationAsReference>
+      </plugin>
+      <pose>0 0 0 0 0 0</pose>
+    </sensor>
+    <!--}-->
+    </gazebo>
+    <gazebo reference="${namespace}/vio_link">
       <material>Gazebo/DarkGrey</material>
     </gazebo>

File: models/mrs_robots_description/urdf/f330.xacro (robot description, xacro)
@@ -546,15 +546,28 @@
   <!--}-->
   <!-- VIO {-->
-  <!-- fisheye forward {-->
+  <!-- fisheye forward with imu {-->
   <xacro:if value="${optionals['enable_vio']}">
-    <xacro:fisheye_camera_macro
+    <xacro:vio_macro
       namespace="${namespace}"
       parent_link="base_link"
-      camera_suffix="fisheye_camera"
-      frame_rate="45"
-      noise="0.000"
       parent_frame_name="${namespace}/fcu"
       camera_frame_name="${namespace}/fisheye_camera_optical"
       sensor_base_frame_name="${namespace}/fisheye_camera"
+      frame_rate="45"
+      horizontal_fov="${rad180}"
+      image_width="752"
+      image_height="480"
+      lens_type="custom"
+      lens_c1="1.05"
+      lens_c2="4"
+      lens_f="1.0"
+      lens_fun="tan"
+      lens_scale="true"
+      lens_cutoff_angle="${rad90}"
+      lens_texture_size="512"
+      min_distance="0.02"
+      max_distance="40"
+      camera_noise_mean="0.0"
+      camera_noise_stddev="0.0"
       x="0.107"
       y="0"
@@ -563,33 +576,18 @@
       pitch="0"
       yaw="0.0"
+      imu_rate="125.0"
+      imu_topic="imu_vio"
+      imu_noise_mean="0.0"
       >
-  </xacro:fisheye_camera_macro>
-  <xacro:visual_macro
-    robot_namespace="${namespace}"
-    name="bluefox_mount"
-    mesh_file="${bluefox_mount_mesh}"
-    mesh_scale="${mesh_scale}"
-    parent="base_link"
-    color="Black">
-    <origin xyz="0 0 0" rpy="0 0 ${-rad90}" />
-  </xacro:visual_macro>
-  <!--}-->
-  <!-- High rate IMU {-->
-  <xacro:custom_imu_plugin_macro
-    namespace="${namespace}"
-    body_name="base_link"
-    topic_name ="imu_vio"
-    service_name ="imu_vio_service"
-    gaussian_noise="0.0"
-    update_rate="125.0"
-    frame_name="${namespace}/fisheye_camera_optical"
-    x="0"
-    y="0"
-    z="0"
-    roll="${rad90}"
-    pitch="${rad90}"
-    yaw="0"
-    >
-  </xacro:custom_imu_plugin_macro>
+    </xacro:vio_macro>
+    <xacro:visual_macro
+      robot_namespace="${namespace}"
+      name="bluefox_mount"
+      mesh_file="${bluefox_mount_mesh}"
+      mesh_scale="${mesh_scale}"
+      parent="base_link"
+      color="Black">
+      <origin xyz="0 0 0" rpy="0 0 ${-rad90}" />
+    </xacro:visual_macro>
   <!--}-->
   </xacro:if>

Commit message: vio axes update

File: models/mrs_robots_description/urdf/component_snippets.xacro (robot description, xacro)
@@ -995,5 +995,5 @@
     horizontal_fov image_width image_height min_distance max_distance lens_type lens_c1 lens_c2 lens_f lens_fun lens_scale lens_cutoff_angle lens_texture_size x y z roll pitch yaw
    camera_noise_mean camera_noise_stddev imu_rate imu_topic imu_noise_mean">
-    <link name="${namespace}/vio_link">
+    <link name="${namespace}/vio_camera_link">
       <visual>
         <origin xyz="0 0 0" rpy="${rad90} 0 0" />
@@ -1003,10 +1003,18 @@
       </visual>
     </link>
-    <joint name="${namespace}/vio_joint" type="fixed">
+    <joint name="${namespace}/vio_camera_joint" type="fixed">
       <origin xyz="${x} ${y} ${z}" rpy="${roll} ${pitch} ${yaw}"/>
       <parent link="${parent_link}" />
-      <child link="${namespace}/vio_link" />
-    </joint>
-    <gazebo reference="${namespace}/vio_link">
+      <child link="${namespace}/vio_camera_link" />
+    </joint>
+    <link name="${namespace}/vio_imu_link">
+      <pose>0 0 0 0 0 0</pose>
+    </link>
+    <joint name="${namespace}/vio_imu_joint" type="fixed">
+      <origin xyz="0 0 0" rpy="${rad90} 0 0"/> <!-- TODO maybe some tweaking here is necessary -->
+      <parent link="${namespace}/vio_camera_link" />
+      <child link="${namespace}/vio_imu_link" />
+    </joint>
+    <gazebo reference="${namespace}/vio_camera_link">
       <!-- wide angle camera {-->
       <sensor type="wideanglecamera" name="${namespace}_vio_camera">
@@ -1066,25 +1074,27 @@
         </plugin>
       </sensor>
-      <!--}-->
+    </gazebo>
+    <!--}-->
     <!-- imu {-->
-    <sensor name="imu_sensor" type="imu">
-      <always_on>true</always_on>
-      <update_rate>${imu_rate}</update_rate>
-      <visualize>true</visualize>
-      <topic>__default_topic__</topic>
-      <plugin filename="libgazebo_ros_imu_sensor.so" name="imu_plugin">
-        <topicName>${imu_topic}</topicName>
-        <bodyName>${namespace}/vio_link</bodyName>
-        <updateRateHZ>${imu_rate}</updateRateHZ>
-        <gaussianNoise>${imu_noise_mean}</gaussianNoise>
-        <xyzOffset>0 0 0</xyzOffset>
-        <rpyOffset>0 0 0</rpyOffset>
-        <frameName>${namespace}/vio_link</frameName>
-        <initialOrientationAsReference>false</initialOrientationAsReference>
-      </plugin>
-      <pose>0 0 0 0 0 0</pose>
-    </sensor>
+    <gazebo reference="${namespace}/vio_imu_link">
+      <sensor name="imu_sensor" type="imu">
+        <always_on>true</always_on>
+        <update_rate>${imu_rate}</update_rate>
+        <visualize>true</visualize>
+        <topic>__default_topic__</topic>
+        <plugin filename="libgazebo_ros_imu_sensor.so" name="imu_plugin">
+          <topicName>${imu_topic}</topicName>
+          <bodyName>${namespace}/vio_imu_link</bodyName>
+          <updateRateHZ>${imu_rate}</updateRateHZ>
+          <gaussianNoise>${imu_noise_mean}</gaussianNoise>
+          <xyzOffset>0 0 0</xyzOffset>
+          <rpyOffset>0 0 0</rpyOffset>
+          <frameName>${namespace}/vio_camera_link</frameName>
+          <initialOrientationAsReference>false</initialOrientationAsReference>
+        </plugin>
+        <pose>0 0 0 0 0 0</pose>
+      </sensor>
+    </gazebo>
     <!--}-->
-    </gazebo>
     <gazebo reference="${namespace}/vio_link">
       <material>Gazebo/DarkGrey</material>

Commit message: update timepix placement

File: models/mrs_robots_description/urdf/component_snippets.xacro (robot description, xacro)
@@ -2311,7 +2311,7 @@
     <link name="${name}_link">
       <visual>
-        <origin xyz="0 0 0" rpy="0 0 0" />
-        <geometry>
-          <box size="0.02 0.1 0.1" />
+        <origin xyz="0 0.05 0" rpy="0 0 0" />
+        <geometry>
+          <box size="0.02 0.09 0.02" />
         </geometry>
       </visual>

File: models/mrs_robots_description/urdf/f450.xacro (robot description, xacro)
@@ -1033,5 +1033,5 @@
       parent="base_link"
       color="Green">
-      <origin xyz="0 0 0" rpy="0 0 0" />
+      <origin xyz="0.115 -0.05 -0.05" rpy="0 0 0" />
     </xacro:timepix_macro>
   </xacro:if>

File: models/mrs_robots_description/urdf/f550.xacro (robot description, xacro)
@@ -1089,5 +1089,5 @@
       parent="base_link"
       color="Green">
-      <origin xyz="0 0 0" rpy="0 0 0" />
+      <origin xyz="0.115 -0.05 -0.05" rpy="0 0 0" />
     </xacro:timepix_macro>
   </xacro:if>

File: models/mrs_robots_description/urdf/t650.xacro (robot description, xacro)
@@ -947,5 +947,5 @@
       parent="base_link"
       color="Green">
-      <origin xyz="0 0 0" rpy="0 0 0" />
+      <origin xyz="0.115 -0.05 -0.05" rpy="0 0 0" />
     </xacro:timepix_macro>
   </xacro:if>

Commit message: update sensor definitions for vio

File: models/mrs_robots_description/urdf/component_snippets.xacro (robot description, xacro)
@@ -623,21 +623,33 @@
   </xacro:macro>
   <!--}-->
-  <!-- Macro to add custom imu{-->
-  <!-- Macro to add a custom IMU. -->
-  <xacro:macro name="custom_imu_plugin_macro"
-    params="namespace body_name topic_name service_name gaussian_noise update_rate
-    frame_name x y z roll pitch yaw">
-    <gazebo>
-      <plugin name="imu_plugin" filename="libgazebo_ros_imu.so">
-        <alwaysOn>true</alwaysOn>
-        <bodyName>${body_name}</bodyName>
-        <topicName>${topic_name}</topicName>
-        <serviceName>${service_name}</serviceName>
-        <gaussianNoise>${gaussian_noise}</gaussianNoise>
-        <updateRate>${update_rate}</updateRate>
-        <frameName>${frame_name}</frameName>
-        <xyzOffset>${x} ${y} ${z}</xyzOffset>
-        <rpyOffset>${roll} ${pitch} ${yaw}</rpyOffset>
-      </plugin>
+  <!-- Macro to add imu with configurable rate {-->
+  <xacro:macro name="custom_imu_macro"
+    params="namespace parent_link sensor_name update_rate topic_name noise_mean *origin">
+    <link name="${namespace}/${sensor_name}_link">
+      <pose>0 0 0 0 0 0</pose>
+    </link>
+    <joint name="${namespace}/${sensor_name}_joint" type="fixed">
+      <xacro:insert_block name="origin" />
+      <parent link="${parent_link}" />
+      <child link="${namespace}/${sensor_name}_link" />
+    </joint>
+    <gazebo reference="${namespace}/${sensor_name}_link">
+      <sensor name="${sensor_name}" type="imu">
+        <always_on>true</always_on>
+        <update_rate>${update_rate}</update_rate>
+        <visualize>true</visualize>
+        <topic>__default_topic__</topic>
+        <plugin filename="libgazebo_ros_imu_sensor.so" name="imu_plugin">
+          <topicName>${topic_name}</topicName>
+          <bodyName>${namespace}/${sensor_name}_link</bodyName>
+          <updateRateHZ>${imu_rate}</updateRateHZ>
+          <gaussianNoise>${imu_noise_mean}</gaussianNoise>
+          <xyzOffset>0 0 0</xyzOffset>
+          <rpyOffset>0 0 0</rpyOffset>
+          <frameName>${parent_link}</frameName>
+          <initialOrientationAsReference>false</initialOrientationAsReference>
+        </plugin>
+        <pose>0 0 0 0 0 0</pose>
+      </sensor>
     </gazebo>
   </xacro:macro>
@@ -986,116 +998,4 @@
     </gazebo>
     <gazebo reference="${namespace}/camera_${camera_suffix}_link">
-      <material>Gazebo/DarkGrey</material>
-    </gazebo>
-  </xacro:macro>
-  <!--}-->
-  <!-- Macro to add a fisheye camera with integrated imu {-->
-  <xacro:macro name="vio_macro"
-    params="namespace parent_link camera_frame_name sensor_base_frame_name frame_rate parent_frame_name
-    horizontal_fov image_width image_height min_distance max_distance lens_type lens_c1 lens_c2 lens_f lens_fun lens_scale lens_cutoff_angle lens_texture_size x y z roll pitch yaw
-   camera_noise_mean camera_noise_stddev imu_rate imu_topic imu_noise_mean">
-    <link name="${namespace}/vio_camera_link">
-      <visual>
-        <origin xyz="0 0 0" rpy="${rad90} 0 0" />
-        <geometry>
-          <mesh filename="package://mrs_robots_description/meshes/sensors/bluefox.dae" scale="1 1 1" />
-        </geometry>
-      </visual>
-    </link>
-    <joint name="${namespace}/vio_camera_joint" type="fixed">
-      <origin xyz="${x} ${y} ${z}" rpy="${roll} ${pitch} ${yaw}"/>
-      <parent link="${parent_link}" />
-      <child link="${namespace}/vio_camera_link" />
-    </joint>
-    <link name="${namespace}/vio_imu_link">
-      <pose>0 0 0 0 0 0</pose>
-    </link>
-    <joint name="${namespace}/vio_imu_joint" type="fixed">
-      <origin xyz="0 0 0" rpy="${rad90} 0 0"/> <!-- TODO maybe some tweaking here is necessary -->
-      <parent link="${namespace}/vio_camera_link" />
-      <child link="${namespace}/vio_imu_link" />
-    </joint>
-    <gazebo reference="${namespace}/vio_camera_link">
-      <!-- wide angle camera {-->
-      <sensor type="wideanglecamera" name="${namespace}_vio_camera">
-        <update_rate>${frame_rate}</update_rate>
-        <camera name="head">
-          <horizontal_fov>${horizontal_fov}</horizontal_fov>
-          <image>
-            <width>${image_width}</width>
-            <height>${image_height}</height>
-          </image>
-          <clip>
-            <near>${min_distance}</near>
-            <far>${max_distance}</far>
-          </clip>
-          <noise>
-            <type>gaussian</type>
-            <!-- Noise is sampled independently per pixel on each frame.
-            That pixel's noise value is added to each of its color
-            channels, which at that point lie in the range [0,1]. -->
-            <mean>${camera_noise_mean}</mean>
-            <stddev>${camera_noise_stddev}</stddev>
-          </noise>
-          <lens>
-            <type>${lens_type}</type>
-            <custom_function>
-              <c1>${lens_c1}</c1>
-              <c2>${lens_c2}</c2>
-              <f>${lens_f}</f>
-              <fun>${lens_fun}</fun>
-            </custom_function>
-            <scale_to_hfov>${lens_scale}</scale_to_hfov>
-            <cutoff_angle>${lens_cutoff_angle}</cutoff_angle>
-            <env_texture_size>${lens_texture_size}</env_texture_size>
-          </lens>
-        </camera>
-        <plugin name="${namespace}_vio_camera_controller" filename="libMRSGazeboCameraPlugin.so">
-          <alwaysOn>true</alwaysOn>
-          <updateRate>${frame_rate}</updateRate>
-          <cameraName>vio_camera</cameraName>
-          <imageTopicName>image_raw</imageTopicName>
-          <cameraInfoTopicName>camera_info</cameraInfoTopicName>
-          <frameName>/${camera_frame_name}</frameName>
-          <hackBaseline>0.0</hackBaseline>
-          <distortionK1>0.0</distortionK1>
-          <distortionK2>0.0</distortionK2>
-          <distortionK3>0.0</distortionK3>
-          <distortionT1>0.0</distortionT1>
-          <distortionT2>0.0</distortionT2>
-          <parentFrameName>${parent_frame_name}</parentFrameName>
-          <sensorBaseFrameName>${sensor_base_frame_name}</sensorBaseFrameName>
-          <x>${x}</x>
-          <y>${y}</y>
-          <z>${z}</z>
-          <roll>${roll}</roll>
-          <pitch>${pitch}</pitch>
-          <yaw>${yaw}</yaw>
-        </plugin>
-      </sensor>
-    </gazebo>
-    <!--}-->
-    <!-- imu {-->
-    <gazebo reference="${namespace}/vio_imu_link">
-      <sensor name="imu_sensor" type="imu">
-        <always_on>true</always_on>
-        <update_rate>${imu_rate}</update_rate>
-        <visualize>true</visualize>
-        <topic>__default_topic__</topic>
-        <plugin filename="libgazebo_ros_imu_sensor.so" name="imu_plugin">
-          <topicName>${imu_topic}</topicName>
-          <bodyName>${namespace}/vio_imu_link</bodyName>
-          <updateRateHZ>${imu_rate}</updateRateHZ>
-          <gaussianNoise>${imu_noise_mean}</gaussianNoise>
-          <xyzOffset>0 0 0</xyzOffset>
-          <rpyOffset>0 0 0</rpyOffset>
-          <frameName>${namespace}/vio_camera_link</frameName>
-          <initialOrientationAsReference>false</initialOrientationAsReference>
-        </plugin>
-        <pose>0 0 0 0 0 0</pose>
-      </sensor>
-    </gazebo>
-    <!--}-->
-    <gazebo reference="${namespace}/vio_link">
       <material>Gazebo/DarkGrey</material>
     </gazebo>
@@ -2073,4 +1973,38 @@
   </xacro:macro>
   <!--}-->
+  <!-- Macro to add a fisheye camera with integrated imu {-->
+  <xacro:macro name="vio_macro"
+    params="namespace parent_link camera_frame_name sensor_base_frame_name frame_rate parent_frame_name
+    horizontal_fov image_width image_height min_distance max_distance lens_type lens_c1 lens_c2 lens_f lens_fun lens_scale lens_cutoff_angle lens_texture_size x y z roll pitch yaw
+   camera_noise_mean imu_rate imu_topic imu_noise_mean">
+    <xacro:fisheye_camera_macro
+      namespace="${namespace}"
+      parent_link="${parent_link}"
+      camera_suffix="vio"
+      frame_rate="${frame_rate}"
+      noise="${camera_noise_mean}"
+      x="${x}"
+      y="${y}"
+      z="${z}"
+      roll="${roll}"
+      pitch="${pitch}"
+      yaw="${yaw}"
+      camera_frame_name="${camera_frame_name}"
+      sensor_base_frame_name="${sensor_base_frame_name}"
+      parent_frame_name="${parent_frame_name}"
+      >
+    </xacro:fisheye_camera_macro>
+    <xacro:custom_imu_macro
+      namespace="${namespace}"
+      parent_link="${namespace}/camera_vio_link"
+      sensor_name="vio_imu"
+      update_rate="${imu_rate}"
+      topic_name="${imu_topic}"
+      noise_mean="${imu_noise_mean}"
+      >
+      <origin xyz="0 0 0" rpy="${rad90} 0 0"/>
+    </xacro:custom_imu_macro>
+  </xacro:macro>
+  <!--}-->
   <!-- ========================== other sensors ========================= -->
   <!-- Macro to add a Teraranger Tower Evo {-->

File: models/mrs_robots_description/urdf/f330.xacro (robot description, xacro)
@@ -569,5 +569,4 @@
       max_distance="40"
       camera_noise_mean="0.0"
-      camera_noise_stddev="0.0"
       x="0.107"
       y="0"

Commit message: [vio]: update topics and frames

File: models/mrs_robots_description/urdf/component_snippets.xacro (robot description, xacro)
@@ -977,6 +977,6 @@
           <updateRate>${frame_rate}</updateRate>
           <cameraName>${camera_suffix}</cameraName>
-          <imageTopicName>image_raw</imageTopicName>
-          <cameraInfoTopicName>camera_info</cameraInfoTopicName>
+          <imageTopicName>camera/image_raw</imageTopicName>
+          <cameraInfoTopicName>camera/camera_info</cameraInfoTopicName>
           <frameName>/${camera_frame_name}</frameName>
           <hackBaseline>0.0</hackBaseline>
@@ -2003,5 +2003,5 @@
       noise_mean="${imu_noise_mean}"
       >
-      <origin xyz="0 0 0" rpy="${rad90} 0 0"/>
+      <origin xyz="0 0 0" rpy="${-rad90} 0 0"/>
     </xacro:custom_imu_macro>
   </xacro:macro>

File: models/mrs_robots_description/urdf/f330.xacro (robot description, xacro)
@@ -576,5 +576,5 @@
       yaw="0.0"
       imu_rate="125.0"
-      imu_topic="imu_vio"
+      imu_topic="vio/imu"
       imu_noise_mean="0.0"
       >
