Commit message: remove individual sensor names for each ouster type: all ousters are now named os

File: models/mrs_robots_description/urdf/component_snippets.xacro (robot description, xacro)
@@ -1364,7 +1364,7 @@
     <xacro:property name="frame_imu" value="${namespace}/${sensor_name}_imu" />
       <!-- topics -->
-    <xacro:property name="topic_lidar" value="/${namespace}/${sensor_name}_cloud_node/points" />
-    <xacro:property name="topic_imu" value="/${namespace}/${sensor_name}_cloud_node/imu" />
-    <xacro:property name="topic_diag" value="/${namespace}/${sensor_name}_cloud_node/diag" />
+    <xacro:property name="topic_lidar" value="/${namespace}/${sensor_name}_cloud_nodelet/points" />
+    <xacro:property name="topic_imu" value="/${namespace}/${sensor_name}_cloud_nodelet/imu" />
+    <xacro:property name="topic_diag" value="/${namespace}/${sensor_name}_cloud_nodelet/diag" />
       <!-- tf from sensor to lidar -->
     <xacro:property name="lidar_x" value="0" />

File: models/mrs_robots_description/urdf/f450.xacro (robot description, xacro)
@@ -636,10 +636,8 @@
     <xacro:property name="ouster_model" value="${optionals['ouster_model']}" />
     <!-- OS1-16 Generation 1 (default) -->
-    <xacro:property name="sensor_name" value="os1" />
     <xacro:property name="lasers" value="16" />
     <xacro:property name="vfov_angle" value="33.2" />
     <xacro:property name="range" value="120" />
     <xacro:if value="${ouster_model == 'OS1-16'}">
-      <xacro:property name="sensor_name" value="os1" />
       <xacro:property name="lasers" value="16" />
       <xacro:property name="vfov_angle" value="33.2" />
@@ -649,5 +647,4 @@
     <!-- OS0-32 -->
     <xacro:if value="${ouster_model == 'OS0-32'}">
-      <xacro:property name="sensor_name" value="os0" />
       <xacro:property name="lasers" value="32" />
       <xacro:property name="vfov_angle" value="90" />
@@ -656,5 +653,4 @@
     <!-- OS0-64 -->
     <xacro:if value="${ouster_model == 'OS0-64'}">
-      <xacro:property name="sensor_name" value="os0" />
       <xacro:property name="lasers" value="64" />
       <xacro:property name="vfov_angle" value="90" />
@@ -663,5 +659,4 @@
     <!-- OS0-128 -->
     <xacro:if value="${ouster_model == 'OS0-128'}">
-      <xacro:property name="sensor_name" value="os0" />
       <xacro:property name="lasers" value="128" />
       <xacro:property name="vfov_angle" value="90" />
@@ -672,5 +667,4 @@
     <!-- OS1-32 Generation 2 -->
     <xacro:if value="${ouster_model == 'OS1-32'}">
-      <xacro:property name="sensor_name" value="os1" />
       <xacro:property name="lasers" value="32" />
       <xacro:property name="vfov_angle" value="45" />
@@ -679,5 +673,4 @@
     <!-- OS1-64 Generation 2 -->
     <xacro:if value="${ouster_model == 'OS1-64'}">
-      <xacro:property name="sensor_name" value="os1" />
       <xacro:property name="lasers" value="64" />
       <xacro:property name="vfov_angle" value="45" />
@@ -686,5 +679,4 @@
     <!-- OS1-128 Generation 2 -->
     <xacro:if value="${ouster_model == 'OS1-128'}">
-      <xacro:property name="sensor_name" value="os1" />
       <xacro:property name="lasers" value="128" />
       <xacro:property name="vfov_angle" value="45" />
@@ -695,5 +687,4 @@
     <!-- OS2-32 -->
     <xacro:if value="${ouster_model == 'OS2-32'}">
-      <xacro:property name="sensor_name" value="os2" />
       <xacro:property name="lasers" value="32" />
       <xacro:property name="vfov_angle" value="22.5" />
@@ -702,5 +693,4 @@
     <!-- OS2-64 -->
     <xacro:if value="${ouster_model == 'OS2-64'}">
-      <xacro:property name="sensor_name" value="os2" />
       <xacro:property name="lasers" value="64" />
       <xacro:property name="vfov_angle" value="22.5" />
@@ -709,5 +699,4 @@
     <!-- OS2-128 -->
     <xacro:if value="${ouster_model == 'OS2-128'}">
-      <xacro:property name="sensor_name" value="os2" />
       <xacro:property name="lasers" value="128" />
       <xacro:property name="vfov_angle" value="22.5" />
@@ -717,5 +706,5 @@
   <xacro:ouster_macro
     namespace="${namespace}"
-    sensor_name="${sensor_name}"
+    sensor_name="os"
     x="0"
     y="0"

File: models/mrs_robots_description/urdf/f550.xacro (robot description, xacro)
@@ -695,10 +695,8 @@
     <xacro:property name="ouster_model" value="${optionals['ouster_model']}" />
     <!-- OS1-16 Generation 1 (default) -->
-    <xacro:property name="sensor_name" value="os1" />
     <xacro:property name="lasers" value="16" />
     <xacro:property name="vfov_angle" value="33.2" />
     <xacro:property name="range" value="120" />
     <xacro:if value="${ouster_model == 'OS1-16'}">
-      <xacro:property name="sensor_name" value="os1" />
       <xacro:property name="lasers" value="16" />
       <xacro:property name="vfov_angle" value="33.2" />
@@ -708,5 +706,4 @@
     <!-- OS0-32 -->
     <xacro:if value="${ouster_model == 'OS0-32'}">
-      <xacro:property name="sensor_name" value="os0" />
       <xacro:property name="lasers" value="32" />
       <xacro:property name="vfov_angle" value="90" />
@@ -715,5 +712,4 @@
     <!-- OS0-64 -->
     <xacro:if value="${ouster_model == 'OS0-64'}">
-      <xacro:property name="sensor_name" value="os0" />
       <xacro:property name="lasers" value="64" />
       <xacro:property name="vfov_angle" value="90" />
@@ -722,5 +718,4 @@
     <!-- OS0-128 -->
     <xacro:if value="${ouster_model == 'OS0-128'}">
-      <xacro:property name="sensor_name" value="os0" />
       <xacro:property name="lasers" value="128" />
       <xacro:property name="vfov_angle" value="90" />
@@ -731,5 +726,4 @@
     <!-- OS1-32 Generation 2 -->
     <xacro:if value="${ouster_model == 'OS1-32'}">
-      <xacro:property name="sensor_name" value="os1" />
       <xacro:property name="lasers" value="32" />
       <xacro:property name="vfov_angle" value="45" />
@@ -738,5 +732,4 @@
     <!-- OS1-64 Generation 2 -->
     <xacro:if value="${ouster_model == 'OS1-64'}">
-      <xacro:property name="sensor_name" value="os1" />
       <xacro:property name="lasers" value="64" />
       <xacro:property name="vfov_angle" value="45" />
@@ -745,5 +738,4 @@
     <!-- OS1-128 Generation 2 -->
     <xacro:if value="${ouster_model == 'OS1-128'}">
-      <xacro:property name="sensor_name" value="os1" />
       <xacro:property name="lasers" value="128" />
       <xacro:property name="vfov_angle" value="45" />
@@ -754,5 +746,4 @@
     <!-- OS2-32 -->
     <xacro:if value="${ouster_model == 'OS2-32'}">
-      <xacro:property name="sensor_name" value="os2" />
       <xacro:property name="lasers" value="32" />
       <xacro:property name="vfov_angle" value="22.5" />
@@ -761,5 +752,4 @@
     <!-- OS2-64 -->
     <xacro:if value="${ouster_model == 'OS2-64'}">
-      <xacro:property name="sensor_name" value="os2" />
       <xacro:property name="lasers" value="64" />
       <xacro:property name="vfov_angle" value="22.5" />
@@ -768,5 +758,4 @@
     <!-- OS2-128 -->
     <xacro:if value="${ouster_model == 'OS2-128'}">
-      <xacro:property name="sensor_name" value="os2" />
       <xacro:property name="lasers" value="128" />
       <xacro:property name="vfov_angle" value="22.5" />
@@ -776,5 +765,5 @@
   <xacro:ouster_macro
     namespace="${namespace}"
-    sensor_name="${sensor_name}"
+    sensor_name="os"
     x="0"
     y="0"

File: models/mrs_robots_description/urdf/t650.xacro (robot description, xacro)
@@ -595,10 +595,8 @@
   <xacro:property name="ouster_model" value="${optionals['ouster_model']}" />
     <!-- OS1-16 Generation 1 (default) -->
-    <xacro:property name="sensor_name" value="os1" />
     <xacro:property name="lasers" value="16" />
     <xacro:property name="vfov_angle" value="33.2" />
     <xacro:property name="range" value="120" />
     <xacro:if value="${ouster_model == 'OS1-16'}">
-      <xacro:property name="sensor_name" value="os1" />
       <xacro:property name="lasers" value="16" />
       <xacro:property name="vfov_angle" value="33.2" />
@@ -607,5 +605,4 @@
     <!-- OS1-32 Generation 1 -->
     <xacro:if value="${ouster_model == 'OS1-32G1'}">
-      <xacro:property name="sensor_name" value="os1" />
       <xacro:property name="lasers" value="32" />
       <xacro:property name="vfov_angle" value="33.2" />
@@ -615,5 +612,4 @@
     <!-- OS0-32 -->
     <xacro:if value="${ouster_model == 'OS0-32'}">
-      <xacro:property name="sensor_name" value="os0" />
       <xacro:property name="lasers" value="32" />
       <xacro:property name="vfov_angle" value="90" />
@@ -622,5 +618,4 @@
     <!-- OS0-64 -->
     <xacro:if value="${ouster_model == 'OS0-64'}">
-      <xacro:property name="sensor_name" value="os0" />
       <xacro:property name="lasers" value="64" />
       <xacro:property name="vfov_angle" value="90" />
@@ -629,5 +624,4 @@
     <!-- OS0-128 -->
     <xacro:if value="${ouster_model == 'OS0-128'}">
-      <xacro:property name="sensor_name" value="os0" />
       <xacro:property name="lasers" value="128" />
       <xacro:property name="vfov_angle" value="90" />
@@ -638,5 +632,4 @@
     <!-- OS1-32 Generation 2 -->
     <xacro:if value="${ouster_model == 'OS1-32'}">
-      <xacro:property name="sensor_name" value="os1" />
       <xacro:property name="lasers" value="32" />
       <xacro:property name="vfov_angle" value="45" />
@@ -645,5 +638,4 @@
     <!-- OS1-64 Generation 2 -->
     <xacro:if value="${ouster_model == 'OS1-64'}">
-      <xacro:property name="sensor_name" value="os1" />
       <xacro:property name="lasers" value="64" />
       <xacro:property name="vfov_angle" value="45" />
@@ -652,5 +644,4 @@
     <!-- OS1-128 Generation 2 -->
     <xacro:if value="${ouster_model == 'OS1-128'}">
-      <xacro:property name="sensor_name" value="os1" />
       <xacro:property name="lasers" value="128" />
       <xacro:property name="vfov_angle" value="45" />
@@ -661,5 +652,4 @@
     <!-- OS2-32 -->
     <xacro:if value="${ouster_model == 'OS2-32'}">
-      <xacro:property name="sensor_name" value="os2" />
       <xacro:property name="lasers" value="32" />
       <xacro:property name="vfov_angle" value="22.5" />
@@ -668,5 +658,4 @@
     <!-- OS2-64 -->
     <xacro:if value="${ouster_model == 'OS2-64'}">
-      <xacro:property name="sensor_name" value="os2" />
       <xacro:property name="lasers" value="64" />
       <xacro:property name="vfov_angle" value="22.5" />
@@ -675,5 +664,4 @@
     <!-- OS2-128 -->
     <xacro:if value="${ouster_model == 'OS2-128'}">
-      <xacro:property name="sensor_name" value="os2" />
       <xacro:property name="lasers" value="128" />
       <xacro:property name="vfov_angle" value="22.5" />
@@ -683,5 +671,5 @@
   <xacro:ouster_macro
     namespace="${namespace}"
-    sensor_name="${sensor_name}"
+    sensor_name="os"
     x="0"
     y="0"

Commit message: Add tilt compensation param for servo camera and light

File: models/mrs_robots_description/urdf/component_snippets.xacro (robot description, xacro)
@@ -1936,5 +1936,5 @@
   <!--}-->
   <!-- Macro to add a camera mounted on virtual servo {-->
-  <xacro:macro name="servo_camera_macro" params="namespace name parent offset_x offset_y offset_z offset_yaw offset_roll offset_pitch update_rate max_pitch_rate camera_type">
+  <xacro:macro name="servo_camera_macro" params="namespace name parent offset_x offset_y offset_z offset_yaw offset_roll offset_pitch update_rate max_pitch_rate camera_type compensate_tilt">
       <joint name="${name}_joint" type="revolute">
           <parent link="${parent}"/>
@@ -1969,4 +1969,5 @@
           <joint_name>${name}_joint</joint_name>
           <camera_type>${camera_type}</camera_type>
+          <compensate_tilt>${compensate_tilt}</compensate_tilt>
         </plugin>
       </gazebo>
@@ -2314,5 +2315,5 @@
   <!--}-->
   <!-- Macro to add a light {-->
-  <xacro:macro name="light_macro" params="namespace name parent offset_x offset_y offset_z offset_yaw offset_roll offset_pitch update_rate max_pitch_rate initial_on ">
+  <xacro:macro name="light_macro" params="namespace name parent offset_x offset_y offset_z offset_yaw offset_roll offset_pitch update_rate max_pitch_rate initial_on compensate_tilt ">
       <joint name="${name}_joint" type="revolute">
           <parent link="${parent}"/>
@@ -2346,4 +2347,5 @@
           <max_pitch_rate>${max_pitch_rate}</max_pitch_rate>
           <initial_on>${initial_on}</initial_on>
+          <compensate_tilt>${compensate_tilt}</compensate_tilt>
         </plugin>
       </gazebo>

File: models/mrs_robots_description/urdf/f450.xacro (robot description, xacro)
@@ -987,5 +987,6 @@
       max_pitch_rate="0.1"
       camera_type="servo_camera"
-      update_rate="30.0">
+      update_rate="30.0"
+      compensate_tilt="true">
     </xacro:servo_camera_macro>
   </xacro:if>
@@ -1154,5 +1155,6 @@
       max_pitch_rate="0.1"
       initial_on="1"
-      update_rate="30.0">
+      update_rate="30.0"
+      compensate_tilt="true">
     </xacro:light_macro>
   </xacro:if>

File: models/mrs_robots_description/urdf/f550.xacro (robot description, xacro)
@@ -1043,5 +1043,6 @@
       max_pitch_rate="0.1"
       camera_type="servo_camera"
-      update_rate="30.0">
+      update_rate="30.0"
+      compensate_tilt="true">
     </xacro:servo_camera_macro>
   </xacro:if>
@@ -1153,5 +1154,6 @@
       max_pitch_rate="0.1"
       initial_on="1"
-      update_rate="30.0">
+      update_rate="30.0"
+      compensate_tilt="true">
     </xacro:light_macro>
   </xacro:if>

File: models/mrs_robots_description/urdf/t650.xacro (robot description, xacro)
@@ -900,5 +900,6 @@
       max_pitch_rate="0.1"
       camera_type="servo_camera"
-      update_rate="30.0">
+      update_rate="30.0"
+      compensate_tilt="true">
     </xacro:servo_camera_macro>
   </xacro:if>
@@ -1031,5 +1032,6 @@
       max_pitch_rate="0.1"
       initial_on="1"
-      update_rate="30.0">
+      update_rate="30.0"
+      compensate_tilt="true">
     </xacro:light_macro>
   </xacro:if>
