Commit message: added realsense_up_down parameter for 2 realsense cameras pointing up and down

File: models/mrs_robots_description/urdf/component_snippets.xacro (robot description, xacro)
@@ -1535,7 +1535,7 @@
   <!-- Macro to add an Intel Realsense D435 {-->
   <xacro:macro name="realsense_macro"
-    params="namespace parent_link parent_frame_name camera_suffix x y z roll pitch yaw enable_realistic_realsense">
+    params="namespace realsense_namespace parent_link parent_frame_name camera_suffix x y z roll pitch yaw enable_realistic_realsense">
     <!-- visual links and joints {-->
-    <link name="${namespace}/camera_${camera_suffix}">
+    <link name="${realsense_namespace}/camera_${camera_suffix}">
       <visual>
         <origin xyz="0.0 0.0 0" rpy="-${rad90} 0 -${rad90}" />
@@ -1546,5 +1546,5 @@
       </visual>
     </link>
-    <link name="${namespace}/camera_${camera_suffix}_glass_link">
+    <link name="${realsense_namespace}/camera_${camera_suffix}_glass_link">
       <visual>
         <origin xyz="0.0 0.0 0" rpy="-${rad90} 0 -${rad90}" />
@@ -1555,17 +1555,18 @@
       </visual>
     </link>
-    <joint name="${namespace}/camera_${camera_suffix}_joint" type="fixed">
+    <joint name="${realsense_namespace}/camera_${camera_suffix}_joint" type="fixed">
       <origin xyz="${x} ${y} ${z}" rpy="${roll} ${pitch} ${yaw}"/>
       <parent link="${parent_link}" />
-      <child link="${namespace}/camera_${camera_suffix}" />
-    </joint>
-    <joint name="${namespace}/camera_${camera_suffix}_glass_joint" type="fixed">
+      <child link="${realsense_namespace}/camera_${camera_suffix}" />
+    </joint>
+    <joint name="${realsense_namespace}/camera_${camera_suffix}_glass_joint" type="fixed">
       <origin xyz="0 0 0 " rpy="0 0 0"/>
-      <parent link="${namespace}/camera_${camera_suffix}" />
-      <child link="${namespace}/camera_${camera_suffix}_glass_link" />
+      <parent link="${realsense_namespace}/camera_${camera_suffix}" />
+      <child link="${realsense_namespace}/camera_${camera_suffix}_glass_link" />
     </joint>
     <!--}-->
     <gazebo>
       <plugin name="${camera_suffix}_plugin" filename="libMRSGazeboRealsensePlugin.so">
+        <realsense_namespace>${realsense_namespace}</realsense_namespace>
         <useRealistic>${enable_realistic_realsense}</useRealistic>
         <noisePerMeter>0.2</noisePerMeter>
@@ -1586,10 +1587,10 @@
     </gazebo>
     <!-- sensors {-->
-    <gazebo reference="${namespace}/camera_${camera_suffix}">
+    <gazebo reference="${realsense_namespace}/camera_${camera_suffix}">
       <!-- rgb camera {-->
-      <sensor name="${namespace}/color" type="camera">
+      <sensor name="${namespace}/${realsense_namespace}/color" type="camera">
         <!-- <pose frame="">0 -0.046 0.004 0 0 0</pose> -->
         <pose frame="">0 0 -0.0115 0 0 0</pose>
-        <camera name="${namespace}/camera_${camera_suffix}">
+        <camera name="${realsense_namespace}/camera_${camera_suffix}">
           <!-- <horizontal_fov>1.211259</horizontal_fov> -->
           <horizontal_fov>1.211259</horizontal_fov>
@@ -1615,9 +1616,9 @@
       <!--}-->
       <!-- infra stereo {-->
-      <sensor name="${namespace}/infra_stereo" type="multicamera">
+      <sensor name="${namespace}/${realsense_namespace}/infra_stereo" type="multicamera">
         <always_on>1</always_on>
         <update_rate>30</update_rate>
         <visualize>0</visualize>
-        <camera name="${namespace}/infra1">
+        <camera name="${namespace}/${realsense_namespace}/infra1">
           <!-- <horizontal_fov>1.7523106</horizontal_fov> -->
           <horizontal_fov>1.211259</horizontal_fov>
@@ -1637,5 +1638,5 @@
           </noise>
         </camera>
-        <camera name="${namespace}/infra2">
+        <camera name="${namespace}/${realsense_namespace}/infra2">
           <pose>0 0.05 0 0 0 0</pose>
           <!-- <horizontal_fov>1.7523106</horizontal_fov> -->
@@ -1660,8 +1661,8 @@
       <!-- (unused) infra2 {-->
         <!-- <sensor name="infra2" type="camera"> -->
-        <!-- <parent link="${namespace}/camera_${camera_suffix}"/> -->
+        <!-- <parent link="${realsense_namespace}/camera_${camera_suffix}"/> -->
         <!-- <pose>0 -1.0325 0 0 0 0</pose> -->
-        <!--   <pose frame="${namespace}/camera_${camera_suffix}_infra2">0 -1.0325 0 0 0 0</pose> -->
-        <!--   <camera name="${namespace}/camera_${camera_suffix}_infra2"> -->
+        <!--   <pose frame="${realsense_namespace}/camera_${camera_suffix}_infra2">0 -1.0325 0 0 0 0</pose> -->
+        <!--   <camera name="${realsense_namespace}/camera_${camera_suffix}_infra2"> -->
           <!-- <horizontal_fov>1.7523106</horizontal_fov> -->
           <!--     <horizontal_fov>1.211259</horizontal_fov> -->
@@ -1687,7 +1688,7 @@
           <!--}-->
       <!-- aligned depth to color {-->
-      <sensor name="${namespace}/aligned_depth_to_color" type="depth">
+        <sensor name="${namespace}/${realsense_namespace}/aligned_depth_to_color" type="depth">
         <pose>0 -0.0115 0.0 0 0 0</pose>
-        <camera name="${namespace}/camera_${camera_suffix}">
+        <camera name="${realsense_namespace}/camera_${camera_suffix}">
           <horizontal_fov>1.211259</horizontal_fov>
           <image>
@@ -1718,8 +1719,8 @@
     </gazebo>
     <!--}-->
-    <gazebo reference="${namespace}/camera_${camera_suffix}">
+    <gazebo reference="${realsense_namespace}/camera_${camera_suffix}">
       <material>Gazebo/White</material>
     </gazebo>
-    <gazebo reference="${namespace}/camera_${camera_suffix}_glass_link">
+    <gazebo reference="${realsense_namespace}/camera_${camera_suffix}_glass_link">
       <material>Gazebo/BlackTransparent</material>
     </gazebo>

File: models/mrs_robots_description/urdf/f450.xacro (robot description, xacro)
@@ -799,4 +799,5 @@
     <xacro:realsense_macro
       namespace="${namespace}"
+      realsense_namespace=""
       parent_link="base_link"
       camera_suffix="realsense_down"
@@ -817,4 +818,5 @@
     <xacro:realsense_macro
       namespace="${namespace}"
+      realsense_namespace=""
       parent_link="base_link"
       camera_suffix="realsense_front_pitched"
@@ -835,4 +837,5 @@
     <xacro:realsense_macro
       namespace="${namespace}"
+      realsense_namespace=""
       parent_link="base_link"
       camera_suffix="realsense_front"
@@ -853,4 +856,5 @@
     <xacro:realsense_macro
       namespace="${namespace}"
+      realsense_namespace=""
       parent_link="base_link"
       camera_suffix="realsense_up"
@@ -862,4 +866,38 @@
       roll="0"
       pitch="-${rad90}"
+      yaw="0">
+    </xacro:realsense_macro>
+  </xacro:if>
+  <!--}-->
+  <!-- up_down {-->
+  <xacro:if value="${optionals['enable_realsense_up_down']}">
+    <!-- sensor -->
+    <xacro:realsense_macro
+      namespace="${namespace}"
+      realsense_namespace="up_rgbd"
+      parent_link="base_link"
+      camera_suffix="realsense_up"
+      parent_frame_name="${namespace}/fcu"
+      enable_realistic_realsense="${optionals['use_realistic_realsense']}"
+      x="-0.01"
+      y="-0.07"
+      z="0.05"
+      roll="0"
+      pitch="-${rad90}"
+      yaw="${rad90}">
+    </xacro:realsense_macro>
+    <!-- sensor -->
+    <xacro:realsense_macro
+      namespace="${namespace}"
+      realsense_namespace="down_rgbd"
+      parent_link="base_link"
+      camera_suffix="realsense_down"
+      parent_frame_name="${namespace}/fcu"
+      enable_realistic_realsense="${optionals['use_realistic_realsense']}"
+      x="0.12"
+      y="0"
+      z="-0.05"
+      roll="0"
+      pitch="+${rad90}"
       yaw="0">
     </xacro:realsense_macro>

File: models/mrs_robots_description/urdf/f550.xacro (robot description, xacro)
@@ -835,4 +835,5 @@
     <xacro:realsense_macro
       namespace="${namespace}"
+      realsense_namespace=""
       parent_link="base_link"
       camera_suffix="realsense_top"
@@ -852,4 +853,5 @@
     <xacro:realsense_macro
       namespace="${namespace}"
+      realsense_namespace=""
       parent_link="base_link"
       camera_suffix="realsense_down"
@@ -870,4 +872,5 @@
     <xacro:realsense_macro
       namespace="${namespace}"
+      realsense_namespace=""
       parent_link="base_link"
       camera_suffix="realsense_front_pitched"
@@ -891,4 +894,5 @@
     <xacro:realsense_macro
       namespace="${namespace}"
+      realsense_namespace=""
       parent_link="base_link"
       camera_suffix="realsense_front"
@@ -909,4 +913,5 @@
     <xacro:realsense_macro
       namespace="${namespace}"
+      realsense_namespace=""
       parent_link="base_link"
       camera_suffix="realsense_up"
@@ -918,4 +923,38 @@
       roll="0"
       pitch="-${rad90}"
+      yaw="0">
+    </xacro:realsense_macro>
+  </xacro:if>
+  <!--}-->
+  <!-- up_down {-->
+  <xacro:if value="${optionals['enable_realsense_up_down']}">
+    <!-- sensor -->
+    <xacro:realsense_macro
+      namespace="${namespace}"
+      realsense_namespace="up_rgbd"
+      parent_link="base_link"
+      camera_suffix="realsense_up"
+      parent_frame_name="${namespace}/fcu"
+      enable_realistic_realsense="${optionals['use_realistic_realsense']}"
+      x="-0.01"
+      y="-0.07"
+      z="0.05"
+      roll="0"
+      pitch="-${rad90}"
+      yaw="${rad90}">
+    </xacro:realsense_macro>
+    <!-- sensor -->
+    <xacro:realsense_macro
+      namespace="${namespace}"
+      realsense_namespace="down_rgbd"
+      parent_link="base_link"
+      camera_suffix="realsense_down"
+      parent_frame_name="${namespace}/fcu"
+      enable_realistic_realsense="${optionals['use_realistic_realsense']}"
+      x="0.12"
+      y="0"
+      z="-0.05"
+      roll="0"
+      pitch="+${rad90}"
       yaw="0">
     </xacro:realsense_macro>

File: models/mrs_robots_description/urdf/t650.xacro (robot description, xacro)
@@ -741,4 +741,5 @@
     <xacro:realsense_macro
       namespace="${namespace}"
+      realsense_namespace=""
       parent_link="base_link"
       camera_suffix="realsense_front"
@@ -759,4 +760,5 @@
     <xacro:realsense_macro
       namespace="${namespace}"
+      realsense_namespace=""
       parent_link="base_link"
       camera_suffix="realsense_up"
@@ -768,4 +770,57 @@
       roll="0"
       pitch="-${rad90}"
+      yaw="0">
+    </xacro:realsense_macro>
+  </xacro:if>
+  <!--}-->
+  <!-- down {-->
+  <xacro:if value="${optionals['enable_realsense_down']}">
+    <!-- sensor -->
+    <xacro:realsense_macro
+      namespace="${namespace}"
+      realsense_namespace=""
+      parent_link="base_link"
+      camera_suffix="realsense_down"
+      parent_frame_name="${namespace}/fcu"
+      enable_realistic_realsense="${optionals['use_realistic_realsense']}"
+      x="0.1"
+      y="0"
+      z="-0.05"
+      roll="0"
+      pitch="+${rad90}"
+      yaw="0">
+    </xacro:realsense_macro>
+  </xacro:if>
+  <!--}-->
+  <!-- up_down {-->
+  <xacro:if value="${optionals['enable_realsense_up_down']}">
+    <!-- sensor -->
+    <xacro:realsense_macro
+      namespace="${namespace}"
+      realsense_namespace="up_rgbd"
+      parent_link="base_link"
+      camera_suffix="realsense_up"
+      parent_frame_name="${namespace}/fcu"
+      enable_realistic_realsense="${optionals['use_realistic_realsense']}"
+      x="-0.01"
+      y="-0.07"
+      z="0.05"
+      roll="0"
+      pitch="-${rad90}"
+      yaw="${rad90}">
+    </xacro:realsense_macro>
+    <!-- sensor -->
+    <xacro:realsense_macro
+      namespace="${namespace}"
+      realsense_namespace="down_rgbd"
+      parent_link="base_link"
+      camera_suffix="realsense_down"
+      parent_frame_name="${namespace}/fcu"
+      enable_realistic_realsense="${optionals['use_realistic_realsense']}"
+      x="0.12"
+      y="0"
+      z="-0.05"
+      roll="0"
+      pitch="+${rad90}"
       yaw="0">
     </xacro:realsense_macro>

Commit message: add rad120 to component_snippets.xacro

File: models/mrs_robots_description/urdf/component_snippets.xacro (robot description, xacro)
@@ -38,4 +38,5 @@
   <xacro:property name="rad95" value="${95*pi/180}" />
   <xacro:property name="rad115" value="${115*pi/180}" />
+  <xacro:property name="rad120" value="${120*pi/180}" />
   <xacro:property name="rad135" value="${135*pi/180}" />
   <xacro:property name="rad150" value="${150*pi/180}" />

Commit message: added ground truth plugin to all uavs, added custom mag plugin

File: models/mrs_robots_description/urdf/component_snippets.xacro (robot description, xacro)
@@ -462,5 +462,5 @@
   <xacro:macro name="magnetometer_plugin_macro" params="namespace pub_rate noise_density random_walk bias_correlation_time mag_topic">
     <gazebo>
-      <plugin name="magnetometer_plugin" filename="libgazebo_magnetometer_plugin.so">
+      <plugin name="magnetometer_plugin" filename="libMRSGazeboMagnetometerPlugin.so">
         <robotNamespace>${namespace}</robotNamespace>
         <pubRate>${pub_rate}</pubRate>
@@ -469,4 +469,16 @@
         <biasCorrelationTime>${bias_correlation_time}</biasCorrelationTime>
         <magTopic>${mag_topic}</magTopic>
+      </plugin>
+    </gazebo>
+  </xacro:macro>
+  <!--}-->
+  <!-- Macro to add the groundtruth_plugin{-->
+  <xacro:macro name="groundtruth_plugin_macro" params="namespace home_latitude home_longitude home_altitude">
+    <gazebo>
+      <plugin name="groundtruth_plugin" filename="libgazebo_groundtruth_plugin.so">
+        <robotNamespace>${namespace}</robotNamespace>
+        <homeLatitude>${home_latitude}</homeLatitude>
+        <homeLongitude>${home_longitude}</homeLongitude>
+        <homeAltitude>${home_altitude}</homeAltitude>
       </plugin>
     </gazebo>

File: models/mrs_robots_description/urdf/f330.xacro (robot description, xacro)
@@ -477,5 +477,14 @@
   </xacro:magnetometer_plugin_macro>
   <!--}-->
-  <!-- Barometer {-->
+   <!-- Groundtruth {-->
+  <xacro:groundtruth_plugin_macro
+    namespace="${namespace}"
+    home_latitude="0.0"
+    home_longitude="0.0"
+    home_altitude="0.0"
+    >
+  </xacro:groundtruth_plugin_macro>
+  <!--}-->
+ <!-- Barometer {-->
   <xacro:barometer_plugin_macro
   namespace="${namespace}"

File: models/mrs_robots_description/urdf/f450.xacro (robot description, xacro)
@@ -478,5 +478,14 @@
   </xacro:magnetometer_plugin_macro>
   <!--}-->
-  <!-- Barometer {-->
+   <!-- Groundtruth {-->
+  <xacro:groundtruth_plugin_macro
+    namespace="${namespace}"
+    home_latitude="0.0"
+    home_longitude="0.0"
+    home_altitude="0.0"
+    >
+  </xacro:groundtruth_plugin_macro>
+  <!--}-->
+ <!-- Barometer {-->
   <xacro:barometer_plugin_macro
   namespace="${namespace}"

File: models/mrs_robots_description/urdf/f550.xacro (robot description, xacro)
@@ -536,4 +536,13 @@
     >
   </xacro:magnetometer_plugin_macro>
+  <!--}-->
+   <!-- Groundtruth {-->
+  <xacro:groundtruth_plugin_macro
+    namespace="${namespace}"
+    home_latitude="0.0"
+    home_longitude="0.0"
+    home_altitude="0.0"
+    >
+  </xacro:groundtruth_plugin_macro>
   <!--}-->
   <!-- Barometer {-->

File: models/mrs_robots_description/urdf/t650.xacro (robot description, xacro)
@@ -452,4 +452,13 @@
     >
   </xacro:magnetometer_plugin_macro>
+  <!--}-->
+  <!-- Groundtruth {-->
+  <xacro:groundtruth_plugin_macro
+    namespace="${namespace}"
+    home_latitude="0.0"
+    home_longitude="0.0"
+    home_altitude="0.0"
+    >
+  </xacro:groundtruth_plugin_macro>
   <!--}-->
   <!-- Barometer {-->

File: models/mrs_robots_description/urdf/x500.xacro (robot description, xacro)
@@ -481,4 +481,13 @@
   </xacro:magnetometer_plugin_macro>
   <!--}-->
+   <!-- Groundtruth {-->
+  <xacro:groundtruth_plugin_macro
+    namespace="${namespace}"
+    home_latitude="0.0"
+    home_longitude="0.0"
+    home_altitude="0.0"
+    >
+  </xacro:groundtruth_plugin_macro>
+  <!--}-->
   <!-- Barometer {-->
   <xacro:barometer_plugin_macro

Commit message: add timepix3 sensor to x500 and t650

File: models/mrs_robots_description/urdf/component_snippets.xacro (robot description, xacro)
@@ -2278,4 +2278,32 @@
   </xacro:macro>
   <!--}-->
+  <!-- Macro to add a Timepix3 event camera {-->
+  <xacro:macro name="timepix3_macro" params="namespace name parent color material thickness max_message_window sensor_suffix *origin">
+    <joint name="${name}_joint" type="fixed">
+      <xacro:insert_block name="origin" />
+      <parent link="${parent}" />
+      <child link="${name}_link" />
+    </joint>
+    <link name="${name}_link">
+      <visual>
+        <origin xyz="0 0.05 0" rpy="0 0 0" />
+        <geometry>
+          <box size="0.02 0.09 0.02" />
+        </geometry>
+      </visual>
+    </link>
+    <gazebo reference="${name}_link">
+      <material>Gazebo/${color}</material>
+    </gazebo>
+    <gazebo>
+      <plugin name="gazebo_timepix3" filename="libgazebo_timepix3.so" >
+        <material>${material}</material>                 <!-- string -->
+        <size>${thickness} 0.01408 0.01408</size>     <!-- [m m m] -->
+        <max_message_window>${max_message_window}</max_message_window> <!-- [s] -->
+        <sensor_suffix>${sensor_suffix}</sensor_suffix> <!-- [s] -->
+      </plugin>
+    </gazebo>
+  </xacro:macro>
+  <!--}-->
   <!-- Macro to add a water gun {-->
   <xacro:macro name="water_gun_macro" params="namespace name parent muzzle_velocity particle_capacity spread spawning_reservoir offset_x offset_y offset_z size_x size_y size_z *origin">

File: models/mrs_robots_description/urdf/t650.xacro (robot description, xacro)
@@ -1004,4 +1004,19 @@
   </xacro:if>
   <!--}-->
+  <!-- Timepix3 {-->
+  <xacro:if value="${optionals['enable_timepix3']}">
+    <xacro:timepix3_macro
+      namespace="${namespace}"
+      name="timepix3"
+      parent="base_link"
+      color="Green"
+      material="cdte"
+      thickness="0.002"
+      max_message_window="1.0"
+      sensor_suffix="">
+      <origin xyz="0.115 -0.05 -0.05" rpy="0 0 0" />
+    </xacro:timepix3_macro>
+  </xacro:if>
+  <!--}-->
 <!-- Water gun {-->
 <xacro:if value="${optionals['enable_water_gun']}">

File: models/mrs_robots_description/urdf/x500.xacro (robot description, xacro)
@@ -472,4 +472,19 @@
   </xacro:gps_macro>
   <!--}-->
+  <!-- Timepix3 {-->
+  <xacro:if value="${optionals['enable_timepix3']}">
+    <xacro:timepix3_macro
+      namespace="${namespace}"
+      name="timepix3"
+      parent="base_link"
+      color="Green"
+      material="cdte"
+      thickness="0.002"
+      max_message_window="1.0"
+      sensor_suffix="">
+      <origin xyz="0.115 -0.05 -0.05" rpy="0 0 0" />
+    </xacro:timepix3_macro>
+  </xacro:if>
+  <!--}-->
   <!-- Magnetometer {-->
   <xacro:magnetometer_plugin_macro

Commit message: rotated vio IMU to correspond with the real drone

File: models/mrs_robots_description/urdf/component_snippets.xacro (robot description, xacro)
@@ -2018,5 +2018,5 @@
       noise_mean="${imu_noise_mean}"
       >
-      <origin xyz="0 0 0" rpy="${-rad90} 0 0"/>
+      <origin xyz="0 0 0" rpy="${-rad90} 0 ${-rad90}"/>
     </xacro:custom_imu_macro>
   </xacro:macro>
