Commit message: new realsense loading, fixed multiple instances

File: models/mrs_robots_description/urdf/component_snippets.xacro (robot description, xacro)
@@ -1548,7 +1548,7 @@
   <!-- Macro to add an Intel Realsense D435 {-->
   <xacro:macro name="realsense_macro"
-    params="namespace realsense_namespace parent_link parent_frame_name camera_suffix x y z roll pitch yaw enable_realistic_realsense">
+    params="namespace camera_name parent_link parent_frame_name camera_suffix x y z roll pitch yaw enable_realistic_realsense">
     <!-- visual links and joints {-->
-    <link name="${realsense_namespace}/camera_${camera_suffix}">
+    <link name="${camera_name}/camera${camera_suffix}">
       <visual>
         <origin xyz="0.0 0.0 0" rpy="-${rad90} 0 -${rad90}" />
@@ -1559,5 +1559,5 @@
       </visual>
     </link>
-    <link name="${realsense_namespace}/camera_${camera_suffix}_glass_link">
+    <link name="${camera_name}/camera${camera_suffix}_glass_link">
       <visual>
         <origin xyz="0.0 0.0 0" rpy="-${rad90} 0 -${rad90}" />
@@ -1568,18 +1568,19 @@
       </visual>
     </link>
-    <joint name="${realsense_namespace}/camera_${camera_suffix}_joint" type="fixed">
+    <joint name="${camera_name}/camera${camera_suffix}_joint" type="fixed">
       <origin xyz="${x} ${y} ${z}" rpy="${roll} ${pitch} ${yaw}"/>
       <parent link="${parent_link}" />
-      <child link="${realsense_namespace}/camera_${camera_suffix}" />
-    </joint>
-    <joint name="${realsense_namespace}/camera_${camera_suffix}_glass_joint" type="fixed">
+      <child link="${camera_name}/camera${camera_suffix}" />
+    </joint>
+    <joint name="${camera_name}/camera${camera_suffix}_glass_joint" type="fixed">
       <origin xyz="0 0 0 " rpy="0 0 0"/>
-      <parent link="${realsense_namespace}/camera_${camera_suffix}" />
-      <child link="${realsense_namespace}/camera_${camera_suffix}_glass_link" />
+      <parent link="${camera_name}/camera${camera_suffix}" />
+      <child link="${camera_name}/camera${camera_suffix}_glass_link" />
     </joint>
     <!--}-->
     <gazebo>
-      <plugin name="${camera_suffix}_plugin" filename="libMRSGazeboRealsensePlugin.so">
-        <realsense_namespace>${realsense_namespace}</realsense_namespace>
+      <plugin name="${camera_name}${camera_suffix}_plugin" filename="libMRSGazeboRealsensePlugin.so">
+        <camera_name>${camera_name}</camera_name>
+        <camera_suffix>${camera_suffix}</camera_suffix>
         <useRealistic>${enable_realistic_realsense}</useRealistic>
         <noisePerMeter>0.2</noisePerMeter>
@@ -1600,10 +1601,10 @@
     </gazebo>
     <!-- sensors {-->
-    <gazebo reference="${realsense_namespace}/camera_${camera_suffix}">
+    <gazebo reference="${camera_name}/camera${camera_suffix}">
       <!-- rgb camera {-->
-      <sensor name="${namespace}/${realsense_namespace}/color" type="camera">
+      <sensor name="${namespace}/${camera_name}${camera_suffix}_color" type="camera">
         <!-- <pose frame="">0 -0.046 0.004 0 0 0</pose> -->
         <pose frame="">0 0 -0.0115 0 0 0</pose>
-        <camera name="${realsense_namespace}/camera_${camera_suffix}">
+        <camera name="${camera_name}${camera_suffix}/camera">
           <!-- <horizontal_fov>1.211259</horizontal_fov> -->
           <horizontal_fov>1.211259</horizontal_fov>
@@ -1629,9 +1630,9 @@
       <!--}-->
       <!-- infra stereo {-->
-      <sensor name="${namespace}/${realsense_namespace}/infra_stereo" type="multicamera">
+      <sensor name="${namespace}/${camera_name}${camera_suffix}_infra_stereo" type="multicamera">
         <always_on>1</always_on>
         <update_rate>30</update_rate>
         <visualize>0</visualize>
-        <camera name="${namespace}/${realsense_namespace}/infra1">
+        <camera name="${namespace}/${camera_name}${camera_suffix}/infra1">
           <!-- <horizontal_fov>1.7523106</horizontal_fov> -->
           <horizontal_fov>1.211259</horizontal_fov>
@@ -1651,5 +1652,5 @@
           </noise>
         </camera>
-        <camera name="${namespace}/${realsense_namespace}/infra2">
+        <camera name="${namespace}/${camera_name}${camera_suffix}/infra2">
           <pose>0 0.05 0 0 0 0</pose>
           <!-- <horizontal_fov>1.7523106</horizontal_fov> -->
@@ -1674,8 +1675,8 @@
       <!-- (unused) infra2 {-->
         <!-- <sensor name="infra2" type="camera"> -->
-        <!-- <parent link="${realsense_namespace}/camera_${camera_suffix}"/> -->
+        <!-- <parent link="${camera_name}${camera_suffix}_camera_${camera_suffix}"/> -->
         <!-- <pose>0 -1.0325 0 0 0 0</pose> -->
-        <!--   <pose frame="${realsense_namespace}/camera_${camera_suffix}_infra2">0 -1.0325 0 0 0 0</pose> -->
-        <!--   <camera name="${realsense_namespace}/camera_${camera_suffix}_infra2"> -->
+        <!--   <pose frame="${camera_name}${camera_suffix}/camera_infra2">0 -1.0325 0 0 0 0</pose> -->
+        <!--   <camera name="${camera_name}${camera_suffix}/camera_${camera_suffix}_infra2"> -->
           <!-- <horizontal_fov>1.7523106</horizontal_fov> -->
           <!--     <horizontal_fov>1.211259</horizontal_fov> -->
@@ -1701,7 +1702,7 @@
           <!--}-->
       <!-- aligned depth to color {-->
-        <sensor name="${namespace}/${realsense_namespace}/aligned_depth_to_color" type="depth">
+        <sensor name="${namespace}/${camera_name}${camera_suffix}_aligned_depth_to_color" type="depth">
         <pose>0 -0.0115 0.0 0 0 0</pose>
-        <camera name="${realsense_namespace}/camera_${camera_suffix}">
+        <camera name="${camera_name}/camera${camera_suffix}">
           <horizontal_fov>1.211259</horizontal_fov>
           <image>
@@ -1732,8 +1733,8 @@
     </gazebo>
     <!--}-->
-    <gazebo reference="${realsense_namespace}/camera_${camera_suffix}">
+    <gazebo reference="${camera_name}/camera${camera_suffix}">
       <material>Gazebo/White</material>
     </gazebo>
-    <gazebo reference="${realsense_namespace}/camera_${camera_suffix}_glass_link">
+    <gazebo reference="${camera_name}/camera${camera_suffix}_glass_link">
       <material>Gazebo/BlackTransparent</material>
     </gazebo>

File: models/mrs_robots_description/urdf/f330.xacro (robot description, xacro)
@@ -544,7 +544,7 @@
     <xacro:realsense_macro
       namespace="${namespace}"
-      realsense_namespace=""
+      camera_name="rgbd"
+      camera_suffix=""
       parent_link="base_link"
-      camera_suffix="realsense_front"
       parent_frame_name="${namespace}/fcu"
       enable_realistic_realsense="${optionals['use_realistic_realsense']}"

File: models/mrs_robots_description/urdf/f450.xacro (robot description, xacro)
@@ -808,7 +808,7 @@
     <xacro:realsense_macro
       namespace="${namespace}"
-      realsense_namespace=""
-      parent_link="base_link"
-      camera_suffix="realsense_down"
+      camera_name="rgbd"
+      camera_suffix="_down"
+      parent_link="base_link"
       parent_frame_name="${namespace}/fcu"
       enable_realistic_realsense="${optionals['use_realistic_realsense']}"
@@ -827,7 +827,7 @@
     <xacro:realsense_macro
       namespace="${namespace}"
-      realsense_namespace=""
-      parent_link="base_link"
-      camera_suffix="realsense_front_pitched"
+      camera_name="rgbd"
+      camera_suffix="_front_pitched"
+      parent_link="base_link"
       parent_frame_name="${namespace}/fcu"
       enable_realistic_realsense="${optionals['use_realistic_realsense']}"
@@ -846,7 +846,7 @@
     <xacro:realsense_macro
       namespace="${namespace}"
-      realsense_namespace=""
-      parent_link="base_link"
-      camera_suffix="realsense_front"
+      camera_name="rgbd"
+      camera_suffix=""
+      parent_link="base_link"
       parent_frame_name="${namespace}/fcu"
       enable_realistic_realsense="${optionals['use_realistic_realsense']}"
@@ -865,7 +865,7 @@
     <xacro:realsense_macro
       namespace="${namespace}"
-      realsense_namespace=""
-      parent_link="base_link"
-      camera_suffix="realsense_up"
+      camera_name="rgbd"
+      camera_suffix="_up"
+      parent_link="base_link"
       parent_frame_name="${namespace}/fcu"
       enable_realistic_realsense="${optionals['use_realistic_realsense']}"
@@ -875,38 +875,4 @@
       roll="0"
       pitch="-${rad90}"
-      yaw="0">
-    </xacro:realsense_macro>
-  </xacro:if>
-  <!--}-->
-  <!-- up_down {-->
-  <xacro:if value="${optionals['enable_realsense_up_down']}">
-    <!-- sensor -->
-    <xacro:realsense_macro
-      namespace="${namespace}"
-      realsense_namespace="up_rgbd"
-      parent_link="base_link"
-      camera_suffix="realsense_up"
-      parent_frame_name="${namespace}/fcu"
-      enable_realistic_realsense="${optionals['use_realistic_realsense']}"
-      x="-0.01"
-      y="-0.07"
-      z="0.05"
-      roll="0"
-      pitch="-${rad90}"
-      yaw="${rad90}">
-    </xacro:realsense_macro>
-    <!-- sensor -->
-    <xacro:realsense_macro
-      namespace="${namespace}"
-      realsense_namespace="down_rgbd"
-      parent_link="base_link"
-      camera_suffix="realsense_down"
-      parent_frame_name="${namespace}/fcu"
-      enable_realistic_realsense="${optionals['use_realistic_realsense']}"
-      x="0.12"
-      y="0"
-      z="-0.05"
-      roll="0"
-      pitch="+${rad90}"
       yaw="0">
     </xacro:realsense_macro>
@@ -1307,5 +1273,5 @@
     <xacro:visual_macro
       robot_namespace="${namespace}"
-      name="realsense_front_mount"
+      name="realsense_down_mount"
       mesh_file="${realsense_front_down_mount_mesh}"
       mesh_scale="${mesh_scale_milimeters}"

File: models/mrs_robots_description/urdf/f550.xacro (robot description, xacro)
@@ -844,7 +844,7 @@
     <xacro:realsense_macro
       namespace="${namespace}"
-      realsense_namespace=""
-      parent_link="base_link"
-      camera_suffix="realsense_top"
+      camera_name="rgbd"
+      camera_suffix="_top"
+      parent_link="base_link"
       parent_frame_name="${namespace}/fcu"
       enable_realistic_realsense="${optionals['use_realistic_realsense']}"
@@ -862,7 +862,7 @@
     <xacro:realsense_macro
       namespace="${namespace}"
-      realsense_namespace=""
-      parent_link="base_link"
-      camera_suffix="realsense_down"
+      camera_name="rgbd"
+      camera_suffix="_down"
+      parent_link="base_link"
       parent_frame_name="${namespace}/fcu"
       enable_realistic_realsense="${optionals['use_realistic_realsense']}"
@@ -881,7 +881,7 @@
     <xacro:realsense_macro
       namespace="${namespace}"
-      realsense_namespace=""
-      parent_link="base_link"
-      camera_suffix="realsense_front_pitched"
+      camera_name="rgbd"
+      camera_suffix="_front_pitched"
+      parent_link="base_link"
       parent_frame_name="${namespace}/fcu"
       enable_realistic_realsense="${optionals['use_realistic_realsense']}"
@@ -903,7 +903,7 @@
     <xacro:realsense_macro
       namespace="${namespace}"
-      realsense_namespace=""
-      parent_link="base_link"
-      camera_suffix="realsense_front"
+      camera_name="rgbd"
+      camera_suffix=""
+      parent_link="base_link"
       parent_frame_name="${namespace}/fcu"
       enable_realistic_realsense="${optionals['use_realistic_realsense']}"
@@ -922,7 +922,7 @@
     <xacro:realsense_macro
       namespace="${namespace}"
-      realsense_namespace=""
-      parent_link="base_link"
-      camera_suffix="realsense_up"
+      camera_name="rgbd"
+      camera_suffix="_up"
+      parent_link="base_link"
       parent_frame_name="${namespace}/fcu"
       enable_realistic_realsense="${optionals['use_realistic_realsense']}"
@@ -932,38 +932,4 @@
       roll="0"
       pitch="-${rad90}"
-      yaw="0">
-    </xacro:realsense_macro>
-  </xacro:if>
-  <!--}-->
-  <!-- up_down {-->
-  <xacro:if value="${optionals['enable_realsense_up_down']}">
-    <!-- sensor -->
-    <xacro:realsense_macro
-      namespace="${namespace}"
-      realsense_namespace="up_rgbd"
-      parent_link="base_link"
-      camera_suffix="realsense_up"
-      parent_frame_name="${namespace}/fcu"
-      enable_realistic_realsense="${optionals['use_realistic_realsense']}"
-      x="-0.01"
-      y="-0.07"
-      z="0.05"
-      roll="0"
-      pitch="-${rad90}"
-      yaw="${rad90}">
-    </xacro:realsense_macro>
-    <!-- sensor -->
-    <xacro:realsense_macro
-      namespace="${namespace}"
-      realsense_namespace="down_rgbd"
-      parent_link="base_link"
-      camera_suffix="realsense_down"
-      parent_frame_name="${namespace}/fcu"
-      enable_realistic_realsense="${optionals['use_realistic_realsense']}"
-      x="0.12"
-      y="0"
-      z="-0.05"
-      roll="0"
-      pitch="+${rad90}"
       yaw="0">
     </xacro:realsense_macro>
@@ -1280,5 +1246,5 @@
     <xacro:visual_macro
       robot_namespace="${namespace}"
-      name="realsense_front_mount"
+      name="realsense_down_mount"
       mesh_file="${realsense_front_down_mount_mesh}"
       mesh_scale="${mesh_scale_milimeters}"

File: models/mrs_robots_description/urdf/t650.xacro (robot description, xacro)
@@ -750,7 +750,7 @@
     <xacro:realsense_macro
       namespace="${namespace}"
-      realsense_namespace=""
-      parent_link="base_link"
-      camera_suffix="realsense_front"
+      camera_name="rgbd"
+      camera_suffix=""
+      parent_link="base_link"
       parent_frame_name="${namespace}/fcu"
       enable_realistic_realsense="${optionals['use_realistic_realsense']}"
@@ -769,7 +769,7 @@
     <xacro:realsense_macro
       namespace="${namespace}"
-      realsense_namespace=""
-      parent_link="base_link"
-      camera_suffix="realsense_up"
+      camera_name="rgbd"
+      camera_suffix="_up"
+      parent_link="base_link"
       parent_frame_name="${namespace}/fcu"
       enable_realistic_realsense="${optionals['use_realistic_realsense']}"
@@ -788,44 +788,10 @@
     <xacro:realsense_macro
       namespace="${namespace}"
-      realsense_namespace=""
-      parent_link="base_link"
-      camera_suffix="realsense_down"
+      camera_name="rgbd"
+      camera_suffix="_down"
+      parent_link="base_link"
       parent_frame_name="${namespace}/fcu"
       enable_realistic_realsense="${optionals['use_realistic_realsense']}"
       x="0.1"
-      y="0"
-      z="-0.05"
-      roll="0"
-      pitch="+${rad90}"
-      yaw="0">
-    </xacro:realsense_macro>
-  </xacro:if>
-  <!--}-->
-  <!-- up_down {-->
-  <xacro:if value="${optionals['enable_realsense_up_down']}">
-    <!-- sensor -->
-    <xacro:realsense_macro
-      namespace="${namespace}"
-      realsense_namespace="up_rgbd"
-      parent_link="base_link"
-      camera_suffix="realsense_up"
-      parent_frame_name="${namespace}/fcu"
-      enable_realistic_realsense="${optionals['use_realistic_realsense']}"
-      x="-0.01"
-      y="-0.07"
-      z="0.05"
-      roll="0"
-      pitch="-${rad90}"
-      yaw="${rad90}">
-    </xacro:realsense_macro>
-    <!-- sensor -->
-    <xacro:realsense_macro
-      namespace="${namespace}"
-      realsense_namespace="down_rgbd"
-      parent_link="base_link"
-      camera_suffix="realsense_down"
-      parent_frame_name="${namespace}/fcu"
-      enable_realistic_realsense="${optionals['use_realistic_realsense']}"
-      x="0.12"
       y="0"
       z="-0.05"
@@ -1274,5 +1240,5 @@
     <xacro:realsense_macro
       namespace="${namespace}"
-      realsense_namespace=""
+      camera_name=""
       parent_link="base_link"
       camera_suffix="realsense_down"
