Commit message: add models/visuals/sensor setups for NAKI drone

File: models/mrs_robots_description/urdf/component_snippets.xacro (robot description, xacro)
@@ -116,4 +116,23 @@
   </xacro:macro>
   <!--}-->
+  <!-- Macro for visualization of textured mash with collision {-->
+  <xacro:macro name="textured_visual_macro_with_collision"
+    params="robot_namespace name mesh_file mesh_scale parent *origin *collision">
+    <joint name="${name}_joint" type="fixed">
+      <xacro:insert_block name="origin" />
+      <parent link="${parent}" />
+      <child link="${name}_link" />
+    </joint>
+    <link name="${name}_link">
+      <visual>
+        <origin xyz="0 0 0" rpy="0 0 0" />
+        <geometry>
+          <mesh filename="${mesh_file}" scale="${mesh_scale}" />
+        </geometry>
+      </visual>
+      <xacro:insert_block name="collision" />
+    </link>
+  </xacro:macro>
+  <!--}-->
  <!-- Macro for visualization of mash with collision {-->
   <xacro:macro name="visual_macro_with_collision"
@@ -359,5 +378,5 @@
   </xacro:macro>
   <!--}-->
-  <!-- Macro for main multirotor without mesh for simplier physics{-->
+  <!-- Macro for main multirotor without mesh for simplier physics {-->
   <xacro:macro name="multirotor_base_without_mesh_macro"
     params="robot_namespace mass body_radius body_height *inertia">
@@ -380,4 +399,46 @@
         </geometry>
       </collision>
+    </link>
+    <!-- attach multirotor_base_plugin to the base_link -->
+    <gazebo>
+      <plugin filename="libgazebo_multirotor_base_plugin.so" name="rosbag">
+        <robotNamespace>${robot_namespace}</robotNamespace>
+        <linkName>base_link</linkName>
+        <rotorVelocitySlowdownSim>${rotor_velocity_slowdown_sim}</rotorVelocitySlowdownSim>
+      </plugin>
+    </gazebo>
+    <gazebo reference="base_link">
+      <collision name='base_link_inertia_collision'>
+        <surface>
+          <contact>
+            <ode>
+              <min_depth>0.001</min_depth>
+              <max_vel>0.0</max_vel>
+            </ode>
+          </contact>
+          <friction>
+            <ode/>
+          </friction>
+        </surface>
+      </collision>
+    </gazebo>
+  </xacro:macro>
+  <!--}-->
+  <!-- Macro for main multirotor without mesh for simplier physics with collision {-->
+  <xacro:macro name="multirotor_base_without_mesh_with_collision_macro"
+    params="robot_namespace mass *inertia *collision">
+    <link name="base_link"></link>
+    <joint name="base_joint" type="fixed">
+      <origin xyz="0 0 0" rpy="0 0 0" />
+      <parent link="base_link" />
+      <child link="base_link_inertia" />
+    </joint>
+    <link name="base_link_inertia">
+      <inertial>
+        <mass value="${mass}" />  <!-- [kg] -->
+        <origin xyz="0 0 0" />
+        <xacro:insert_block name="inertia" />
+      </inertial>
+      <xacro:insert_block name="collision" />
     </link>
     <!-- attach multirotor_base_plugin to the base_link -->
@@ -1951,5 +2012,5 @@
   <!--}-->
   <!-- Macro to add a camera mounted on virtual servo {-->
-  <xacro:macro name="servo_camera_macro" params="namespace name parent offset_x offset_y offset_z offset_yaw offset_roll offset_pitch update_rate max_pitch_rate camera_type compensate_tilt">
+  <xacro:macro name="servo_camera_macro" params="namespace name parent offset_x offset_y offset_z offset_yaw offset_roll offset_pitch update_rate max_pitch_rate camera_type compensate_tilt *visual">
       <joint name="${name}_joint" type="revolute">
           <parent link="${parent}"/>
@@ -1965,9 +2026,5 @@
               <inertia ixx="1e-5" ixy="0.0" ixz="0.0" iyy="1e-5" iyz="0.0" izz="1e-5"/>
           </inertial>
-        <visual>
-          <geometry>
-            <box size="0.01 0.01 0.01" />
-          </geometry>
-        </visual>
+          <xacro:insert_block name="visual" />
       </link>
       <gazebo>

File: models/mrs_robots_description/urdf/f450.xacro (robot description, xacro)
@@ -1016,4 +1016,9 @@
       update_rate="30.0"
       compensate_tilt="true">
+      <visual>
+        <geometry>
+          <box size="0.01 0.01 0.01" />
+        </geometry>
+      </visual>
     </xacro:servo_camera_macro>
   </xacro:if>

File: models/mrs_robots_description/urdf/f550.xacro (robot description, xacro)
@@ -1059,4 +1059,9 @@
       update_rate="30.0"
       compensate_tilt="true">
+      <visual>
+        <geometry>
+          <box size="0.01 0.01 0.01" />
+        </geometry>
+      </visual>
     </xacro:servo_camera_macro>
   </xacro:if>

File: models/mrs_robots_description/urdf/naki.xacro (robot description, xacro)
@@ -38,19 +38,20 @@
   <!-- Robot parameters and arguments {-->
   <xacro:property name="mass" value="7.00" /> <!-- [kg] -->
-  <xacro:property name="body_radius" value="0.29" /> <!-- [m] -->
-  <xacro:property name="body_height" value="0.45" /> <!-- [m] -->
+  <xacro:property name="body_radius" value="0.47" /> <!-- [m] -->
+  <xacro:property name="body_height" value="0.155" /> <!-- [m] -->
+  <xacro:property name="body_center_z" value="-0.0195" /> <!-- [m] -->
+  <xacro:property name="legs_width" value="0.43" /> <!-- [m] -->
+  <xacro:property name="legs_height" value="0.12" /> <!-- [m] -->
   <xacro:property name="mass_rotor" value="0.005" /> <!-- [kg] -->
   <xacro:property name="radius_rotor" value="0.165" /> <!-- [m] -->
   <xacro:property name="rotor_offset_top" value="0.0235" /> <!-- [m] -->
-  <xacro:property name="arm_length" value="0.29" /> <!-- [m] -->
-  <xacro:property name="arm_height" value="0.015" /> <!-- [m] -->
-  <xacro:property name="board_radius" value="0.065" /> <!-- [m] -->
-  <xacro:property name="board_height" value="0.002" /> <!-- [m] -->
-  <xacro:property name="holder_offset" value="0.02" /> <!-- [m] -->
-  <xacro:property name="leg_offset_z" value="0.098" /> <!-- [m] -->
-  <!-- <xacro:property name="leg_offset_z" value="0.133" /> -->
-  <xacro:property name="leg_offset_r" value="0.0072" /> <!-- [m] -->
-  <xacro:property name="pixhawk_offset" value="0.0075" /> <!-- [m] -->
-  <xacro:arg name="use_battery_mount" default="true" /> <!-- [m] -->
+  <xacro:property name="arm_length_x" value="0.1911" /> <!-- [m] -->
+  <xacro:property name="arm_length_y" value="0.2109" /> <!-- [m] -->
+  <xacro:property name="arm_height" value="0.016" /> <!-- [m] -->
+  <xacro:property name="arm_offset_z" value="0.015" /> <!-- [m] -->
+  <xacro:property name="motor_to_mount" value="0.0095" /> <!-- [m] -->
+  <xacro:property name="motor_z_offset" value="-0.01875" /> <!-- [m] -->
+  <xacro:property name="motor_height" value="0.0235" /> <!-- [m] -->
+  <xacro:property name="pixhawk_offset" value="0.008" /> <!-- [m] -->
   <!--}-->
   <!-- Motor constants {-->
@@ -68,22 +69,12 @@
   <xacro:property name="inertia_body_height" value="0.20" /> <!-- [m] -->
   <!--}-->
-  <!-- TODO -->
   <!-- Meshes {-->
   <!-- drone parts -->
-  <xacro:property name="central_board_mesh_top" value="package://mrs_robots_description/meshes/dji/f450/dji_f450_central_top.dae" />
-  <xacro:property name="central_board_mesh_bottom" value="package://mrs_robots_description/meshes/dji/f450/dji_f450_central_bottom.dae" />
-  <xacro:property name="arm_mesh_file" value="package://mrs_robots_description/meshes/dji/f450/dji_f450_arm.dae" />
-  <xacro:property name="leg_mesh_file" value="package://mrs_robots_description/meshes/dji/f450/dji_f450_leg_170mm.dae"/>
-  <!-- <xacro:property name="leg_mesh_file" value="package://mrs_robots_description/meshes/dji/f450/dji_f450_leg_240mm.dae"/> -->
-  <xacro:property name="rotor_mesh_file" value="package://mrs_robots_description/meshes/dji/f450/dji_f450_rotor.dae" />
-  <xacro:property name="prop_mesh_file" value="package://mrs_robots_description/meshes/dji/f450/dji_f450_prop.dae"/>
+  <xacro:property name="frame_legless_sensorless_file" value="package://mrs_robots_description/meshes/custom/naki/NAKI_legless_frame.dae" />
+  <xacro:property name="legs_file" value="package://mrs_robots_description/meshes/custom/naki/NAKI_legs.dae" />
+  <xacro:property name="rotor_mesh_file" value="package://mrs_robots_description/meshes/custom/naki/dji_f450_rotor.dae" />
+  <xacro:property name="prop_mesh_file" value="package://mrs_robots_description/meshes/custom/naki/NAKI_propeller.dae"/>
+  <xacro:property name="sony_camera_mesh_file" value="package://mrs_robots_description/meshes/custom/naki/NAKI_sony_alpha_6500_w_gimbal_mount.dae"/>
   <xacro:property name="pixhawk_mesh_file" value="package://mrs_robots_description/meshes/sensors/pixhawk.dae" />
-  <xacro:property name="nuc_mesh_file" value="package://mrs_robots_description/meshes/dji/f450/dji_f450_nuc.dae" />
-  <!-- holders -->
-  <xacro:property name="battery_mount_mesh" value="package://mrs_robots_description/meshes/dji/f450/dji_f450_battery_mount.dae" />
-  <xacro:property name="ouster_mount_mesh" value="package://mrs_robots_description/meshes/dji/f450/dji_f450_ouster_mount.dae" />
-  <xacro:property name="garmin_mount_mesh" value="package://mrs_robots_description/meshes/dji/f450/dji_f450_garmin_mount.dae" />
-  <xacro:property name="rplidar_mount_mesh" value="package://mrs_robots_description/meshes/dji/f450/dji_f450_rplidar_mount.dae" />
-  <xacro:property name="realsense_front_mount_mesh" value="package://mrs_robots_description/meshes/dji/f450/dji_f450_realsense_front_pitched_0_mount.dae" />
   <!-- scales -->
   <xacro:property name="mesh_scale" value="1 1 1"/>
@@ -115,223 +106,125 @@
   </xacro:property>
   <!-- Instantiate multirotor_base_macro {-->
-  <xacro:multirotor_base_without_mesh_macro
+  <xacro:multirotor_base_without_mesh_with_collision_macro
     robot_namespace="${namespace}"
     mass="${mass}"
-    body_radius="${body_radius}"
-    body_height="${body_height}"
     >
     <xacro:insert_block name="body_inertia" />
-  </xacro:multirotor_base_without_mesh_macro>
+    <collision>
+      <origin xyz="0 0 ${body_center_z}" rpy="0 0 0" />
+      <geometry>
+        <cylinder radius="${body_radius}" length="${body_height}" />
+      </geometry>
+    </collision>
+  </xacro:multirotor_base_without_mesh_with_collision_macro>
   <!--}-->
   <!--}-->
   <!-- Body parts {-->
   <!-- Boards {-->
+  <xacro:textured_visual_macro
+    robot_namespace="${namespace}"
+    name="frame_legless_sensorless_file"
+    mesh_file="${frame_legless_sensorless_file}"
+    mesh_scale="${mesh_scale}"
+    parent="base_link">
+    <origin xyz="0 0 0" rpy="0 0 0" />
+  </xacro:textured_visual_macro>
+  <xacro:textured_visual_macro_with_collision
+    robot_namespace="${namespace}"
+    name="legs_file"
+    mesh_file="${legs_file}"
+    mesh_scale="${mesh_scale}"
+    parent="base_link">
+    <origin xyz="0 0 0" rpy="0 0 0" />
+    <collision>
+      <!-- Is blocking garmin -->
+      <!-- <origin xyz="0 0 -${body_height/2 + legs_height/2}" rpy="0 0 0"/> -->
+      <!-- <geometry> -->
+        <!-- <box size="${legs_width} ${legs_width} ${legs_height}" /> -->
+      <!-- </geometry> -->
+      <origin xyz="0 0 0" rpy="0 0 0"/>
+      <geometry>
+        <mesh filename="${legs_file}" scale="${mesh_scale}" />
+      </geometry>
+    </collision>
+  </xacro:textured_visual_macro_with_collision>
+  <!--}-->
+  <!-- pixhawk {-->
+   <xacro:visual_macro
+     robot_namespace="${namespace}"
+     name="pixhawk"
+     mesh_file="${pixhawk_mesh_file}"
+     mesh_scale="${mesh_scale}"
+     parent="base_link"
+     color="DarkGrey">
+     <origin xyz="0 0 ${pixhawk_offset}" rpy="0 0 0" />
+   </xacro:visual_macro>
+  <!-- } -->
+  <!-- Rotors {-->
   <xacro:visual_macro
     robot_namespace="${namespace}"
-    name="lower_central_board"
-    mesh_file="${central_board_mesh_bottom}"
-    mesh_scale="${mesh_scale}"
-    parent="base_link"
-    color="DarkGrey">
-    <origin xyz="0 0 -${body_height/2}" rpy="0 0 0" />
+    name="top_front_right_rotor"
+    mesh_file="${rotor_mesh_file}"
+    mesh_scale="${mesh_scale}"
+    parent="base_link"
+    color="Black">
+  <origin xyz="${arm_length_x} -${arm_length_y} ${motor_z_offset + motor_to_mount}" rpy="0 0 0" />
   </xacro:visual_macro>
   <xacro:visual_macro
     robot_namespace="${namespace}"
-    name="upper_central_board"
-    mesh_file="${central_board_mesh_top}"
-    mesh_scale="${mesh_scale}"
-    parent="base_link"
-    color="DarkGrey">
-    <origin xyz="0 0 ${arm_height - body_height/2}" rpy="0 0 0" />
-  </xacro:visual_macro>
-  <!--}-->
-  <!-- Arms {-->
-  <xacro:visual_macro
-    robot_namespace="${namespace}"
-    name="front_right_arm"
-    mesh_file="${arm_mesh_file}"
-    mesh_scale="${mesh_scale}"
-    parent="base_link"
-    color="White">
-    <origin xyz="${board_radius * sin45} -${board_radius * sin45} ${arm_height - body_height/2}" rpy="0 0 -${rad45}" />
+    name="top_back_right_rotor"
+    mesh_file="${rotor_mesh_file}"
+    mesh_scale="${mesh_scale}"
+    parent="base_link"
+    color="Black">
+  <origin xyz="-${arm_length_x} ${arm_length_y} ${motor_z_offset + motor_to_mount}" rpy="0 0 0" />
   </xacro:visual_macro>
   <xacro:visual_macro
     robot_namespace="${namespace}"
-    name="front_left_arm"
-    mesh_file="${arm_mesh_file}"
-    mesh_scale="${mesh_scale}"
-    parent="base_link"
-    color="White">
-    <origin xyz="${board_radius * sin45} ${board_radius * sin45} ${arm_height - body_height/2}" rpy="0 0 ${rad45}" />
+    name="top_front_left_rotor"
+    mesh_file="${rotor_mesh_file}"
+    mesh_scale="${mesh_scale}"
+    parent="base_link"
+    color="Black">
+  <origin xyz="${arm_length_x} ${arm_length_y} ${motor_z_offset + motor_to_mount}" rpy="0 0 0" />
   </xacro:visual_macro>
   <xacro:visual_macro
     robot_namespace="${namespace}"
-    name="back_right_arm"
-    mesh_file="${arm_mesh_file}"
-    mesh_scale="${mesh_scale}"
-    parent="base_link"
-    color="Red">
-    <origin xyz="-${board_radius * sin45} -${board_radius * sin45} ${arm_height - body_height/2}" rpy="0 0 -${rad135}" />
+    name="top_back_left_rotor"
+    mesh_file="${rotor_mesh_file}"
+    mesh_scale="${mesh_scale}"
+    parent="base_link"
+    color="Black">
+  <origin xyz="-${arm_length_x} -${arm_length_y} ${motor_z_offset + motor_to_mount}" rpy="0 0 0" />
   </xacro:visual_macro>
   <xacro:visual_macro
     robot_namespace="${namespace}"
-    name="back_left_arm"
-    mesh_file="${arm_mesh_file}"
-    mesh_scale="${mesh_scale}"
-    parent="base_link"
-    color="Red">
-    <origin xyz="-${board_radius * sin45} ${board_radius * sin45} ${arm_height - body_height/2}" rpy="0 0 ${rad135}" />
-  </xacro:visual_macro>
-  <!--}-->
-  <!-- intel nuc {-->
-  <xacro:visual_macro
-    robot_namespace="${namespace}"
-    name="NUC"
-    mesh_file="${nuc_mesh_file}"
-    mesh_scale="${mesh_scale_milimeters}"
-    parent="base_link"
-    color="DarkGrey">
-    <origin xyz="0 0 0.023" rpy="0 0 0" />
-  </xacro:visual_macro>
-  <!--}-->
-  <!-- pixhawk {-->
-  <xacro:visual_macro
-    robot_namespace="${namespace}"
-    name="pixhawk"
-    mesh_file="${pixhawk_mesh_file}"
-    mesh_scale="${mesh_scale}"
-    parent="base_link"
-    color="DarkGrey">
-    <origin xyz="0 0 -${body_height/2 - pixhawk_offset}" rpy="0 0 0" />
-  </xacro:visual_macro>
-  <!--}-->
-  <!-- legs {-->
-  <xacro:leg_macro
-    robot_namespace="${namespace}"
-    name="front_right_leg"
-    mesh_file="${leg_mesh_file}"
-    mesh_scale="${mesh_scale_milimeters}"
-    parent="base_link"
-    color="White">
-    <origin xyz="${(arm_length - leg_offset_r) * sin45} -${(arm_length - leg_offset_r) * sin45} ${arm_height - body_height/2 - leg_offset_z}" rpy="0 0 ${rad135}" />
-    <collision>
-      <geometry>
-        <cylinder length="0.170" radius="${leg_offset_r}" />
-        <!-- <cylinder length="0.240" radius="${leg_offset_r}" /> -->
-      </geometry>
-    </collision>
-  </xacro:leg_macro>
-  <xacro:leg_macro
-    robot_namespace="${namespace}"
-    name="front_left_leg"
-    mesh_file="${leg_mesh_file}"
-    mesh_scale="${mesh_scale_milimeters}"
-    parent="base_link"
-    color="White">
-    <origin xyz="${(arm_length - leg_offset_r) * sin45} ${(arm_length - leg_offset_r) * sin45} ${arm_height - body_height/2 - leg_offset_z}" rpy="0 0 -${rad135}" />
-    <collision>
-      <geometry>
-        <cylinder length="0.170" radius="${leg_offset_r}" />
-        <!-- <cylinder length="0.240" radius="${leg_offset_r}" /> -->
-      </geometry>
-    </collision>
-  </xacro:leg_macro>
-  <xacro:leg_macro
-    robot_namespace="${namespace}"
-    name="rear_left_leg"
-    mesh_file="${leg_mesh_file}"
-    mesh_scale="${mesh_scale_milimeters}"
-    parent="base_link"
-    color="White">
-    <origin xyz="-${(arm_length - leg_offset_r) * sin45} ${(arm_length - leg_offset_r) * sin45} ${arm_height - body_height/2 - leg_offset_z}" rpy="0 0 -${rad45}" />
-    <collision>
-      <geometry>
-        <cylinder length="0.170" radius="${leg_offset_r}" />
-        <!-- <cylinder length="0.240" radius="${leg_offset_r}" /> -->
-      </geometry>
-    </collision>
-  </xacro:leg_macro>
-  <xacro:leg_macro
-    robot_namespace="${namespace}"
-    name="rear_right_leg"
-    mesh_file="${leg_mesh_file}"
-    mesh_scale="${mesh_scale_milimeters}"
-    parent="base_link"
-    color="White">
-    <origin xyz="-${(arm_length - leg_offset_r) * sin45} -${(arm_length - leg_offset_r) * sin45} ${arm_height - body_height/2 - leg_offset_z}" rpy="0 0 ${rad45}" />
-    <collision>
-      <geometry>
-        <cylinder length="0.170" radius="${leg_offset_r}" />
-        <!-- <cylinder length="0.240" radius="${leg_offset_r}" /> -->
-      </geometry>
-    </collision>
-  </xacro:leg_macro>
-  <!--}-->
-  <!-- Rotors {-->
-  <xacro:visual_macro
-    robot_namespace="${namespace}"
-    name="top_front_right_rotor"
+    name="bottom_front_right_rotor"
     mesh_file="${rotor_mesh_file}"
     mesh_scale="${mesh_scale}"
     parent="base_link"
     color="Black">
-    <origin xyz="${arm_length * sin45} -${arm_length * sin45} ${arm_height - body_height/2}" rpy="0 0 0" />
+  <origin xyz="${arm_length_x} -${arm_length_y} ${motor_z_offset - motor_to_mount}" rpy="0 ${rad180} 0" />
   </xacro:visual_macro>
   <xacro:visual_macro
     robot_namespace="${namespace}"
-    name="top_back_right_rotor"
+    name="bottom_back_right_rotor"
     mesh_file="${rotor_mesh_file}"
     mesh_scale="${mesh_scale}"
     parent="base_link"
     color="Black">
-    <origin xyz="-${arm_length * sin45} -${arm_length * sin45} ${arm_height - body_height/2}" rpy="0 0 0" />
+  <origin xyz="-${arm_length_x} ${arm_length_y} ${motor_z_offset - motor_to_mount}" rpy="0 ${rad180} 0" />
   </xacro:visual_macro>
   <xacro:visual_macro
     robot_namespace="${namespace}"
-    name="top_front_left_rotor"
+    name="bottom_front_left_rotor"
     mesh_file="${rotor_mesh_file}"
     mesh_scale="${mesh_scale}"
     parent="base_link"
     color="Black">
-    <origin xyz="${arm_length * sin45} ${arm_length * sin45} ${arm_height - body_height/2}" rpy="0 0 0" />
+  <origin xyz="${arm_length_x} ${arm_length_y} ${motor_z_offset - motor_to_mount}" rpy="0 ${rad180} 0" />
   </xacro:visual_macro>
   <xacro:visual_macro
     robot_namespace="${namespace}"
-    name="top_back_left_rotor"
-    mesh_file="${rotor_mesh_file}"
-    mesh_scale="${mesh_scale}"
-    parent="base_link"
-    color="Black">
-    <origin xyz="-${arm_length * sin45} ${arm_length * sin45} ${arm_height - body_height/2}" rpy="0 0 0" />
-  </xacro:visual_macro>
-  <xacro:visual_macro
-    robot_namespace="${namespace}"
-    name="bottom_front_right_rotor"
-    mesh_file="${rotor_mesh_file}"
-    mesh_scale="${mesh_scale}"
-    parent="base_link"
-    color="Black">
-    <origin xyz="${arm_length * sin45} -${arm_length * sin45} ${-arm_height - body_height/2}" rpy="0 ${rad180} 0" />
-  </xacro:visual_macro>
-  <xacro:visual_macro
-    robot_namespace="${namespace}"
-    name="bottom_back_right_rotor"
-    mesh_file="${rotor_mesh_file}"
-    mesh_scale="${mesh_scale}"
-    parent="base_link"
-    color="Black">
-    <origin xyz="-${arm_length * sin45} -${arm_length * sin45} ${-arm_height - body_height/2}" rpy="0 ${rad180} 0" />
-  </xacro:visual_macro>
-  <xacro:visual_macro
-    robot_namespace="${namespace}"
-    name="bottom_front_left_rotor"
-    mesh_file="${rotor_mesh_file}"
-    mesh_scale="${mesh_scale}"
-    parent="base_link"
-    color="Black">
-    <origin xyz="${arm_length * sin45} ${arm_length * sin45} ${-arm_height - body_height/2}" rpy="0 ${rad180} 0" />
-  </xacro:visual_macro>
-  <xacro:visual_macro
-    robot_namespace="${namespace}"
     name="bottom_back_left_rotor"
     mesh_file="${rotor_mesh_file}"
@@ -339,5 +232,5 @@
     parent="base_link"
     color="Black">
-    <origin xyz="-${arm_length * sin45} ${arm_length * sin45} ${-arm_height - body_height/2}" rpy="0 ${rad180} 0" />
+  <origin xyz="-${arm_length_x} -${arm_length_y} ${motor_z_offset - motor_to_mount}" rpy="0 ${rad180} 0" />
   </xacro:visual_macro>
   <!--}-->
@@ -361,5 +254,5 @@
     mesh_scale="${mesh_scale_prop_ccw}"
     color="White">
-    <origin xyz="${arm_length * sin45} -${arm_length * sin45} ${arm_height + rotor_offset_top - body_height/2}"  rpy="0 0 0" />
+    <origin xyz="${arm_length_x} -${arm_length_y} ${motor_z_offset + motor_to_mount + motor_height}" rpy="0 0 0" />
     <xacro:insert_block name="rotor_inertia" />
   </xacro:vertical_rotor>
@@ -382,5 +275,5 @@
     mesh_scale="${mesh_scale_prop_ccw}"
     color="White">
-    <origin xyz="-${arm_length * sin45} ${arm_length * sin45} ${arm_height + rotor_offset_top - body_height/2}" rpy="0 0 0" />
+    <origin xyz="-${arm_length_x} ${arm_length_y} ${motor_z_offset + motor_to_mount + motor_height}" rpy="0 0 0" />
     <xacro:insert_block name="rotor_inertia" />
   </xacro:vertical_rotor>
@@ -403,5 +296,5 @@
     mesh_scale="${mesh_scale_prop_cw}"
     color="White">
-    <origin xyz="${arm_length * sin45} ${arm_length * sin45} ${arm_height + rotor_offset_top - body_height/2}" rpy="0 0 0" />
+    <origin xyz="${arm_length_x} ${arm_length_y} ${motor_z_offset + motor_to_mount + motor_height}" rpy="0 0 0" />
     <xacro:insert_block name="rotor_inertia" />
   </xacro:vertical_rotor>
@@ -424,5 +317,5 @@
     mesh_scale="${mesh_scale_prop_cw}"
     color="White">
-    <origin xyz="-${arm_length * sin45} -${arm_length * sin45} ${arm_height + rotor_offset_top - body_height/2}" rpy="0 0 0" />
+    <origin xyz="-${arm_length_x} -${arm_length_y} ${motor_z_offset + motor_to_mount + motor_height}" rpy="0 0 0" />
     <xacro:insert_block name="rotor_inertia" />
   </xacro:vertical_rotor>
@@ -430,5 +323,5 @@
     robot_namespace="${namespace}"
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
File: models/mrs_robots_description/urdf/t650.xacro (robot description, xacro)
@@ -932,4 +932,9 @@
       update_rate="30.0"
       compensate_tilt="true">
+      <visual>
+        <geometry>
+          <box size="0.01 0.01 0.01" />
+        </geometry>
+      </visual>
     </xacro:servo_camera_macro>
   </xacro:if>
