Commit message: add macro for ultrasonic sensors; add them to NAKI drone

File: models/mrs_robots_description/urdf/component_snippets.xacro (robot description, xacro)
@@ -785,5 +785,5 @@
   <!-- Macro to add the rangefinder_plugin {-->
   <xacro:macro name="rangefinder_macro"
-    params="namespace parent_link rangefinder_suffix parent_frame_name rangefinder_frame_name topic
+    params="namespace parent_link parent_frame_name rangefinder_frame_name topic
     frame_rate fov min_distance max_distance resolution noise
     x y z roll pitch yaw
@@ -1091,5 +1091,4 @@
       parent_link="${parent_link}"
       frame_rate="100"
-      rangefinder_suffix="garmin${orientation}"
       rangefinder_frame_name="${namespace}/garmin${orientation}"
       parent_frame_name="${namespace}/fcu"
@@ -1125,6 +1124,5 @@
       parent_link="${parent_link}"
       frame_rate="100"
-      rangefinder_suffix="teraranger"
-      rangefinder_frame_name="${nacamespace}/teraranger"
+      rangefinder_frame_name="${namespace}/teraranger"
       parent_frame_name="${namespace}/fcu"
       topic="teraranger/range"
@@ -1145,4 +1143,36 @@
         <geometry>
           <box size=".027 .033 0.015" />
+        </geometry>
+      </visual>
+    </xacro:rangefinder_macro>
+  </xacro:macro>
+  <!--}-->
+  <!-- Macro to add a URM37 ultrasound {-->
+  <xacro:macro name="ultrasonic_sensor_macro" params="namespace parent_link suffix x y z yaw pitch roll">
+    <xacro:rangefinder_macro
+      namespace="${namespace}"
+      name="ultrasonic${suffix}"
+      color="DarkGrey"
+      parent_link="${parent_link}"
+      frame_rate="40"
+      rangefinder_frame_name="${namespace}/ultrasonic${suffix}"
+      parent_frame_name="${namespace}/fcu"
+      topic="ultrasonic${suffix}/range"
+      fov="0.698131701"
+      min_distance="0.04"
+      max_distance="5.0"
+      resolution= "0.01"
+      noise="0.04"
+      x="${x}"
+      y="${y}"
+      z="${z}"
+      yaw="${yaw}"
+      pitch="${pitch}"
+      roll="${roll}"
+      >
+      <visual>
+        <origin xyz="0 0 0" rpy="0 0 0" />
+        <geometry>
+          <mesh filename="package://mrs_robots_description/meshes/sensors/ultrasonic_URM37.dae" scale="1 1 1" />
         </geometry>
       </visual>

File: models/mrs_robots_description/urdf/naki.xacro (robot description, xacro)
@@ -54,4 +54,7 @@
   <xacro:property name="motor_height" value="0.0235" /> <!-- [m] -->
   <xacro:property name="pixhawk_offset" value="0.008" /> <!-- [m] -->
+  <xacro:property name="ultrasonic_x" value="0.3173" /> <!-- [m] -->
+  <xacro:property name="ultrasonic_y" value="0.3390" /> <!-- [m] -->
+  <xacro:property name="ultrasonic_yaw" value="0.822463619" /> <!-- [rad] -->
   <!--}-->
   <!-- Motor constants {-->
@@ -404,4 +407,5 @@
     <xacro:insert_block name="rotor_inertia" />
   </xacro:vertical_rotor>
+  <!--}-->
   <!--}-->
   <!--}-->
@@ -525,5 +529,4 @@
   </xacro:if>
   <!--}-->
-  <!-- ====================== Documentation sensors ==================== -->
   <!-- ======================= rangefinder sensors ======================-->
   <!-- Garmin {-->
@@ -557,4 +560,86 @@
       >
     </xacro:garmin_macro>
+  </xacro:if>
+  <!--}-->
+  <!-- Ultrasonic sensors {-->
+  <xacro:if value="${optionals['enable_omni_ultrasounds']}">
+    <!-- Down -->
+    <xacro:ultrasonic_sensor_macro
+      namespace="${namespace}"
+      parent_link="base_link"
+      suffix="_down"
+      x="0.02"
+      y="0.0"
+      z="-0.1535"
+      roll="0"
+      pitch="${rad90}"
+      yaw="0"
+      >
+    </xacro:ultrasonic_sensor_macro>
+    <!-- Up -->
+    <xacro:ultrasonic_sensor_macro
+      namespace="${namespace}"
+      parent_link="base_link"
+      suffix="_up"
+      x="-0.1686"
+      y="0"
+      z="0.001"
+      roll="0"
+      pitch="-${rad90}"
+      yaw="0"
+      >
+    </xacro:ultrasonic_sensor_macro>
+    <!-- Front left -->
+    <xacro:ultrasonic_sensor_macro
+      namespace="${namespace}"
+      parent_link="base_link"
+      suffix="_fl"
+      x="${ultrasonic_x}"
+      y="${ultrasonic_y}"
+      z="-0.019"
+      roll="0"
+      pitch="0"
+      yaw="${ultrasonic_yaw}"
+      >
+    </xacro:ultrasonic_sensor_macro>
+    <!-- Front right -->
+    <xacro:ultrasonic_sensor_macro
+      namespace="${namespace}"
+      parent_link="base_link"
+      suffix="_fr"
+      x="${ultrasonic_x}"
+      y="-${ultrasonic_y}"
+      z="-0.019"
+      roll="0"
+      pitch="0"
+      yaw="-${ultrasonic_yaw}"
+      >
+    </xacro:ultrasonic_sensor_macro>
+    <!-- Back left -->
+    <xacro:ultrasonic_sensor_macro
+      namespace="${namespace}"
+      parent_link="base_link"
+      suffix="_bl"
+      x="-${ultrasonic_x}"
+      y="${ultrasonic_y}"
+      z="-0.019"
+      roll="0"
+      pitch="0"
+      yaw="${ultrasonic_yaw + rad90}"
+      >
+    </xacro:ultrasonic_sensor_macro>
+    <!-- Back right -->
+    <xacro:ultrasonic_sensor_macro
+      namespace="${namespace}"
+      parent_link="base_link"
+      suffix="_br"
+      x="-${ultrasonic_x}"
+      y="-${ultrasonic_y}"
+      z="-0.019"
+      roll="0"
+      pitch="0"
+      yaw="-${ultrasonic_yaw + rad90}"
+      >
+    </xacro:ultrasonic_sensor_macro>
   </xacro:if>
   <!--}-->

Commit message: add safety led macro

File: models/mrs_robots_description/urdf/component_snippets.xacro (robot description, xacro)
@@ -2482,4 +2482,28 @@
   </xacro:macro>
   <!--}-->
+  <!-- Macro to add a safety_led {-->
+  <xacro:macro name="safety_led_macro" params="namespace name parent failure_duration_threshold x y z roll pitch yaw">
+    <joint name="${name}_joint" type="fixed">
+      <origin xyz="${x} ${y} ${z}" rpy="${roll} ${pitch} ${yaw}" />
+      <parent link="${parent}" />
+      <child link="${name}_link" />
+    </joint>
+    <link name="${name}_link" >
+    </link>
+    <gazebo>
+      <plugin name="safety_led_plugin" filename="libMRSSafetyLedPlugin.so">
+        <model_name>safety_led</model_name>
+        <failure_duration_threshold>0.2</failure_duration_threshold>
+        <model_spawn_delay>5.0</model_spawn_delay>
+        <x>${x}</x>
+        <y>${y}</y>
+        <z>${z}</z>
+        <roll>${roll}</roll>
+        <pitch>${pitch}</pitch>
+        <yaw>${yaw}</yaw>
+      </plugin>
+    </gazebo>
+  </xacro:macro>
+  <!--}-->
   <!-- Macro to add a UV LED{-->
   <xacro:macro name="uvled_macro"

File: models/mrs_robots_description/urdf/naki.xacro (robot description, xacro)
@@ -814,4 +814,20 @@
   </xacro:if>
   <!--}-->
+  <!-- Safety LED {-->
+  <xacro:if value="${optionals['enable_safety_led']}">
+    <xacro:safety_led_macro
+      namespace="${namespace}"
+      name="safety_led"
+      parent="base_link"
+      failure_duration_threshold="0.2"
+      x="-0.202"
+      y="0.0"
+      z="-0.0195"
+      roll="0.0"
+      pitch="0.0"
+      yaw="3.1415">
+    </xacro:safety_led_macro>
+  </xacro:if>
+  <!--}-->
   <!-- ================================================================== -->
   <!-- ||         other equipment definitions (holders, boxes ...)     || -->

Commit message: fix naki propellers rotation

File: models/mrs_robots_description/urdf/component_snippets.xacro (robot description, xacro)
@@ -2494,5 +2494,5 @@
       <plugin name="safety_led_plugin" filename="libMRSSafetyLedPlugin.so">
         <model_name>safety_led</model_name>
-        <failure_duration_threshold>0.2</failure_duration_threshold>
+        <failure_duration_threshold>${failure_duration_threshold}</failure_duration_threshold>
         <model_spawn_delay>5.0</model_spawn_delay>
         <x>${x}</x>

File: models/mrs_robots_description/urdf/naki.xacro (robot description, xacro)
@@ -37,5 +37,5 @@
   <!-- ================================================================== -->
   <!-- Robot parameters and arguments {-->
-  <xacro:property name="mass" value="7.00" /> <!-- [kg] -->
+  <xacro:property name="mass" value="7.50" /> <!-- [kg] -->
   <xacro:property name="body_radius" value="0.47" /> <!-- [m] -->
   <xacro:property name="body_height" value="0.155" /> <!-- [m] -->
@@ -82,6 +82,6 @@
   <!-- scales -->
   <xacro:property name="mesh_scale" value="1 1 1"/>
-  <xacro:property name="mesh_scale_prop_ccw" value="1 1 1"/>
-  <xacro:property name="mesh_scale_prop_cw" value="-1 1 1"/>
+  <xacro:property name="mesh_scale_prop_ccw" value="-1 1 1"/>
+  <xacro:property name="mesh_scale_prop_cw" value="1 1 1"/>
   <xacro:property name="mesh_scale_milimeters" value="0.001 0.001 0.001" />
   <!--}-->
@@ -326,5 +326,5 @@
     robot_namespace="${namespace}"
     suffix="bottom_front_right"
-    direction="ccw"
+    direction="cw"
     motor_constant="${motor_constant}"
     moment_constant="${moment_constant}"
@@ -339,7 +339,7 @@
     rolling_moment_coefficient="${rolling_moment_coefficient}"
     mesh_file="${prop_mesh_file}"
-    mesh_scale="${mesh_scale_prop_ccw}"
+    mesh_scale="${mesh_scale_prop_cw}"
     color="White">
-    <origin xyz="${arm_length_x} -${arm_length_y} ${motor_z_offset - motor_to_mount - motor_height}" rpy="${rad180} 0 0" />
+    <origin xyz="${arm_length_x} -${arm_length_y} ${motor_z_offset - motor_to_mount - motor_height}" rpy="0 0 0" />
     <xacro:insert_block name="rotor_inertia" />
   </xacro:vertical_rotor>
@@ -347,5 +347,5 @@
     robot_namespace="${namespace}"
     suffix="bottom_back_left"
-    direction="ccw"
+    direction="cw"
     motor_constant="${motor_constant}"
     moment_constant="${moment_constant}"
@@ -360,7 +360,7 @@
     rolling_moment_coefficient="${rolling_moment_coefficient}"
     mesh_file="${prop_mesh_file}"
-    mesh_scale="${mesh_scale_prop_ccw}"
+    mesh_scale="${mesh_scale_prop_cw}"
     color="White">
-    <origin xyz="-${arm_length_x} ${arm_length_y} ${motor_z_offset - motor_to_mount - motor_height}" rpy="${rad180} 0 0" />
+    <origin xyz="-${arm_length_x} ${arm_length_y} ${motor_z_offset - motor_to_mount - motor_height}" rpy="0 0 0" />
     <xacro:insert_block name="rotor_inertia" />
   </xacro:vertical_rotor>
@@ -368,5 +368,5 @@
     robot_namespace="${namespace}"
     suffix="bottom_front_left"
-    direction="cw"
+    direction="ccw"
     motor_constant="${motor_constant}"
     moment_constant="${moment_constant}"
@@ -381,7 +381,7 @@
     rolling_moment_coefficient="${rolling_moment_coefficient}"
     mesh_file="${prop_mesh_file}"
-    mesh_scale="${mesh_scale_prop_cw}"
+    mesh_scale="${mesh_scale_prop_ccw}"
     color="White">
-    <origin xyz="${arm_length_x} ${arm_length_y} ${motor_z_offset - motor_to_mount - motor_height}" rpy="${rad180} 0 0" />
+    <origin xyz="${arm_length_x} ${arm_length_y} ${motor_z_offset - motor_to_mount - motor_height}" rpy="0 0 0" />
     <xacro:insert_block name="rotor_inertia" />
   </xacro:vertical_rotor>
@@ -389,5 +389,5 @@
     robot_namespace="${namespace}"
     suffix="bottom_back_right"
-    direction="cw"
+    direction="ccw"
     motor_constant="${motor_constant}"
     moment_constant="${moment_constant}"
@@ -402,7 +402,7 @@
     rolling_moment_coefficient="${rolling_moment_coefficient}"
     mesh_file="${prop_mesh_file}"
-    mesh_scale="${mesh_scale_prop_cw}"
+    mesh_scale="${mesh_scale_prop_ccw}"
     color="White">
-    <origin xyz="-${arm_length_x} -${arm_length_y} ${motor_z_offset - motor_to_mount - motor_height}" rpy="${rad180} 0 0" />
+    <origin xyz="-${arm_length_x} -${arm_length_y} ${motor_z_offset - motor_to_mount - motor_height}" rpy="0 0 0" />
     <xacro:insert_block name="rotor_inertia" />
   </xacro:vertical_rotor>

Commit message: ouster diag topic defaults now to os_cloud_nodelet/is_alive to match hw driver

File: models/mrs_robots_description/urdf/component_snippets.xacro (robot description, xacro)
@@ -1470,5 +1470,5 @@
     <xacro:property name="topic_lidar" value="/${namespace}/${sensor_name}_cloud_nodelet/points" />
     <xacro:property name="topic_imu" value="/${namespace}/${sensor_name}_cloud_nodelet/imu" />
-    <xacro:property name="topic_diag" value="/${namespace}/${sensor_name}_cloud_nodelet/diag" />
+    <xacro:property name="topic_diag" value="/${namespace}/${sensor_name}_cloud_nodelet/is_alive" />
       <!-- tf from sensor to lidar -->
     <xacro:property name="lidar_x" value="0" />

Commit message: Update servo camera macro

File: models/mrs_robots_description/urdf/component_snippets.xacro (robot description, xacro)
@@ -2042,36 +2042,77 @@
   <!--}-->
   <!-- Macro to add a camera mounted on virtual servo {-->
-  <xacro:macro name="servo_camera_macro" params="namespace name parent offset_x offset_y offset_z offset_yaw offset_roll offset_pitch update_rate max_pitch_rate camera_type compensate_tilt *visual">
-      <joint name="${name}_joint" type="revolute">
-          <parent link="${parent}"/>
-          <child link="${name}_link"/>
-          <axis xyz="0 1 0"/>
-          <dynamics damping="0.05" friction="0.05"/>
-          <limit upper="1.57" lower="-1.57" effort="1" velocity="10" />
-          <origin xyz="${offset_x} ${offset_y} ${offset_z}" rpy="0.0 0.0 0.0"/>
-      </joint>
-      <link name="${name}_link">
-          <inertial>
-              <mass value="1e-3" />
-              <inertia ixx="1e-5" ixy="0.0" ixz="0.0" iyy="1e-5" iyz="0.0" izz="1e-5"/>
-          </inertial>
-          <xacro:insert_block name="visual" />
-      </link>
-      <gazebo>
-        <plugin name="servo_camera_plugin" filename="libMRSGazeboServoCameraPlugin.so">
-          <offset_x>${offset_x}</offset_x>
-          <offset_y>${offset_y}</offset_y>
-          <offset_z>${offset_z}</offset_z>
-          <offset_pitch>${offset_pitch}</offset_pitch>
-          <offset_yaw>${offset_yaw}</offset_yaw>
-          <offset_roll>${offset_roll}</offset_roll>
-          <spawning_frame>${parent}</spawning_frame>
-          <update_rate>${update_rate}</update_rate>
-          <max_pitch_rate>${max_pitch_rate}</max_pitch_rate>
-          <joint_name>${name}_joint</joint_name>
-          <camera_type>${camera_type}</camera_type>
-          <compensate_tilt>${compensate_tilt}</compensate_tilt>
+  <xacro:macro name="servo_camera_macro" params="namespace name parent offset_x offset_y offset_z offset_yaw offset_roll offset_pitch pitch_update_rate max_pitch min_pitch max_pitch_rate compensate_tilt parent_frame_name sensor_base_frame_name camera_frame_name camera_update_rate horizontal_fov img_width img_height *visual">
+    <joint name="${namespace}_servo_camera_joint" type="revolute">
+      <parent link="${parent}"/>
+      <child link="${namespace}_servo_camera_link"/>
+      <axis xyz="0 1 0"/>
+      <dynamics damping="0.05" friction="0.05"/>
+      <limit upper="1.57" lower="-1.57" effort="1" velocity="10" />
+      <origin xyz="${offset_x} ${offset_y} ${offset_z}" rpy="0.0 0.0 0.0"/>
+    </joint>
+    <link name="${namespace}_servo_camera_link">
+      <inertial>
+        <mass value="1e-3" />
+        <inertia ixx="1e-5" ixy="0.0" ixz="0.0" iyy="1e-5" iyz="0.0" izz="1e-5"/>
+      </inertial>
+      <xacro:insert_block name="visual" />
+    </link>
+    <gazebo reference="${namespace}_servo_camera_link">
+      <sensor type="camera" name="servo_camera">
+        <update_rate>${camera_update_rate}</update_rate>
+        <camera name="head">
+          <horizontal_fov>${horizontal_fov}</horizontal_fov>
+          <image>
+            <width>${img_width}</width>
+            <height>${img_height}</height>
+          </image>
+          <clip>
+            <near>0.25</near>
+            <far>100</far>
+          </clip>
+          <noise>
+            <type>gaussian</type>
+              <!-- Noise is sampled independently per pixel on each frame.
+                That pixel's noise value is added to each of its color
+              channels, which at that point lie in the range [0,1]. -->
+            <mean>0.0</mean>
+            <stddev>0.01</stddev>
+          </noise>
+        </camera>
+        <plugin name="${namespace}_servo_camera_controller" filename="libMRSGazeboCameraPlugin.so">
+          <alwaysOn>true</alwaysOn>
+          <updateRate>${camera_update_rate}</updateRate>
+          <cameraName>servo_camera</cameraName>
+          <imageTopicName>image_raw</imageTopicName>
+          <cameraInfoTopicName>camera_info</cameraInfoTopicName>
+          <frameName>${camera_frame_name}</frameName>
+          <hackBaseline>0.0</hackBaseline>
+          <distortionK1>0.0</distortionK1>
+          <distortionK2>0.0</distortionK2>
+          <distortionK3>0.0</distortionK3>
+          <distortionT1>0.0</distortionT1>
+          <distortionT2>0.0</distortionT2>
+          <x>0.0</x>
+          <y>0.0</y>
+          <z>0.0</z>
+          <roll>0.0</roll>
+          <pitch>0.0</pitch>
+          <yaw>0.0</yaw>
+          <parentFrameName>${parent_frame_name}</parentFrameName>
+          <sensorBaseFrameName>${sensor_base_frame_name}</sensorBaseFrameName>
         </plugin>
-      </gazebo>
+      </sensor>
+    </gazebo>
+    <gazebo>
+      <plugin name="servo_camera_plugin" filename="libMRSGazeboServoCameraPlugin.so">
+        <spawning_frame>${parent}</spawning_frame>
+        <update_rate>${pitch_update_rate}</update_rate>
+        <max_pitch_rate>${max_pitch_rate}</max_pitch_rate>
+        <max_pitch>${max_pitch}</max_pitch>
+        <min_pitch>${min_pitch}</min_pitch>
+        <joint_name>${namespace}_servo_camera_joint</joint_name>
+        <compensate_tilt>${compensate_tilt}</compensate_tilt>
+      </plugin>
+    </gazebo>
   </xacro:macro>
   <!--}-->

File: models/mrs_robots_description/urdf/f450.xacro (robot description, xacro)
@@ -1006,13 +1006,21 @@
       name="servo_camera_macro"
       parent="base_link"
+      parent_frame_name="${namespace}/fcu"
+      camera_frame_name="${namespace}/servo_camera_optical"
+      sensor_base_frame_name="${namespace}/servo_camera"
       offset_x="0.2"
       offset_y="0.0"
-      offset_z="-0.10"
+      offset_z="-0.1"
       offset_roll="0.0"
       offset_yaw="0.0"
       offset_pitch="0.0"
+      pitch_update_rate="5.0"
+      min_pitch="-1.046"
+      max_pitch="1.57"
       max_pitch_rate="0.1"
-      camera_type="servo_camera"
-      update_rate="30.0"
+      camera_update_rate="30"
+      horizontal_fov="1.92"
+      img_width="1920"
+      img_height="1080"
       compensate_tilt="true">
       <visual>

File: models/mrs_robots_description/urdf/f550.xacro (robot description, xacro)
@@ -1049,13 +1049,21 @@
       name="servo_camera_macro"
       parent="base_link"
-      offset_x="0.2"
+      parent_frame_name="${namespace}/fcu"
+      camera_frame_name="${namespace}/servo_camera_optical"
+      sensor_base_frame_name="${namespace}/servo_camera"
+      offset_x="0.2278"
       offset_y="0.0"
-      offset_z="-0.10"
+      offset_z="-0.1378"
       offset_roll="0.0"
       offset_yaw="0.0"
       offset_pitch="0.0"
+      pitch_update_rate="5.0"
+      min_pitch="-1.046"
+      max_pitch="1.57"
       max_pitch_rate="0.1"
-      camera_type="servo_camera"
-      update_rate="30.0"
+      camera_update_rate="30"
+      horizontal_fov="1.92"
+      img_width="1920"
+      img_height="1080"
       compensate_tilt="true">
       <visual>

File: models/mrs_robots_description/urdf/naki.xacro (robot description, xacro)
@@ -777,4 +777,7 @@
     name="servo_camera_macro"
     parent="base_link"
+    parent_frame_name="${namespace}/fcu"
+    camera_frame_name="${namespace}/servo_camera_optical"
+    sensor_base_frame_name="${namespace}/servo_camera"
     offset_x="0.2278"
     offset_y="0.0"
@@ -783,7 +786,12 @@
     offset_yaw="0.0"
     offset_pitch="0.0"
+    pitch_update_rate="5.0"
+    min_pitch="-1.046"
+    max_pitch="1.57"
     max_pitch_rate="0.1"
-    camera_type="servo_camera"
-    update_rate="5.0"
+    camera_update_rate="30"
+    horizontal_fov="1.92"
+    img_width="1920"
+    img_height="1080"
     compensate_tilt="true">
     <visual>

File: models/mrs_robots_description/urdf/t650.xacro (robot description, xacro)
@@ -922,13 +922,21 @@
       name="servo_camera_macro"
       parent="base_link"
+      parent_frame_name="${namespace}/fcu"
+      camera_frame_name="${namespace}/servo_camera_optical"
+      sensor_base_frame_name="${namespace}/servo_camera"
       offset_x="0.2"
       offset_y="0.0"
-      offset_z="-0.10"
+      offset_z="-0.1"
       offset_roll="0.0"
       offset_yaw="0.0"
       offset_pitch="0.0"
+      pitch_update_rate="5.0"
+      min_pitch="-1.046"
+      max_pitch="1.57"
       max_pitch_rate="0.1"
-      camera_type="servo_camera"
-      update_rate="30.0"
+      camera_update_rate="30"
+      horizontal_fov="1.92"
+      img_width="1920"
+      img_height="1080"
       compensate_tilt="true">
       <visual>
