Commit message: Update servo camera xacros

File: models/mrs_robots_description/urdf/component_snippets.xacro (robot description, xacro)
@@ -2042,12 +2042,36 @@
   <!--}-->
   <!-- Macro to add a camera mounted on virtual servo {-->
-  <xacro:macro name="servo_camera_macro" params="namespace name parent offset_x offset_y offset_z offset_yaw offset_roll offset_pitch pitch_update_rate max_pitch min_pitch max_pitch_rate compensate_tilt parent_frame_name sensor_base_frame_name camera_frame_name camera_update_rate horizontal_fov img_width img_height *visual">
-    <joint name="${namespace}_servo_camera_joint" type="revolute">
+  <xacro:macro name="servo_camera_macro" params="namespace name parent offset_pitch_link_x offset_pitch_link_y offset_pitch_link_z offset_pitch_link_yaw offset_pitch_link_roll offset_pitch_link_pitch offset_roll_link_x offset_roll_link_y offset_roll_link_z offset_roll_link_yaw offset_roll_link_roll offset_roll_link_pitch tilt_update_rate max_pitch min_pitch max_pitch_rate max_roll min_roll max_roll_rate compensate_tilt_roll compensate_tilt_pitch parent_frame_name sensor_base_frame_name camera_frame_name camera_update_rate horizontal_fov img_width img_height roll_link_mesh_file pitch_link_mesh_file mesh_scale">
+    <joint name="${namespace}_servo_camera_joint_roll" type="revolute">
       <parent link="${parent}"/>
+      <child link="${namespace}_servo_camera_gimbal_link"/>
+      <axis xyz="1 0 0"/>
+      <dynamics damping="0.05" friction="0.05"/>
+      <limit upper="0.5" lower="-0.5" effort="1" velocity="10" />
+      <origin xyz="${offset_roll_link_x} ${offset_roll_link_y} ${offset_roll_link_z}" rpy="${offset_roll_link_roll} ${offset_roll_link_pitch} ${offset_roll_link_yaw}"/>
+    </joint>
+    <link name="${namespace}_servo_camera_gimbal_link">
+      <inertial>
+        <mass value="1e-3" />
+        <inertia ixx="1e-5" ixy="0.0" ixz="0.0" iyy="1e-5" iyz="0.0" izz="1e-5"/>
+      </inertial>
+      <visual>
+        <geometry>
+          <xacro:if value="${roll_link_mesh_file == ''}">
+            <mesh filename="${roll_link_mesh_file}" scale="${mesh_scale}" />
+          </xacro:if>
+          <xacro:unless value="${roll_link_mesh_file == ''}">
+            <box size="0.01 0.01 0.01" />
+          </xacro:unless>
+        </geometry>
+      </visual>
+    </link>
+    <joint name="${namespace}_servo_camera_joint_pitch" type="revolute">
+      <parent link="${namespace}_servo_camera_gimbal_link"/>
       <child link="${namespace}_servo_camera_link"/>
       <axis xyz="0 1 0"/>
       <dynamics damping="0.05" friction="0.05"/>
       <limit upper="1.57" lower="-1.57" effort="1" velocity="10" />
-      <origin xyz="${offset_x} ${offset_y} ${offset_z}" rpy="0.0 0.0 0.0"/>
+      <origin xyz="${offset_pitch_link_x} ${offset_pitch_link_y} ${offset_pitch_link_z}" rpy="${offset_pitch_link_roll} ${offset_pitch_link_pitch} ${offset_pitch_link_yaw}"/>
     </joint>
     <link name="${namespace}_servo_camera_link">
@@ -2056,5 +2080,14 @@
         <inertia ixx="1e-5" ixy="0.0" ixz="0.0" iyy="1e-5" iyz="0.0" izz="1e-5"/>
       </inertial>
-      <xacro:insert_block name="visual" />
+      <visual>
+        <geometry>
+          <xacro:if value="${pitch_link_mesh_file == ''}">
+            <box size="0.01 0.01 0.01" />
+          </xacro:if>
+          <xacro:unless value="${pitch_link_mesh_file == ''}">
+            <mesh filename="${pitch_link_mesh_file}" scale="${mesh_scale}" />
+          </xacro:unless>
+        </geometry>
+      </visual>
     </link>
     <gazebo reference="${namespace}_servo_camera_link">
@@ -2107,10 +2140,17 @@
       <plugin name="servo_camera_plugin" filename="libMRSGazeboServoCameraPlugin.so">
         <spawning_frame>${parent}</spawning_frame>
-        <update_rate>${pitch_update_rate}</update_rate>
+        <tilt_update_rate>${tilt_update_rate}</tilt_update_rate>
         <max_pitch_rate>${max_pitch_rate}</max_pitch_rate>
         <max_pitch>${max_pitch}</max_pitch>
         <min_pitch>${min_pitch}</min_pitch>
-        <joint_name>${namespace}_servo_camera_joint</joint_name>
-        <compensate_tilt>${compensate_tilt}</compensate_tilt>
+        <max_roll_rate>${max_roll_rate}</max_roll_rate>
+        <max_roll>${max_pitch}</max_roll>
+        <min_roll>${min_pitch}</min_roll>
+        <joint_name_pitch>${namespace}_servo_camera_joint_pitch</joint_name_pitch>
+        <joint_name_roll>${namespace}_servo_camera_joint_roll</joint_name_roll>
+        <parent_link_pitch>${namespace}_servo_camera_gimbal_link</parent_link_pitch>
+        <parent_link_roll>${parent}</parent_link_roll>
+        <compensate_tilt_roll>${compensate_tilt_roll}</compensate_tilt_roll>
+        <compensate_tilt_pitch>${compensate_tilt_pitch}</compensate_tilt_pitch>
       </plugin>
     </gazebo>

File: models/mrs_robots_description/urdf/f450.xacro (robot description, xacro)
@@ -1009,24 +1009,32 @@
       camera_frame_name="${namespace}/servo_camera_optical"
       sensor_base_frame_name="${namespace}/servo_camera"
-      offset_x="0.2"
-      offset_y="0.0"
-      offset_z="-0.1"
-      offset_roll="0.0"
-      offset_yaw="0.0"
-      offset_pitch="0.0"
-      pitch_update_rate="5.0"
-      min_pitch="-1.046"
+      offset_pitch_link_x="0.0"
+      offset_pitch_link_y="0.0"
+      offset_pitch_link_z="0.0"
+      offset_pitch_link_roll="0.0"
+      offset_pitch_link_yaw="0.0"
+      offset_pitch_link_pitch="0.0"
+      offset_roll_link_x="0.2"
+      offset_roll_link_y="0.0"
+      offset_roll_link_z="-0.1"
+      offset_roll_link_roll="0.0"
+      offset_roll_link_yaw="0.0"
+      offset_roll_link_pitch="0.0"
+      tilt_update_rate="5.0"
+      min_pitch="-1.57"
       max_pitch="1.57"
+      min_roll="-0.6"
+      max_roll="0.6"
       max_pitch_rate="0.1"
+      max_roll_rate="0.1"
       camera_update_rate="30"
       horizontal_fov="1.92"
       img_width="1920"
       img_height="1080"
-      compensate_tilt="true">
-      <visual>
-        <geometry>
-          <box size="0.01 0.01 0.01" />
-        </geometry>
-      </visual>
+      compensate_tilt_roll="true"
+      compensate_tilt_pitch="true"
+      pitch_link_mesh_file=""
+      roll_link_mesh_file=""
+      mesh_scale="">
     </xacro:servo_camera_macro>
   </xacro:if>

File: models/mrs_robots_description/urdf/f550.xacro (robot description, xacro)
@@ -1052,24 +1052,32 @@
       camera_frame_name="${namespace}/servo_camera_optical"
       sensor_base_frame_name="${namespace}/servo_camera"
-      offset_x="0.2278"
-      offset_y="0.0"
-      offset_z="-0.1378"
-      offset_roll="0.0"
-      offset_yaw="0.0"
-      offset_pitch="0.0"
-      pitch_update_rate="5.0"
-      min_pitch="-1.046"
+      offset_pitch_link_x="0.0"
+      offset_pitch_link_y="0.0"
+      offset_pitch_link_z="0.0"
+      offset_pitch_link_roll="0.0"
+      offset_pitch_link_yaw="0.0"
+      offset_pitch_link_pitch="0.0"
+      offset_roll_link_x="0.2"
+      offset_roll_link_y="0.0"
+      offset_roll_link_z="-0.1"
+      offset_roll_link_roll="0.0"
+      offset_roll_link_yaw="0.0"
+      offset_roll_link_pitch="0.0"
+      tilt_update_rate="5.0"
+      min_pitch="-1.57"
       max_pitch="1.57"
+      min_roll="-0.6"
+      max_roll="0.6"
       max_pitch_rate="0.1"
+      max_roll_rate="0.1"
       camera_update_rate="30"
       horizontal_fov="1.92"
       img_width="1920"
       img_height="1080"
-      compensate_tilt="true">
-      <visual>
-        <geometry>
-          <box size="0.01 0.01 0.01" />
-        </geometry>
-      </visual>
+      compensate_tilt_roll="true"
+      compensate_tilt_pitch="true"
+      pitch_link_mesh_file=""
+      roll_link_mesh_file=""
+      mesh_scale="">
     </xacro:servo_camera_macro>
   </xacro:if>

File: models/mrs_robots_description/urdf/naki.xacro (robot description, xacro)
@@ -79,4 +79,5 @@
   <xacro:property name="prop_mesh_file" value="package://mrs_robots_description/meshes/custom/naki/NAKI_propeller.dae"/>
   <xacro:property name="sony_camera_mesh_file" value="package://mrs_robots_description/meshes/custom/naki/NAKI_sony_alpha_6500_w_gimbal_mount.dae"/>
+  <xacro:property name="gimbal_mesh_file" value="package://mrs_robots_description/meshes/custom/naki/NAKI_gimbal_movable_part.dae"/>
   <xacro:property name="pixhawk_mesh_file" value="package://mrs_robots_description/meshes/sensors/pixhawk.dae" />
   <!-- scales -->
@@ -780,24 +781,32 @@
     camera_frame_name="${namespace}/servo_camera_optical"
     sensor_base_frame_name="${namespace}/servo_camera"
-    offset_x="0.22597"
-    offset_y="0.00208"
-    offset_z="-0.1366"
-    offset_roll="0.0"
-    offset_yaw="0.0"
-    offset_pitch="0.0"
-    pitch_update_rate="5.0"
+    offset_pitch_link_x="0.12928"
+    offset_pitch_link_y="7.605e-5"
+    offset_pitch_link_z="-0.006051"
+    offset_pitch_link_roll="0.0"
+    offset_pitch_link_yaw="0.0"
+    offset_pitch_link_pitch="0.0"
+    offset_roll_link_x="0.0966901"
+    offset_roll_link_y="0.00200395"
+    offset_roll_link_z="-0.130549"
+    offset_roll_link_roll="0.0"
+    offset_roll_link_yaw="0.0"
+    offset_roll_link_pitch="0.0"
+    tilt_update_rate="5.0"
     min_pitch="-1.046"
     max_pitch="1.57"
-    max_pitch_rate="0.1"
+    min_roll="-0.6"
+    max_roll="0.6"
+    max_pitch_rate="0.2"
+    max_roll_rate="0.2"
     camera_update_rate="30"
     horizontal_fov="1.92"
     img_width="1920"
     img_height="1080"
-    compensate_tilt="true">
-    <visual>
-      <geometry>
-        <mesh filename="${sony_camera_mesh_file}" scale="${mesh_scale}" />
-      </geometry>
-    </visual>
+    compensate_tilt_roll="true"
+    compensate_tilt_pitch="true"
+    pitch_link_mesh_file="${sony_camera_mesh_file}"
+    roll_link_mesh_file="${gimbal_mesh_file}"
+    mesh_scale="${mesh_scale}">
   </xacro:servo_camera_macro>
   <!--}-->

File: models/mrs_robots_description/urdf/t650.xacro (robot description, xacro)
@@ -925,24 +925,32 @@
       camera_frame_name="${namespace}/servo_camera_optical"
       sensor_base_frame_name="${namespace}/servo_camera"
-      offset_x="0.2"
-      offset_y="0.0"
-      offset_z="-0.1"
-      offset_roll="0.0"
-      offset_yaw="0.0"
-      offset_pitch="0.0"
-      pitch_update_rate="5.0"
-      min_pitch="-1.046"
+      offset_pitch_link_x="0.0"
+      offset_pitch_link_y="0.0"
+      offset_pitch_link_z="0.0"
+      offset_pitch_link_roll="0.0"
+      offset_pitch_link_yaw="0.0"
+      offset_pitch_link_pitch="0.0"
+      offset_roll_link_x="0.2"
+      offset_roll_link_y="0.0"
+      offset_roll_link_z="-0.1"
+      offset_roll_link_roll="0.0"
+      offset_roll_link_yaw="0.0"
+      offset_roll_link_pitch="0.0"
+      tilt_update_rate="5.0"
+      min_pitch="-1.57"
       max_pitch="1.57"
+      min_roll="-0.6"
+      max_roll="0.6"
       max_pitch_rate="0.1"
+      max_roll_rate="0.1"
       camera_update_rate="30"
       horizontal_fov="1.92"
       img_width="1920"
       img_height="1080"
-      compensate_tilt="true">
-      <visual>
-        <geometry>
-          <box size="0.01 0.01 0.01" />
-        </geometry>
-      </visual>
+      compensate_tilt_roll="true"
+      compensate_tilt_pitch="true"
+      pitch_link_mesh_file=""
+      roll_link_mesh_file=""
+      mesh_scale="">
     </xacro:servo_camera_macro>
   </xacro:if>

Commit message: update camera lens to 140deg

File: models/mrs_robots_description/urdf/component_snippets.xacro (robot description, xacro)
@@ -40,7 +40,9 @@
   <xacro:property name="rad120" value="${120*pi/180}" />
   <xacro:property name="rad135" value="${135*pi/180}" />
+  <xacro:property name="rad140" value="${140*pi/180}" />
   <xacro:property name="rad150" value="${150*pi/180}" />
   <xacro:property name="rad180" value="${180*pi/180}" />
   <xacro:property name="rad210" value="${210*pi/180}" />
+  <xacro:property name="rad315" value="${315*pi/180}" />
   <xacro:property name="sin30" value="${sin(rad30)}" />
   <xacro:property name="sin45" value="${sin(rad45)}" />
@@ -2652,4 +2654,47 @@
   </xacro:macro>
   <!--}-->
+  <!-- Macro to add a Fisheye 120deg Pylon camera {-->
+  <xacro:macro name="fisheye_camera_pylon_macro"
+    params="namespace parent_link camera_suffix frame_rate noise x y z roll pitch yaw camera_frame_name sensor_base_frame_name parent_frame_name">
+    <xacro:fisheye_macro
+      namespace="${namespace}"
+      parent_link="${parent_link}"
+      camera_suffix="${camera_suffix}"
+      camera_frame_name="${camera_frame_name}"
+      sensor_base_frame_name="${sensor_base_frame_name}"
+      frame_rate="${frame_rate}"
+      horizontal_fov="${rad140}"
+      image_width="1600"
+      image_height="1200"
+      lens_type="custom"
+      lens_c1="1.05"
+      lens_c2="4"
+      lens_f="1.0"
+      lens_fun="tan"
+      lens_scale="true"
+      lens_cutoff_angle="${rad140}"
+      lens_texture_size="512"
+      min_distance="0.02"
+      max_distance="40"
+      noise_mean="0.0"
+      noise_stddev="${noise}"
+      parent_frame_name="${parent_frame_name}"
+      x="${x}"
+      y="${y}"
+      z="${z}"
+      yaw="${yaw}"
+      pitch="${pitch}"
+      roll="${roll}"
+      >
+      <visual>
+        <origin xyz="0 0 0" rpy="${rad90} 0 0" />
+        <geometry>
+          <mesh filename="package://mrs_robots_description/meshes/sensors/bluefox.dae"
+            scale="1 1 1" />
+        </geometry>
+      </visual>
+    </xacro:fisheye_macro>
+  </xacro:macro>
+  <!--}-->
   <!-- ================================================================== -->
   <!-- ||         other equipment definitions (holders, boxes ...)     || -->

File: models/mrs_robots_description/urdf/f450.xacro (robot description, xacro)
@@ -1040,4 +1040,42 @@
   </xacro:if>
   <!--}-->
+  <!-- Basler stereopair {-->
+  <xacro:if value="${optionals['enable_basler_stereopair']}">
+    <xacro:fisheye_camera_pylon_macro
+      namespace="${namespace}"
+      parent_link="base_link"
+      camera_suffix="fleft"
+      frame_rate="40"
+      noise="0.000"
+      parent_frame_name="${namespace}/basler_stereopair/base"
+      camera_frame_name="${namespace}/basler_left_optical"
+      sensor_base_frame_name="${namespace}/basler_left"
+      x="0.083"
+      y="0.083"
+      z="${arm_height + 0.2}"
+      roll="0.0"
+      pitch="0.0"
+      yaw="${rad45}"
+      >
+    </xacro:fisheye_camera_pylon_macro>
+    <xacro:fisheye_camera_pylon_macro
+      namespace="${namespace}"
+      parent_link="base_link"
+      camera_suffix="fright"
+      frame_rate="40"
+      noise="0.000"
+      parent_frame_name="${namespace}/basler_stereopair/base"
+      camera_frame_name="${namespace}/basler_right_optical"
+      sensor_base_frame_name="${namespace}/basler_rigth"
+      x="0.083"
+      y="-0.083"
+      z="${arm_height + 0.2}"
+      roll="0.0"
+      pitch="0.0"
+      yaw="${rad315}"
+      >
+    </xacro:fisheye_camera_pylon_macro>
+  </xacro:if>
+  <!--}-->
   <!-- ========================== other sensors ========================= -->
   <!-- Teraranger Tower Evo {-->
