Commit message: updated f330 motor params

File: models/mrs_robots_description/urdf/f330.xacro (robot description, xacro)
@@ -37,5 +37,5 @@
   <!-- ================================================================== -->
   <!-- Robot parameters and arguments {-->
-  <xacro:property name="mass" value="2.00" /> <!-- [kg] -->
+  <xacro:property name="mass" value="1.35" /> <!-- [kg] -->
   <xacro:property name="body_radius" value="0.08" /> <!-- [m] -->
   <xacro:property name="body_height" value="0.07" /> <!-- [m] -->
@@ -56,5 +56,5 @@
   <!-- Motor constants {-->
   <xacro:property name="rotor_velocity_slowdown_sim" value="0.0159236" />
-  <xacro:property name="motor_constant" value="8.5" /> <!-- [kg.m/s^2] -->
+  <xacro:property name="motor_constant" value="8.91" /> <!-- [kg.m/s^2] -->
   <xacro:property name="moment_constant" value="0.016" /> <!-- [m] -->
   <xacro:property name="time_constant_up" value="${1.0 / 80.0}" /> <!-- [s] -->

Commit message: fixed mavros launch file and px4 RC loss error

File: models/mrs_robots_description/urdf/f330.xacro (robot description, xacro)
@@ -7,5 +7,5 @@
   <xacro:property name="namespace" value="$(arg namespace)" />
   <xacro:property name='model_config_file' value="$(arg model_config_file)"/>
-  <xacro:property name="optionals" value="${load_yaml(model_config_file)}" />
+  <xacro:property name="optionals" value="${xacro.load_yaml(model_config_file)}" />
   <xacro:arg name='name' default='f330' />
   <xacro:arg name='mavlink_addr' default='INADDR_ANY' />

File: models/mrs_robots_description/urdf/f450.xacro (robot description, xacro)
@@ -7,5 +7,5 @@
   <xacro:property name="namespace" value="$(arg namespace)" />
   <xacro:property name='model_config_file' value="$(arg model_config_file)"/>
-  <xacro:property name="optionals" value="${load_yaml(model_config_file)}" />
+  <xacro:property name="optionals" value="${xacro.load_yaml(model_config_file)}" />
   <xacro:arg name='name' default='f450' />
   <xacro:arg name='mavlink_addr' default='INADDR_ANY' />

File: models/mrs_robots_description/urdf/f550.xacro (robot description, xacro)
@@ -7,5 +7,5 @@
   <xacro:property name="namespace" value="$(arg namespace)" />
   <xacro:property name='model_config_file' value="$(arg model_config_file)"/>
-  <xacro:property name="optionals" value="${load_yaml(model_config_file)}" />
+  <xacro:property name="optionals" value="${xacro.load_yaml(model_config_file)}" />
   <xacro:arg name='name' default='f550' />
   <xacro:arg name='mavlink_addr' default='INADDR_ANY' />

File: models/mrs_robots_description/urdf/naki.xacro (robot description, xacro)
@@ -7,5 +7,5 @@
   <xacro:property name="namespace" value="$(arg namespace)" />
   <xacro:property name='model_config_file' value="$(arg model_config_file)"/>
-  <xacro:property name="optionals" value="${load_yaml(model_config_file)}" />
+  <xacro:property name="optionals" value="${xacro.load_yaml(model_config_file)}" />
   <xacro:arg name='name' default='naki' />
   <xacro:arg name='mavlink_addr' default='INADDR_ANY' />

File: models/mrs_robots_description/urdf/t650.xacro (robot description, xacro)
@@ -7,5 +7,5 @@
   <xacro:property name="namespace" value="$(arg namespace)" />
   <xacro:property name='model_config_file' value="$(arg model_config_file)"/>
-  <xacro:property name="optionals" value="${load_yaml(model_config_file)}" />
+  <xacro:property name="optionals" value="${xacro.load_yaml(model_config_file)}" />
   <xacro:arg name='name' default='t650' />
   <xacro:arg name='mavlink_addr' default='INADDR_ANY' />

File: models/mrs_robots_description/urdf/x500.xacro (robot description, xacro)
@@ -7,5 +7,5 @@
   <xacro:property name="namespace" value="$(arg namespace)" />
   <xacro:property name='model_config_file' value="$(arg model_config_file)"/>
-  <xacro:property name="optionals" value="${load_yaml(model_config_file)}" />
+  <xacro:property name="optionals" value="${xacro.load_yaml(model_config_file)}" />
   <xacro:arg name='name' default='x500' />
   <xacro:arg name='mavlink_addr' default='INADDR_ANY' />

Commit message: added enable-vio-down spawn param for downward-facing bluefox camera with imu

File: models/mrs_robots_description/urdf/f330.xacro (robot description, xacro)
@@ -620,6 +620,51 @@
       <origin xyz="0 0 0" rpy="0 0 ${-rad90}" />
     </xacro:visual_macro>
-  <!--}-->
   </xacro:if>
+  <!--}-->
+  <!-- fisheye down with imu {-->
+  <xacro:if value="${optionals['enable_vio_down']}">
+    <xacro:vio_macro
+      namespace="${namespace}"
+      parent_link="base_link"
+      parent_frame_name="${namespace}/fcu"
+      camera_frame_name="${namespace}/fisheye_camera_optical"
+      sensor_base_frame_name="${namespace}/fisheye_camera"
+      frame_rate="45"
+      horizontal_fov="${rad180}"
+      image_width="752"
+      image_height="480"
+      lens_type="custom"
+      lens_c1="1.05"
+      lens_c2="4"
+      lens_f="1.0"
+      lens_fun="tan"
+      lens_scale="true"
+      lens_cutoff_angle="${rad90}"
+      lens_texture_size="512"
+      min_distance="0.02"
+      max_distance="40"
+      camera_noise_mean="0.0"
+      x="0.107"
+      y="0"
+      z="-0.002"
+      roll="0"
+      pitch="${rad90}"
+      yaw="0.0"
+      imu_rate="125.0"
+      imu_topic="vio/imu"
+      imu_noise_mean="0.0"
+      >
+    </xacro:vio_macro>
+    <xacro:visual_macro
+      robot_namespace="${namespace}"
+      name="bluefox_mount"
+      mesh_file="${bluefox_mount_mesh}"
+      mesh_scale="${mesh_scale}"
+      parent="base_link"
+      color="Black">
+      <origin xyz="0 0 0" rpy="0 0 ${-rad90}" />
+    </xacro:visual_macro>
+  </xacro:if>
+  <!--}-->
   <!--} VIO -->
 </robot>

File: models/mrs_robots_description/urdf/f450.xacro (robot description, xacro)
@@ -1342,3 +1342,95 @@
 </xacro:if>
 <!--}-->
+  <!-- VIO {-->
+  <!-- fisheye forward with imu {-->
+  <xacro:if value="${optionals['enable_vio']}">
+    <xacro:vio_macro
+      namespace="${namespace}"
+      parent_link="base_link"
+      parent_frame_name="${namespace}/fcu"
+      camera_frame_name="${namespace}/fisheye_camera_optical"
+      sensor_base_frame_name="${namespace}/fisheye_camera"
+      frame_rate="45"
+      horizontal_fov="${rad180}"
+      image_width="752"
+      image_height="480"
+      lens_type="custom"
+      lens_c1="1.05"
+      lens_c2="4"
+      lens_f="1.0"
+      lens_fun="tan"
+      lens_scale="true"
+      lens_cutoff_angle="${rad90}"
+      lens_texture_size="512"
+      min_distance="0.02"
+      max_distance="40"
+      camera_noise_mean="0.0"
+      x="0.107"
+      y="0"
+      z="-0.002"
+      roll="0"
+      pitch="0"
+      yaw="0.0"
+      imu_rate="125.0"
+      imu_topic="vio/imu"
+      imu_noise_mean="0.0"
+      >
+    </xacro:vio_macro>
+    <!-- <xacro:visual_macro -->
+    <!--   robot_namespace="${namespace}" -->
+    <!--   name="bluefox_mount_vio" -->
+    <!--   mesh_file="${bluefox_mount_mesh}" -->
+    <!--   mesh_scale="${mesh_scale}" -->
+    <!--   parent="base_link" -->
+    <!--   color="Black"> -->
+    <!--   <origin xyz="0 0 0" rpy="0 0 ${-rad90}" /> -->
+    <!-- </xacro:visual_macro> -->
+  </xacro:if>
+  <!--}-->
+  <!-- fisheye down with imu {-->
+  <xacro:if value="${optionals['enable_vio_down']}">
+    <xacro:vio_macro
+      namespace="${namespace}"
+      parent_link="base_link"
+      parent_frame_name="${namespace}/fcu"
+      camera_frame_name="${namespace}/fisheye_camera_optical"
+      sensor_base_frame_name="${namespace}/fisheye_camera"
+      frame_rate="45"
+      horizontal_fov="${rad180}"
+      image_width="752"
+      image_height="480"
+      lens_type="custom"
+      lens_c1="1.05"
+      lens_c2="4"
+      lens_f="1.0"
+      lens_fun="tan"
+      lens_scale="true"
+      lens_cutoff_angle="${rad90}"
+      lens_texture_size="512"
+      min_distance="0.02"
+      max_distance="40"
+      camera_noise_mean="0.0"
+      x="0.1"
+      y="0"
+      z="-0.15"
+      roll="0"
+      pitch="${rad90}"
+      yaw="0.0"
+      imu_rate="125.0"
+      imu_topic="vio/imu"
+      imu_noise_mean="0.0"
+      >
+    </xacro:vio_macro>
+    <!-- <xacro:visual_macro -->
+    <!--   robot_namespace="${namespace}" -->
+    <!--   name="bluefox_mount" -->
+    <!--   mesh_file="${bluefox_mount_mesh}" -->
+    <!--   mesh_scale="${mesh_scale}" -->
+    <!--   parent="base_link" -->
+    <!--   color="Black"> -->
+    <!--   <origin xyz="0 0 0" rpy="0 0 ${-rad90}" /> -->
+    <!-- </xacro:visual_macro> -->
+  </xacro:if>
+  <!--}-->
+  <!--} VIO -->
 </robot>
