Commit message: Adding spawning parameters for the beacon

File: models/mrs_robots_description/urdf/f450.xacro (robot description, xacro)
@@ -1051,8 +1051,51 @@
   </xacro:macro>
   <!--}-->
+  <!-- UV led - beacon configuration {-->
+        <xacro:macro name="uvled_beacon"
+          params="height f namespace parent_link">
+          <!-- UV LED -->
+          <xacro:uvled_macro
+            namespace="${namespace}"
+            parent_link="base_link"
+            number="b1"
+            frequency="${f}">
+            <origin xyz="0.01 0 ${height}-0.05" rpy="0 1.57079632679 0" />
+          </xacro:uvled_macro>
+          <xacro:uvled_macro
+            namespace="${namespace}"
+            parent_link="base_link"
+            number="b2"
+            frequency="${f}">
+            <origin xyz="0 0.01 ${height}-0.05" rpy="0 1.57079632679 1.5708" />
+          </xacro:uvled_macro>
+          <xacro:uvled_macro
+            namespace="${namespace}"
+            parent_link="base_link"
+            number="b3"
+            frequency="${f}">
+            <origin xyz="-0.01 0 ${height}-0.05" rpy="0 1.57079632679 3.14159265359" />
+          </xacro:uvled_macro>
+          <xacro:uvled_macro
+            namespace="${namespace}"
+            parent_link="base_link"
+            number="b4"
+            frequency="${f}">
+            <origin xyz="0 -0.01 ${height}-0.05" rpy="0 1.57079632679 -1.5708" />
+          </xacro:uvled_macro>
+        </xacro:macro>
+  <!--}-->
   <xacro:if value="$(arg enable_uv_leds)">
     <xacro:uvled_quadrotor
       f1="$(arg uvled_fr_l)"
       f2="$(arg uvled_fr_r)"
+      namespace="${namespace}"
+      parent_link="base_link"/>
+  </xacro:if>
+  <!--}-->
+  <!-- UV led beacon {-->
+  <xacro:if value="$(arg enable_uv_leds_beacon)">
+    <xacro:uvled_beacon
+      height="$(arg uvled_beacon_height)"
+      f="$(arg uvled_beacon_f)"
       namespace="${namespace}"
       parent_link="base_link"/>

Commit message: Fixing the height of the beacon - I didn't know that SDF does not support in-string position arithmetic

File: models/mrs_robots_description/urdf/f450.xacro (robot description, xacro)
@@ -1060,5 +1060,5 @@
             number="b1"
             frequency="${f}">
-            <origin xyz="0.01 0 ${height}-0.05" rpy="0 1.57079632679 0" />
+            <origin xyz="0.01 0 ${height}" rpy="0 1.57079632679 0" />
           </xacro:uvled_macro>
           <xacro:uvled_macro
@@ -1067,5 +1067,5 @@
             number="b2"
             frequency="${f}">
-            <origin xyz="0 0.01 ${height}-0.05" rpy="0 1.57079632679 1.5708" />
+            <origin xyz="0 0.01 ${height}" rpy="0 1.57079632679 1.5708" />
           </xacro:uvled_macro>
           <xacro:uvled_macro
@@ -1074,5 +1074,5 @@
             number="b3"
             frequency="${f}">
-            <origin xyz="-0.01 0 ${height}-0.05" rpy="0 1.57079632679 3.14159265359" />
+            <origin xyz="-0.01 0 ${height}" rpy="0 1.57079632679 3.14159265359" />
           </xacro:uvled_macro>
           <xacro:uvled_macro
@@ -1081,5 +1081,5 @@
             number="b4"
             frequency="${f}">
-            <origin xyz="0 -0.01 ${height}-0.05" rpy="0 1.57079632679 -1.5708" />
+            <origin xyz="0 -0.01 ${height}" rpy="0 1.57079632679 -1.5708" />
           </xacro:uvled_macro>
         </xacro:macro>

Commit message: fixed naming of new parameter for uvled_beacon and polished code

File: models/mrs_robots_description/urdf/f450.xacro (robot description, xacro)
@@ -1051,38 +1051,4 @@
   </xacro:macro>
   <!--}-->
-  <!-- UV led - beacon configuration {-->
-        <xacro:macro name="uvled_beacon"
-          params="height f namespace parent_link">
-          <!-- UV LED -->
-          <xacro:uvled_macro
-            namespace="${namespace}"
-            parent_link="base_link"
-            number="b1"
-            frequency="${f}">
-            <origin xyz="0.01 0 ${height}" rpy="0 1.57079632679 0" />
-          </xacro:uvled_macro>
-          <xacro:uvled_macro
-            namespace="${namespace}"
-            parent_link="base_link"
-            number="b2"
-            frequency="${f}">
-            <origin xyz="0 0.01 ${height}" rpy="0 1.57079632679 1.5708" />
-          </xacro:uvled_macro>
-          <xacro:uvled_macro
-            namespace="${namespace}"
-            parent_link="base_link"
-            number="b3"
-            frequency="${f}">
-            <origin xyz="-0.01 0 ${height}" rpy="0 1.57079632679 3.14159265359" />
-          </xacro:uvled_macro>
-          <xacro:uvled_macro
-            namespace="${namespace}"
-            parent_link="base_link"
-            number="b4"
-            frequency="${f}">
-            <origin xyz="0 -0.01 ${height}" rpy="0 1.57079632679 -1.5708" />
-          </xacro:uvled_macro>
-        </xacro:macro>
-  <!--}-->
   <xacro:if value="$(arg enable_uv_leds)">
     <xacro:uvled_quadrotor
@@ -1094,4 +1060,38 @@
   <!--}-->
   <!-- UV led beacon {-->
+  <!-- UV led - beacon configuration {-->
+  <xacro:macro name="uvled_beacon"
+    params="height f namespace parent_link">
+    <!-- UV LED -->
+    <xacro:uvled_macro
+      namespace="${namespace}"
+      parent_link="base_link"
+      number="b1"
+      frequency="${f}">
+      <origin xyz="0.01 0 ${height}" rpy="0 ${rad90} 0" />
+    </xacro:uvled_macro>
+    <xacro:uvled_macro
+      namespace="${namespace}"
+      parent_link="base_link"
+      number="b2"
+      frequency="${f}">
+      <origin xyz="0 0.01 ${height}" rpy="0 ${rad90} ${rad90}" />
+    </xacro:uvled_macro>
+    <xacro:uvled_macro
+      namespace="${namespace}"
+      parent_link="base_link"
+      number="b3"
+      frequency="${f}">
+      <origin xyz="-0.01 0 ${height}" rpy="0 ${rad90} ${rad180}" />
+    </xacro:uvled_macro>
+    <xacro:uvled_macro
+      namespace="${namespace}"
+      parent_link="base_link"
+      number="b4"
+      frequency="${f}">
+      <origin xyz="0 -0.01 ${height}" rpy="0 ${rad90} -${rad90}" />
+    </xacro:uvled_macro>
+  </xacro:macro>
+  <!--}-->
   <xacro:if value="$(arg enable_uv_leds_beacon)">
     <xacro:uvled_beacon

Commit message: towards spawner node

File: models/mrs_robots_description/urdf/f450.xacro (robot description, xacro)
@@ -6,4 +6,6 @@
   -->
   <xacro:property name="namespace" value="$(arg namespace)" />
+  <xacro:property name='model_params_file' value="$(arg model_params_file)"/>
+  <xacro:property name="optionals" value="${load_yaml(model_params_file)}" />
   <xacro:arg name='name' default='f450' />
   <xacro:arg name='mavlink_addr' default='INADDR_ANY' />
@@ -509,5 +511,5 @@
   <!-- ================================================================== -->
   <!-- Ground truth {-->
-  <xacro:if value="$(arg enable_ground_truth)">
+  <xacro:if value="${optionals['enable_ground_truth']}">
     <!-- Mount a generic odometry sensor providing ground truth. -->
     <xacro:odometry_plugin_macro
@@ -529,5 +531,5 @@
   <!-- ======================= rangefinder sensors ======================-->
   <!-- Garmin {-->
-  <xacro:if value="$(arg enable_rangefinder)">
+  <xacro:if value="${optionals['enable_rangefinder']}">
     <xacro:garmin_macro
       namespace="${namespace}"
@@ -545,5 +547,5 @@
   <!--}-->
   <!-- Garmin looking up {-->
-  <xacro:if value="$(arg enable_rangefinder_up)">
+  <xacro:if value="${optionals['enable_rangefinder_up']}">
     <xacro:garmin_macro
       namespace="${namespace}"
@@ -561,5 +563,5 @@
   <!--}-->
   <!-- Teraranger One {-->
-  <xacro:if value="$(arg enable_teraranger)">
+  <xacro:if value="${optionals['enable_teraranger']}">
     <xacro:teraranger_macro
       namespace="${namespace}"
@@ -577,5 +579,5 @@
   <!-- ========================== LIDAR sensors ========================= -->
   <!-- Scanse Sweep {-->
-  <xacro:if value="$(arg enable_scanse_sweep)">
+  <xacro:if value="${optionals['enable_scanse_sweep']}">
     <xacro:scanse_sweep_macro
       namespace="${namespace}"
@@ -591,5 +593,5 @@
   <!--}-->
   <!-- Rplidar {-->
-  <xacro:if value="$(arg enable_rplidar)">
+  <xacro:if value="${optionals['enable_rplidar']}">
     <xacro:rplidar_macro
       namespace="${namespace}"
@@ -605,5 +607,5 @@
   <!--}-->
   <!-- Velodyne  {-->
-  <xacro:if value="$(arg enable_velodyne)">
+  <xacro:if value="${optionals['enable_velodyne']}">
     <!-- VLP-16 (default) -->
     <xacro:property name="sensor_name" value="velodyne" />
@@ -631,5 +633,5 @@
   <!--}-->
   <!-- Ouster {-->
-  <xacro:if value="$(arg enable_ouster)">
+  <xacro:if value="${optionals['enable_ouster']}">
   <xacro:property name="ouster_model" value="$(arg ouster_model)" />
     <!-- OS1-16 Generation 1 (default) -->
@@ -735,5 +737,5 @@
   <!-- Fisheye camera placements{-->
   <!-- classic {-->
-  <xacro:if value="$(arg enable_fisheye_camera)">
+  <xacro:if value="${optionals['enable_fisheye_camera']}">
     <xacro:fisheye_camera_macro
       namespace="${namespace}"
@@ -758,5 +760,5 @@
   <!-- Bluefox placements{-->
   <!-- reverse {-->
-  <xacro:if value="$(arg enable_bluefox_camera_reverse)">
+  <xacro:if value="${optionals['enable_bluefox_camera_reverse']}">
     <xacro:bluefox_camera_macro
       namespace="${namespace}"
@@ -780,5 +782,5 @@
   <!--}-->
   <!-- classic {-->
-  <xacro:if value="$(arg enable_bluefox_camera)">
+  <xacro:if value="${optionals['enable_bluefox_camera']}">
     <xacro:bluefox_camera_macro
       namespace="${namespace}"
@@ -804,5 +806,5 @@
   <!-- Realsense placements {-->
   <!-- down {-->
-  <xacro:if value="$(arg enable_realsense_down)">
+  <xacro:if value="${optionals['enable_realsense_down']}">
     <!-- sensor -->
     <xacro:realsense_macro
@@ -822,5 +824,5 @@
   <!--}-->
   <!-- front pitched {-->
-  <xacro:if value="$(arg enable_realsense_front_pitched)">
+  <xacro:if value="${optionals['enable_realsense_front_pitched']}">
     <!-- sensor -->
     <xacro:realsense_macro
@@ -840,5 +842,5 @@
   <!--}-->
   <!-- front {-->
-  <xacro:if value="$(arg enable_realsense_front)">
+  <xacro:if value="${optionals['enable_realsense_front']}">
     <!-- sensor -->
     <xacro:realsense_macro
@@ -858,5 +860,5 @@
   <!--}-->
   <!-- up {-->
-  <xacro:if value="$(arg enable_realsense_up)">
+  <xacro:if value="${optionals['enable_realsense_up']}">
     <!-- sensor -->
     <xacro:realsense_macro
@@ -878,5 +880,5 @@
   <!-- Mobius placements {-->
   <!-- down {-->
-  <xacro:if value="$(arg enable_mobius_camera_down)">
+  <xacro:if value="${optionals['enable_mobius_camera_down']}">
     <xacro:mobius_camera_macro
       namespace="${namespace}"
@@ -898,5 +900,5 @@
   <!--}-->
   <!-- front {-->
-  <xacro:if value="$(arg enable_mobius_camera_front)">
+  <xacro:if value="${optionals['enable_mobius_camera_front']}">
     <xacro:mobius_camera_macro
       namespace="${namespace}"
@@ -918,5 +920,5 @@
   <!--}-->
   <!-- back left {-->
-  <xacro:if value="$(arg enable_mobius_camera_back_left)">
+  <xacro:if value="${optionals['enable_mobius_camera_back_left']}">
     <xacro:mobius_camera_macro
       namespace="${namespace}"
@@ -938,5 +940,5 @@
   <!--}-->
   <!-- back right {-->
-  <xacro:if value="$(arg enable_mobius_camera_back_right)">
+  <xacro:if value="${optionals['enable_mobius_camera_back_right']}">
     <xacro:mobius_camera_macro
       namespace="${namespace}"
@@ -959,5 +961,5 @@
   <!--} Mobius placements -->
   <!-- UV camera {-->
-  <xacro:if value="$(arg enable_uv_camera)">
+  <xacro:if value="${optionals['enable_uv_camera']}">
     <xacro:uvcam_macro
       namespace="${namespace}"
@@ -983,5 +985,5 @@
   <!--}-->
   <!-- Servo camera {-->
-  <xacro:if value="$(arg enable_servo_camera)">
+  <xacro:if value="${optionals['enable_servo_camera']}">
     <xacro:servo_camera_macro
       namespace="${namespace}"
@@ -1002,5 +1004,5 @@
   <!-- ========================== other sensors ========================= -->
   <!-- Teraranger Tower Evo {-->
-  <xacro:if value="$(arg enable_teraranger_tower_evo)">
+  <xacro:if value="${optionals['enable_teraranger_tower_evo']}">
     <xacro:teraranger_tower_evo_macro
       namespace="${namespace}"
@@ -1014,5 +1016,5 @@
   <!--}-->
   <!-- Magnetic gripper {-->
-  <xacro:if value="$(arg enable_magnetic_gripper)">
+  <xacro:if value="${optionals['enable_magnetic_gripper']}">
     <xacro:magnet_gripper_macro
       namespace="${namespace}"
@@ -1025,5 +1027,5 @@
   <!--}-->
   <!-- Timepix {-->
-  <xacro:if value="$(arg enable_timepix)">
+  <xacro:if value="${optionals['enable_timepix']}">
     <xacro:timepix_macro
       namespace="${namespace}"
@@ -1098,5 +1100,5 @@
   </xacro:macro>
   <!--}-->
-  <xacro:if value="$(arg enable_uv_leds)">
+  <xacro:if value="${optionals['enable_uv_leds']}">
     <xacro:uvled_quadrotor
       f1="$(arg uvled_fr_l)"
@@ -1141,5 +1143,5 @@
   </xacro:macro>
   <!--}-->
-  <xacro:if value="$(arg enable_uv_leds_beacon)">
+  <xacro:if value="${optionals['enable_uv_leds_beacon']}">
     <xacro:uvled_beacon
       height="0.15"
@@ -1150,5 +1152,5 @@
   <!--}-->
   <!-- Light {-->
-  <xacro:if value="$(arg enable_light)">
+  <xacro:if value="${optionals['enable_light']}">
     <xacro:light_macro
       namespace="${namespace}"
@@ -1172,5 +1174,5 @@
   <!-- ============================= holders ============================ -->
   <!-- Ouster and Velodyne mount {-->
-  <xacro:if value="${('$(arg enable_ouster)' == 'true') or ('$(arg enable_velodyne)' == 'true')}">
+  <xacro:if value="${(optionals['enable_ouster'] == 'true') or (optionals['enable_velodyne'] == 'true')}">
     <xacro:visual_macro
       robot_namespace="${namespace}"
@@ -1185,5 +1187,5 @@
   <!--}-->
   <!-- Rplidar and scanse mount {-->
-  <xacro:if value="${('$(arg enable_rplidar)' == 'true') or ('$(arg enable_scanse_sweep)' == 'true')}">
+  <xacro:if value="${(optionals['enable_rplidar'] == 'true') or (optionals['enable_scanse_sweep'] == 'true')}">
     <xacro:visual_macro
       robot_namespace="${namespace}"
@@ -1198,5 +1200,5 @@
   <!--}-->
   <!-- Garmin mount {-->
-  <xacro:if value="$(arg enable_rangefinder)">
+  <xacro:if value="${optionals['enable_rangefinder']}">
     <xacro:visual_macro
       robot_namespace="${namespace}"
@@ -1211,5 +1213,5 @@
   <!--}-->
   <!-- Bluefox mount {-->
-  <xacro:if value="$(arg enable_rangefinder)">
+  <xacro:if value="${optionals['enable_rangefinder']}">
     <xacro:visual_macro
       robot_namespace="${namespace}"
@@ -1224,5 +1226,5 @@
   <!--}-->
   <!-- Realsense front mount {-->
-  <xacro:if value="$(arg enable_realsense_front)">
+  <xacro:if value="${optionals['enable_realsense_front']}">
     <xacro:visual_macro
       robot_namespace="${namespace}"
@@ -1237,5 +1239,5 @@
   <!--}-->
   <!-- Realsense front pitched mount {-->
-  <xacro:if value="$(arg enable_realsense_front_pitched)">
+  <xacro:if value="${optionals['enable_realsense_front_pitched']}">
     <xacro:visual_macro
       robot_namespace="${namespace}"
@@ -1250,5 +1252,5 @@
   <!--}-->
   <!-- Realsense down mount {-->
-  <xacro:if value="$(arg enable_realsense_down)">
+  <xacro:if value="${optionals['enable_realsense_down']}">
     <xacro:visual_macro
       robot_namespace="${namespace}"
@@ -1263,5 +1265,5 @@
   <!--}-->
   <!-- UVDAR mount {-->
-  <xacro:if value="$(arg enable_uv_camera)">
+  <xacro:if value="${optionals['enable_uv_camera']}">
     <xacro:visual_macro
       robot_namespace="${namespace}"
@@ -1277,5 +1279,5 @@
   <!-- ========================== other sensors ========================= -->
   <!-- Whycon box {-->
-  <xacro:if value="$(arg enable_whycon_box)">
+  <xacro:if value="${optionals['enable_whycon_box']}">
     <xacro:box_macro
       robot_namespace="${namespace}"
@@ -1289,5 +1291,5 @@
   <!--}-->
   <!-- Pendulum {-->
-  <xacro:if value="$(arg enable_pendulum)">
+  <xacro:if value="${optionals['enable_pendulum']}">
     <xacro:pendulum
       parent="base_link">
