Commit message: working f550, despawning still ends in segfaults (I blame plugins used by px4)

File: models/mrs_robots_description/urdf/f450.xacro (robot description, xacro)
@@ -627,5 +627,5 @@
       max_range="${range}"
       noise="0.01"
-      enable_gpu_ray="$(arg use_gpu_ray)"
+      enable_gpu_ray="${optionals['use_gpu_ray']}"
       >
     </xacro:velodyne_macro>
@@ -634,5 +634,5 @@
   <!-- Ouster {-->
   <xacro:if value="${optionals['enable_ouster']}">
-  <xacro:property name="ouster_model" value="$(arg ouster_model)" />
+    <xacro:property name="ouster_model" value="${optionals['ouster_model']}" />
     <!-- OS1-16 Generation 1 (default) -->
     <xacro:property name="sensor_name" value="os1" />
@@ -729,5 +729,5 @@
     max_range="${range}"
     noise="0.03"
-    enable_gpu_ray="$(arg use_gpu_ray)"
+    enable_gpu_ray="${optionals['use_gpu_ray']}"
     >
   </xacro:ouster_macro>
@@ -813,5 +813,5 @@
       camera_suffix="realsense_down"
       parent_frame_name="${namespace}/fcu"
-      enable_realistic_realsense="$(arg use_realistic_realsense)"
+      enable_realistic_realsense="${optionals['use_realistic_realsense']}"
       x="0.153"
       y="0"
@@ -831,5 +831,5 @@
       camera_suffix="realsense_front_pitched"
       parent_frame_name="${namespace}/fcu"
-      enable_realistic_realsense="$(arg use_realistic_realsense)"
+      enable_realistic_realsense="${optionals['use_realistic_realsense']}"
       x="0.16"
       y="0"
@@ -849,5 +849,5 @@
       camera_suffix="realsense_front"
       parent_frame_name="${namespace}/fcu"
-      enable_realistic_realsense="$(arg use_realistic_realsense)"
+      enable_realistic_realsense="${optionals['use_realistic_realsense']}"
       x="0.155"
       y="0"
@@ -867,5 +867,5 @@
       camera_suffix="realsense_up"
       parent_frame_name="${namespace}/fcu"
-      enable_realistic_realsense="$(arg use_realistic_realsense)"
+      enable_realistic_realsense="${optionals['use_realistic_realsense']}"
       x="0.07"
       y="0"
@@ -968,6 +968,6 @@
       frame_rate="80"
       camera_publish_topic="/${namespace}/uvdar_bluefox_left/image_raw"
-      calibration_file="$(arg uvcam_calib_file)"
-      occlusions="$(arg uvcam_occlusions)">
+      calibration_file="${optionals['uvcam_calib_file']}"
+      occlusions="${optionals['uvcam_occlusions']}">
     <origin xyz="0.037 0.1175 0.05" rpy="0 0 ${rad70}" />
     </xacro:uvcam_macro>
@@ -978,6 +978,6 @@
       frame_rate="80"
       camera_publish_topic="/${namespace}/uvdar_bluefox_right/image_raw"
-      calibration_file="$(arg uvcam_calib_file)"
-      occlusions="$(arg uvcam_occlusions)">
+      calibration_file="${optionals['uvcam_calib_file']}"
+      occlusions="${optionals['uvcam_occlusions']}">
     <origin xyz="0.037 -0.1175 0.05" rpy="0 0 -${rad70}" />
     </xacro:uvcam_macro>
@@ -1102,6 +1102,6 @@
   <xacro:if value="${optionals['enable_uv_leds']}">
     <xacro:uvled_quadrotor
-      f1="$(arg uvled_fr_l)"
-      f2="$(arg uvled_fr_r)"
+      f1="${optionals['uvled_fr_l']}"
+      f2="${optionals['uvled_fr_r']}"
       namespace="${namespace}"
       parent_link="base_link"/>
@@ -1146,5 +1146,5 @@
     <xacro:uvled_beacon
       height="0.15"
-      f="$(arg uvled_beacon_f)"
+      f="${optionals['uvled_beacon_f']}"
       namespace="${namespace}"
       parent_link="base_link"/>

File: models/mrs_robots_description/urdf/f550.xacro (robot description, xacro)
@@ -6,4 +6,6 @@
   -->
   <xacro:property name="namespace" value="$(arg namespace)" />
+  <xacro:property name='model_params_file' value="$(arg model_params_file)"/>
+  <xacro:property name="optionals" value="${load_yaml(model_params_file)}" />
   <xacro:arg name='name' default='f550' />
   <xacro:arg name='mavlink_addr' default='INADDR_ANY' />
@@ -568,5 +570,5 @@
   <!-- ================================================================== -->
   <!-- Ground truth {-->
-  <xacro:if value="$(arg enable_ground_truth)">
+  <xacro:if value="${optionals['enable_ground_truth']}">
     <!-- Mount a generic odometry sensor providing ground truth. -->
     <xacro:odometry_plugin_macro
@@ -588,5 +590,5 @@
   <!-- ======================= rangefinder sensors ======================-->
   <!-- Garmin {-->
-  <xacro:if value="$(arg enable_rangefinder)">
+  <xacro:if value="${optionals['enable_rangefinder']}">
     <xacro:garmin_macro
       namespace="${namespace}"
@@ -604,5 +606,5 @@
   <!--}-->
   <!-- Garmin looking up {-->
-  <xacro:if value="$(arg enable_rangefinder_up)">
+  <xacro:if value="${optionals['enable_rangefinder_up']}">
     <xacro:garmin_macro
       namespace="${namespace}"
@@ -620,5 +622,5 @@
   <!--}-->
   <!-- Teraranger One {-->
-  <xacro:if value="$(arg enable_teraranger)">
+  <xacro:if value="${optionals['enable_teraranger']}">
     <xacro:teraranger_macro
       namespace="${namespace}"
@@ -636,5 +638,5 @@
   <!-- ========================== LIDAR sensors ========================= -->
   <!-- Scanse Sweep {-->
-  <xacro:if value="$(arg enable_scanse_sweep)">
+  <xacro:if value="${optionals['enable_scanse_sweep']}">
     <xacro:scanse_sweep_macro
       namespace="${namespace}"
@@ -650,5 +652,5 @@
   <!--}-->
   <!-- Rplidar {-->
-  <xacro:if value="$(arg enable_rplidar)">
+  <xacro:if value="${optionals['enable_rplidar']}">
     <xacro:rplidar_macro
       namespace="${namespace}"
@@ -664,5 +666,5 @@
   <!--}-->
   <!-- Velodyne  {-->
-  <xacro:if value="$(arg enable_velodyne)">
+  <xacro:if value="${optionals['enable_velodyne']}">
     <!-- VLP-16 (default) -->
     <xacro:property name="sensor_name" value="velodyne" />
@@ -684,5 +686,5 @@
       max_range="${range}"
       noise="0.01"
-      enable_gpu_ray="$(arg use_gpu_ray)"
+      enable_gpu_ray="${optionals['use_gpu_ray']}"
       >
     </xacro:velodyne_macro>
@@ -690,6 +692,6 @@
   <!--}-->
   <!-- Ouster {-->
-  <xacro:if value="$(arg enable_ouster)">
-  <xacro:property name="ouster_model" value="$(arg ouster_model)" />
+  <xacro:if value="${optionals['enable_ouster']}">
+    <xacro:property name="ouster_model" value="${optionals['ouster_model']}" />
     <!-- OS1-16 Generation 1 (default) -->
     <xacro:property name="sensor_name" value="os1" />
@@ -786,5 +788,5 @@
     max_range="${range}"
     noise="0.03"
-    enable_gpu_ray="$(arg use_gpu_ray)"
+    enable_gpu_ray="${optionals['use_gpu_ray']}"
     >
   </xacro:ouster_macro>
@@ -794,5 +796,5 @@
   <!-- Bluefox placements{-->
   <!-- reverse {-->
-  <xacro:if value="$(arg enable_bluefox_camera_reverse)">
+  <xacro:if value="${optionals['enable_bluefox_camera_reverse']}">
     <xacro:bluefox_camera_macro
       namespace="${namespace}"
@@ -816,5 +818,5 @@
   <!--}-->
   <!-- classic {-->
-  <xacro:if value="$(arg enable_bluefox_camera)">
+  <xacro:if value="${optionals['enable_bluefox_camera']}">
     <xacro:bluefox_camera_macro
       namespace="${namespace}"
@@ -840,5 +842,5 @@
   <!-- Realsense placements {-->
   <!-- top {-->
-  <xacro:if value="$(arg enable_realsense_top)">
+  <xacro:if value="${optionals['enable_realsense_top']}">
     <!-- sensor -->
     <xacro:realsense_macro
@@ -847,5 +849,5 @@
       camera_suffix="realsense_top"
       parent_frame_name="${namespace}/fcu"
-      enable_realistic_realsense="$(arg use_realistic_realsense)"
+      enable_realistic_realsense="${optionals['use_realistic_realsense']}"
       x="0.085"
       y="-0.041"
@@ -858,5 +860,5 @@
   <!--}-->
   <!-- down {-->
-  <xacro:if value="$(arg enable_realsense_down)">
+  <xacro:if value="${optionals['enable_realsense_down']}">
     <xacro:realsense_macro
       namespace="${namespace}"
@@ -864,5 +866,5 @@
       camera_suffix="realsense_down"
       parent_frame_name="${namespace}/fcu"
-      enable_realistic_realsense="$(arg use_realistic_realsense)"
+      enable_realistic_realsense="${optionals['use_realistic_realsense']}"
       x="0.22"
       y="0"
@@ -875,5 +877,5 @@
   <!--}-->
   <!-- front pitched {-->
-  <xacro:if value="$(arg enable_realsense_front_pitched)">
+  <xacro:if value="${optionals['enable_realsense_front_pitched']}">
     <!-- sensor -->
     <xacro:realsense_macro
@@ -882,5 +884,5 @@
       camera_suffix="realsense_front_pitched"
       parent_frame_name="${namespace}/fcu"
-      enable_realistic_realsense="$(arg use_realistic_realsense)"
+      enable_realistic_realsense="${optionals['use_realistic_realsense']}"
       x="0.226"
       y="0"
@@ -896,5 +898,5 @@
   <!--}-->
   <!-- front {-->
-  <xacro:if value="$(arg enable_realsense_front)">
+  <xacro:if value="${optionals['enable_realsense_front']}">
     <!-- sensor -->
     <xacro:realsense_macro
@@ -903,5 +905,5 @@
       camera_suffix="realsense_front"
       parent_frame_name="${namespace}/fcu"
-      enable_realistic_realsense="$(arg use_realistic_realsense)"
+      enable_realistic_realsense="${optionals['use_realistic_realsense']}"
       x="0.223"
       y="0"
@@ -914,5 +916,5 @@
   <!--}-->
   <!-- up {-->
-  <xacro:if value="$(arg enable_realsense_up)">
+  <xacro:if value="${optionals['enable_realsense_up']}">
     <!-- sensor -->
     <xacro:realsense_macro
@@ -921,5 +923,5 @@
       camera_suffix="realsense_up"
       parent_frame_name="${namespace}/fcu"
-      enable_realistic_realsense="$(arg use_realistic_realsense)"
+      enable_realistic_realsense="${optionals['use_realistic_realsense']}"
       x="0.07"
       y="0"
@@ -934,5 +936,5 @@
   <!-- Mobius placements {-->
   <!-- down {-->
-  <xacro:if value="$(arg enable_mobius_camera_down)">
+  <xacro:if value="${optionals['enable_mobius_camera_down']}">
     <xacro:mobius_camera_macro
       namespace="${namespace}"
@@ -954,5 +956,5 @@
   <!--}-->
   <!-- front {-->
-  <xacro:if value="$(arg enable_mobius_camera_front)">
+  <xacro:if value="${optionals['enable_mobius_camera_front']}">
     <xacro:mobius_camera_macro
       namespace="${namespace}"
@@ -974,5 +976,5 @@
   <!--}-->
   <!-- back left {-->
-  <xacro:if value="$(arg enable_mobius_camera_back_left)">
+  <xacro:if value="${optionals['enable_mobius_camera_back_left']}">
     <xacro:mobius_camera_macro
       namespace="${namespace}"
@@ -994,5 +996,5 @@
   <!--}-->
   <!-- back right {-->
-  <xacro:if value="$(arg enable_mobius_camera_back_right)">
+  <xacro:if value="${optionals['enable_mobius_camera_back_right']}">
     <xacro:mobius_camera_macro
       namespace="${namespace}"
@@ -1015,5 +1017,5 @@
   <!--} Mobius placements -->
   <!-- UV camera {-->
-  <xacro:if value="$(arg enable_uv_camera)">
+  <xacro:if value="${optionals['enable_uv_camera']}">
     <xacro:uvcam_macro
       namespace="${namespace}"
@@ -1022,5 +1024,5 @@
       frame_rate="80"
       camera_publish_topic="/${namespace}/uvdar_bluefox_left/image_raw"
-      calibration_file="$(arg uvcam_calib_file)">
+      calibration_file="${optionals['uvcam_calib_file']}">
     <origin xyz="0.037 0.1175 0.05" rpy="0 0 ${rad70}" />
     </xacro:uvcam_macro>
@@ -1031,5 +1033,5 @@
       frame_rate="80"
       camera_publish_topic="/${namespace}/uvdar_bluefox_right/image_raw"
-      calibration_file="$(arg uvcam_calib_file)">
+      calibration_file="${optionals['uvcam_calib_file']}">
     <origin xyz="0.037 -0.1175 0.05" rpy="0 0 -${rad70}" />
     </xacro:uvcam_macro>
@@ -1037,5 +1039,5 @@
   <!--}-->
   <!-- Servo camera {-->
-  <xacro:if value="$(arg enable_servo_camera)">
+  <xacro:if value="${optionals['enable_servo_camera']}">
     <xacro:servo_camera_macro
       namespace="${namespace}"
@@ -1056,5 +1058,5 @@
   <!-- ========================== other sensors ========================= -->
   <!-- Teraranger Tower Evo {-->
-  <xacro:if value="$(arg enable_teraranger_tower_evo)">
+  <xacro:if value="${optionals['enable_teraranger_tower_evo']}">
     <xacro:teraranger_tower_evo_macro
       namespace="${namespace}"
@@ -1068,5 +1070,5 @@
   <!--}-->
   <!-- Magnetic gripper {-->
-  <xacro:if value="$(arg enable_magnetic_gripper)">
+  <xacro:if value="${optionals['enable_magnetic_gripper']}">
     <xacro:magnet_gripper_macro
       namespace="${namespace}"
@@ -1079,5 +1081,5 @@
   <!--}-->
   <!-- Timepix {-->
-  <xacro:if value="$(arg enable_timepix)">
+  <xacro:if value="${optionals['enable_timepix']}">
     <xacro:timepix_macro
       namespace="${namespace}"
@@ -1138,8 +1140,8 @@
   </xacro:macro>
   <!--}-->
-  <xacro:if value="$(arg enable_uv_leds)">
+  <xacro:if value="${optionals['enable_uv_leds']}">
     <xacro:uvled_hexarotor
-      f1="$(arg uvled_fr_l)"
-      f2="$(arg uvled_fr_r)"
+      f1="$(arg uvled_fr_l']}"
+      f2="$(arg uvled_fr_r']}"
       namespace="${namespace}"
       parent_link="base_link"/>
@@ -1147,5 +1149,5 @@
   <!--}-->
   <!-- Light {-->
-  <xacro:if value="$(arg enable_light)">
+  <xacro:if value="${optionals['enable_light']}">
     <xacro:light_macro
       namespace="${namespace}"
@@ -1169,5 +1171,5 @@
   <!-- ============================= holders ============================ -->
   <!-- Ouster and Velodyne mount {-->
-  <xacro:if value="${('$(arg enable_ouster)' == 'true') or ('$(arg enable_velodyne)' == 'true')}">
+  <xacro:if value="${(optionals['enable_ouster'] == 'true') or (optionals['enable_velodyne'] == 'true')}">
     <xacro:visual_macro
       robot_namespace="${namespace}"
@@ -1182,5 +1184,5 @@
   <!--}-->
   <!-- Rplidar and scanse mount {-->
-  <xacro:if value="${('$(arg enable_rplidar)' == 'true') or ('$(arg enable_scanse_sweep)' == 'true')}">
+  <xacro:if value="${(optionals['enable_rplidar'] == 'true') or (optionals['enable_scanse_sweep'] == 'true')}">
     <xacro:visual_macro
       robot_namespace="${namespace}"
@@ -1195,5 +1197,5 @@
   <!--}-->
   <!-- Realsense top mount {-->
-  <xacro:if value="$(arg enable_realsense_top)">
+  <xacro:if value="${optionals['enable_realsense_top']}">
     <xacro:visual_macro
       robot_namespace="${namespace}"
@@ -1208,5 +1210,5 @@
   <!--}-->
   <!-- Realsense front mount {-->
-  <xacro:if value="$(arg enable_realsense_front)">
+  <xacro:if value="${optionals['enable_realsense_front']}">
     <xacro:visual_macro
       robot_namespace="${namespace}"
@@ -1221,5 +1223,5 @@
   <!--}-->
   <!-- Realsense front pitched mount {-->
-  <xacro:if value="$(arg enable_realsense_front_pitched)">
+  <xacro:if value="${optionals['enable_realsense_front_pitched']}">
     <xacro:visual_macro
       robot_namespace="${namespace}"
@@ -1234,5 +1236,5 @@
   <!--}-->
   <!-- Realsense down mount {-->
-  <xacro:if value="$(arg enable_realsense_down)">
+  <xacro:if value="${optionals['enable_realsense_down']}">
     <xacro:visual_macro
       robot_namespace="${namespace}"
@@ -1247,5 +1249,5 @@
   <!--}-->
   <!-- UVDAR mount {-->
-  <xacro:if value="$(arg enable_uv_camera)">
+  <xacro:if value="${optionals['enable_uv_camera']}">
     <xacro:visual_macro
       robot_namespace="${namespace}"
@@ -1260,5 +1262,5 @@
   <!--}-->
   <!-- left leg for front sensors between legs (realsenses) {-->
-  <xacro:if value="${('$(arg enable_realsense_front)' == 'true') or ('$(arg enable_realsense_front_pitched)' == 'true') or ('$(arg enable_realsense_down)' == 'true')}">
+  <xacro:if value="${(optionals['enable_realsense_front'] == 'true') or (optionals['enable_realsense_front_pitched'] == 'true') or (optionals['enable_realsense_down'] == 'true')}">
     <xacro:leg_macro
       robot_namespace="${namespace}"
@@ -1327,5 +1329,5 @@
   </xacro:macro>
   <!--}-->
-  <xacro:if value="${('$(arg enable_realsense_top)' == 'true')}">
+  <xacro:if value="${optionals['enable_realsense_top']}">
     <xacro:top_holder_macro
       namespace="${namespace}"
@@ -1337,5 +1339,5 @@
   <!-- ========================== other sensors ========================= -->
 <!-- Whycon box {-->
-<xacro:if value="$(arg enable_whycon_box)">
+<xacro:if value="${optionals['enable_whycon_box']}">
   <xacro:box_macro
     robot_namespace="${namespace}"
@@ -1348,5 +1350,5 @@
 <!--}-->
 <!-- Pendulum {-->
-<xacro:if value="$(arg enable_pendulum)">
+<xacro:if value="${optionals['enable_pendulum']}">
   <xacro:pendulum
     parent="base_link">
@@ -1355,5 +1357,5 @@
 <!--}-->
 <!-- Ball holder {-->
-<xacro:if value="$(arg enable_ball_holder)">
+<xacro:if value="${optionals['enable_ball_holder']}">
   <xacro:ball_holder
       parent="base_link">

Commit message: minor naming update

File: models/mrs_robots_description/urdf/f450.xacro (robot description, xacro)
@@ -6,6 +6,6 @@
   -->
   <xacro:property name="namespace" value="$(arg namespace)" />
-  <xacro:property name='model_params_file' value="$(arg model_params_file)"/>
-  <xacro:property name="optionals" value="${load_yaml(model_params_file)}" />
+  <xacro:property name='model_config_file' value="$(arg model_config_file)"/>
+  <xacro:property name="optionals" value="${load_yaml(model_config_file)}" />
   <xacro:arg name='name' default='f450' />
   <xacro:arg name='mavlink_addr' default='INADDR_ANY' />

File: models/mrs_robots_description/urdf/f550.xacro (robot description, xacro)
@@ -6,6 +6,6 @@
   -->
   <xacro:property name="namespace" value="$(arg namespace)" />
-  <xacro:property name='model_params_file' value="$(arg model_params_file)"/>
-  <xacro:property name="optionals" value="${load_yaml(model_params_file)}" />
+  <xacro:property name='model_config_file' value="$(arg model_config_file)"/>
+  <xacro:property name="optionals" value="${load_yaml(model_config_file)}" />
   <xacro:arg name='name' default='f550' />
   <xacro:arg name='mavlink_addr' default='INADDR_ANY' />

File: models/mrs_robots_description/urdf/t650.xacro (robot description, xacro)
@@ -6,6 +6,6 @@
   -->
   <xacro:property name="namespace" value="$(arg namespace)" />
-  <xacro:property name='model_params_file' value="$(arg model_params_file)"/>
-  <xacro:property name="optionals" value="${load_yaml(model_params_file)}" />
+  <xacro:property name='model_config_file' value="$(arg model_config_file)"/>
+  <xacro:property name="optionals" value="${load_yaml(model_config_file)}" />
   <xacro:arg name='name' default='t650' />
   <xacro:arg name='mavlink_addr' default='INADDR_ANY' />

Commit message: add spawning poses loading

File: models/mrs_robots_description/urdf/f450.xacro (robot description, xacro)
@@ -48,5 +48,5 @@
   <xacro:property name="board_height" value="0.002" /> <!-- [m] -->
   <xacro:property name="holder_offset" value="0.02" /> <!-- [m] -->
-  <xacro:property name="leg_offset_z" value="0.098" />
+  <xacro:property name="leg_offset_z" value="0.098" /> <!-- [m] -->
   <!-- <xacro:property name="leg_offset_z" value="0.133" /> -->
   <xacro:property name="leg_offset_r" value="0.0072" /> <!-- [m] -->
@@ -803,5 +803,5 @@
 </xacro:if>
 <!--}-->
-  <!--} Bluefox placements -->
+  <!--} Other camera placements -->
   <!-- Realsense placements {-->
   <!-- down {-->

File: models/mrs_robots_description/urdf/t650.xacro (robot description, xacro)
@@ -45,5 +45,5 @@
   <xacro:property name="propeller_offset" value="0.01" /> <!-- [m] -->
   <xacro:property name="arm_length" value="0.3" /> <!-- [m] -->
-  <xacro:property name="leg_height" value="0.24" />
+  <xacro:property name="leg_height" value="0.24" /> <!-- [m] -->
   <!-- <xacro:property name="leg_height" value="0.15" /> -->
   <xacro:property name="leg_offset_r" value="0.05" /> <!-- [m] -->

Commit message: updated f450 motor param

File: models/mrs_robots_description/urdf/f450.xacro (robot description, xacro)
@@ -56,5 +56,5 @@
   <!-- Motor constants {-->
   <xacro:property name="rotor_velocity_slowdown_sim" value="0.0159236" />
-  <xacro:property name="motor_constant" value="8.5" /> <!-- [kg.m/s^2] -->
+  <xacro:property name="motor_constant" value="10.04544" /> <!-- [kg.m/s^2] -->
   <xacro:property name="moment_constant" value="0.016" /> <!-- [m] -->
   <xacro:property name="time_constant_up" value="${1.0 / 80.0}" /> <!-- [s] -->

Commit message: Adding the third/back camera to simulation

File: models/mrs_robots_description/urdf/f450.xacro (robot description, xacro)
@@ -987,6 +987,6 @@
   <!--}-->
   <!--} Mobius placements -->
-  <!-- UV camera {-->
-  <xacro:if value="${optionals['enable_uv_camera']}">
+  <!-- Dual UV cameras {-->
+  <xacro:if value="${optionals['enable_dual_uv_cameras']}">
     <xacro:uvcam_macro
       namespace="${namespace}"
@@ -997,5 +997,5 @@
       calibration_file="${optionals['uvcam_calib_file']}"
       occlusions="${optionals['uvcam_occlusions']}">
-    <origin xyz="0.037 0.1175 0.05" rpy="0 0 ${rad70}" />
+    <origin xyz="0.03 0.10 0.06" rpy="0 0 ${rad70}" />
     </xacro:uvcam_macro>
     <xacro:uvcam_macro
@@ -1007,5 +1007,19 @@
       calibration_file="${optionals['uvcam_calib_file']}"
       occlusions="${optionals['uvcam_occlusions']}">
-    <origin xyz="0.037 -0.1175 0.05" rpy="0 0 -${rad70}" />
+    <origin xyz="0.03 -0.10 0.06" rpy="0 0 -${rad70}" />
+    </xacro:uvcam_macro>
+  </xacro:if>
+  <!--}-->
+  <!-- Back UV camera {-->
+  <xacro:if value="${optionals['enable_back_uv_camera']}">
+    <xacro:uvcam_macro
+      namespace="${namespace}"
+      parent_link="base_link"
+      number="3"
+      frame_rate="60"
+      camera_publish_topic="/${namespace}/uvdar_bluefox_back/image_raw"
+      calibration_file="${optionals['uvcam_calib_file']}"
+      occlusions="${optionals['uvcam_occlusions']}">
+    <origin xyz="-0.1 0.0 -0.02" rpy="${rad90} 0 ${rad180}" />
     </xacro:uvcam_macro>
   </xacro:if>
@@ -1294,5 +1308,5 @@
   <!--}-->
   <!-- UVDAR mount {-->
-  <xacro:if value="${optionals['enable_uv_camera']}">
+  <xacro:if value="${optionals['enable_dual_uv_cameras']}">
     <xacro:visual_macro
       robot_namespace="${namespace}"

Commit message: Implemented f550.sdf.jinja, changed f450.sdf.jinja Copied rotor file from f550/ and renamed it to dji_f450_rotor

File: models/mrs_robots_description/urdf/f450.xacro (robot description, xacro)
@@ -328,5 +328,5 @@
     mesh_scale="${mesh_scale_prop_ccw}"
     color="White">
-    <origin xyz="${arm_length * sin45} -${arm_length * sin45} ${arm_height + rotor_offset_top - body_height/2}"  rpy="0 0 0" />
+    <origin xyz="${arm_length_battery_mount = tr * sin45} -${arm_length * sin45} ${arm_height + rotor_offset_top - body_height/2}"  rpy="0 0 0" />
     <xacro:insert_block name="rotor_inertia" />
   </xacro:vertical_rotor>

Commit message: Accidently changed f450.xarco, changing in back

File: models/mrs_robots_description/urdf/f450.xacro (robot description, xacro)
@@ -328,5 +328,5 @@
     mesh_scale="${mesh_scale_prop_ccw}"
     color="White">
-    <origin xyz="${arm_length_battery_mount = tr * sin45} -${arm_length * sin45} ${arm_height + rotor_offset_top - body_height/2}"  rpy="0 0 0" />
+    <origin xyz="${arm_length * sin45} -${arm_length * sin45} ${arm_height + rotor_offset_top - body_height/2}"  rpy="0 0 0" />
     <xacro:insert_block name="rotor_inertia" />
   </xacro:vertical_rotor>
